File: kicad/cm4-robo-controller.kicad_sch (KiCad schematic)
At the start: 10 parts, among them J1 KF7620-7.62-2P

Commit message: Mods
Parts:
- added D50: SMCJ18A_C53260906, MyParts:SMC_L6.9-W5.9-LS7.9-RD, symbol MyParts:SMCJ18A_C53260906
- added D59: BZT52C15, MyParts:SOD-123_L2.7-W1.6-LS3.7-RD, symbol MyParts:BZT52C15
- added F2: 15A, MyParts:FUSE-TH_4P-L19.8-W6.7_3557-2, symbol MyParts:3557-2
- added Q12: SP40P04NK, MyParts:PDFN-8_L6.0-W5.0-P1.27_HGQ065NE4A, symbol MyParts:SP40P04NK
- added R139: 47kΩ, MyParts:R0402, symbol MyParts:0402WGF4702TCE
- added TP28, TP29: TestPoint_Small, TestPoint:TestPoint_Pad_D1.5mm, symbol Connector:TestPoint_Small
- F1: footprint MyParts:F1206 -> MyParts:FUSE-TH_4P-L19.8-W6.7_3557-2; symbol MyParts:BSMD1206C-1500T -> MyParts:3557-2; Fuse (none) -> Littelfuse 0287005.PXCN (ATO 5A); LCSC Part C41367229 -> C352820; MPN BSMD1206C-1500T -> 3557-2; Manufacturer BHFUSE -> Keystone; Pkg Type SMD 1206 -> THT
Connections:
- net CHASSIS: now also TP28.1
- net PGND: now also D50.2 (A), R139.2
- net V_BAT: now also F1.2
- net at J1.1: now also Q12.5 (D), Q12.6 (D), Q12.7 (D), Q12.8 (D), Q12.9 (D); no longer F1.2
- new net: D59.1 (K), F1.3, F1.4, F2.3, F2.4, Q12.1 (S), Q12.2 (S), Q12.3 (S)
- new net: D59.2 (A), Q12.4 (G), R139.1
- new net V_MOTOR: D50.1 (C), F2.1, F2.2, TP29.1
Other:
- sheet GPS ports: added 5V; removed none
- sheet Robo ports: added V_MOTOR; removed V_BAT
- note added: "Give Q12's drain tab a solid copper pour; it dissipates about 0.55 W worst case."
- note added: "V_BAT (J1): 12.8 V nom, 10.0 V min, 14.6 V max (charging). Survives 18 V max (TVS). Reverse battery: Q12 P-FET blocks it; survives -14.6 V, nothing conducts, no fuse blows."
- note added: "V_MOTOR (A1 BAT+, via F2 15 A): motors 7.5 A max (F-SD-H-450 actuator 5.5 A + worm motor 2 A). F1 5 A feeds the CM4 board branch (V_BAT) only. F1/F2: Keystone 3557-2 holders; fit Littelfuse ATO 0287005.PXCN (5 A) / 0287015.PXCN (15 A)."
- note removed: "V_BAT (J1): 12.8 V nom, 10.0 V min, 14.6 V max (charging). Survives 18 V max (TVS); reverse: D2 clamps -1 V, F1 opens."
- moved on the sheet: D2, J1
