File: kicad/cm4-robo-controller.kicad_sch (KiCad schematic)
At the start: 9 parts

Commit message: IPC footprint renaming, battery sim added
Parts:
- C1: footprint MyParts:C1206 -> MyPartsIPC:CAPC3216X180N
- R2: footprint MyParts:R1206 -> MyPartsIPC:RESC3216X70N
- TP1, TP2: now left out of the parts list
Changed lines of the file:
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@@
-		)
-	)
-	(netclass_flag ""
-		(length 2.54)
-		(shape round)
-		(at 119.38 77.47 0)
-		(effects
-			(font
-				(size 1.27 1.27)
-			)
-			(justify left top)
-		)
-		(property "Net Class" "V_BAT"
-			(at 119.38 73.152 0)
-			(show_name no)
-			(do_not_autoplace no)
-			(effects
-				(font
-					(size 1.27 1.27)
-					(italic yes)
-				)
-			)
-		)
-		(property "VOLTAGE_NOM" "12.8V"
-			(at 119.38 71.12 0)
-			(hide yes)
-			(show_name no)
-			(do_not_autoplace no)
-			(effects
-				(font
-					(size 1.27 1.27)
-				)
-			)
-		)
-		(property "VOLTAGE_MIN" "10.0V"
-			(at 119.38 71.12 0)
-			(hide yes)
-			(show_name no)
-			(do_not_autoplace no)
-			(effects
-				(font
-					(size 1.27 1.27)
-				)
-			)
-		)
-		(property "VOLTAGE_MAX" "14.6V"
-			(at 119.38 71.12 0)
-			(hide yes)
-			(show_name no)
-			(do_not_autoplace no)
-			(effects
-				(font
-					(size 1.27 1.27)
-				)
-			)
-		)
-		(property "VOLTAGE_EXCURSION_MAX" "18.0V"
-			(at 119.38 71.12 0)
-			(hide yes)
-			(show_name no)
-			(do_not_autoplace no)
-			(effects
-				(font
-					(size 1.27 1.27)
-				)
-			)
 		)
 	)
@@
 		(body_style 1)
 		(exclude_from_sim no)
-		(in_bom yes)
+		(in_bom no)
 		(on_board yes)
 		(in_pos_files yes)
@@
 			)
 		)
-		(property "Footprint" "MyParts:R1206"
+		(property "Footprint" "MyPartsIPC:RESC3216X70N"
 			(at 91.44 161.29 0)
 			(hide yes)
@@
 			)
 		)
-		(property "Footprint" "MyParts:C1206"
+		(property "Footprint" "MyPartsIPC:CAPC3216X180N"
 			(at 91.44 171.45 0)
 			(hide yes)
@@
 		(body_style 1)
 		(exclude_from_sim no)
-		(in_bom yes)
+		(in_bom no)
 		(on_board yes)
 		(in_pos_files yes)
