File: kicad/RCM4.kicad_sch (KiCad schematic)
At the start: 19 parts, among them U19 74LVC1G07SE-7

Commit message: Ready to start layout
Parts:
- renumbered C108 to C2, D54 to D4, D55 to D5, LED3 to LED2, R5 to R3, R3 to R4, R4 to R5, R134 to R6, R133 to R7, R132 to R8, R131 to R9, TP13 to TP3, TP30 to TP4, TP22 to TP5, TP12 to TP6, TP14 to TP7, U19 to U1
Changed lines of the file:
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@@
 		(in_pos_files yes)
 		(dnp no)
-		(property "Reference" "TP30"
+		(property "Reference" "TP4"
 			(at 151.384 134.366 0)
 			(show_name no)
@@
 			(project "cm4-robo-controller"
 				(path "/c1285fbe-5f56-49a8-9041-410713cbe619/3cc0f123-2315-4414-aa85-3a1a0bb694eb"
-					(reference "TP30")
+					(reference "TP4")
 					(unit 1)
 				)
@@
 		(in_pos_files yes)
 		(dnp no)
-		(property "Reference" "R133"
+		(property "Reference" "R7"
 			(at 35.56 149.098 90)
 			(show_name no)
@@
 			(project "cm4-robo-controller"
 				(path "/c1285fbe-5f56-49a8-9041-410713cbe619/3cc0f123-2315-4414-aa85-3a1a0bb694eb"
-					(reference "R133")
+					(reference "R7")
 					(unit 1)
 				)
@@
 		(in_pos_files yes)
 		(dnp no)
-		(property "Reference" "R131"
+		(property "Reference" "R9"
 			(at 151.13 185.674 90)
 			(show_name no)
@@
 			(project "cm4-robo-controller"
 				(path "/c1285fbe-5f56-49a8-9041-410713cbe619/3cc0f123-2315-4414-aa85-3a1a0bb694eb"
-					(reference "R131")
+					(reference "R9")
 					(unit 1)
 				)
@@
 		(in_pos_files yes)
 		(dnp no)
-		(property "Reference" "LED3"
+		(property "Reference" "LED2"
 			(at 139.7 191.135 0)
 			(show_name no)
@@
 			(project "cm4-robo-controller"
 				(path "/c1285fbe-5f56-49a8-9041-410713cbe619/3cc0f123-2315-4414-aa85-3a1a0bb694eb"
-					(reference "LED3")
+					(reference "LED2")
 					(unit 1)
 				)
@@
 		(dnp no)
 		(fields_autoplaced yes)
-		(property "Reference" "R5"
+		(property "Reference" "R3"
 			(at 135.89 48.2599 0)
 			(show_name no)
@@
 			(project "cm4-robo-controller"
 				(path "/c1285fbe-5f56-49a8-9041-410713cbe619/3cc0f123-2315-4414-aa85-3a1a0bb694eb"
-					(reference "R5")
+					(reference "R3")
 					(unit 1)
 				)
@@
 		(in_pos_files yes)
 		(dnp no)
-		(property "Reference" "R134"
+		(property "Reference" "R6"
 			(at 35.56 143.002 90)
 			(show_name no)
@@
 			(project "cm4-robo-controller"
 				(path "/c1285fbe-5f56-49a8-9041-410713cbe619/3cc0f123-2315-4414-aa85-3a1a0bb694eb"
-					(reference "R134")
+					(reference "R6")
 					(unit 1)
 				)
@@
 		(in_pos_files yes)
 		(dnp no)
-		(property "Reference" "R132"
+		(property "Reference" "R8"
 			(at 95.885 175.895 0)
 			(show_name no)
@@
 			(project "cm4-robo-controller"
 				(path "/c1285fbe-5f56-49a8-9041-410713cbe619/3cc0f123-2315-4414-aa85-3a1a0bb694eb"
-					(reference "R132")
+					(reference "R8")
 					(unit 1)
 				)
@@
 		(in_pos_files no)
 		(dnp no)
-		(property "Reference" "TP22"
+		(property "Reference" "TP5"
 			(at 152.4 142.24 0)
 			(show_name no)
@@
 			(project "rcm_dish_controller"
 				(path "/10d7c3e5-be4d-4306-a59e-500b86bd141f/a4b43769-68f4-4111-a02f-817ae260783a"
-					(reference "TP22")
+					(reference "TP5")
 					(unit 1)
 				)
@@
 			(project "cm4-robo-controller"
 				(path "/c1285fbe-5f56-49a8-9041-410713cbe619/3cc0f123-2315-4414-aa85-3a1a0bb694eb"
-					(reference "TP22")
+					(reference "TP5")
 					(unit 1)
 				)
@@
 		(in_pos_files no)
 		(dnp no)
-		(property "Reference" "TP14"
+		(property "Reference" "TP7"
 			(at 128.27 186.182 0)
 			(show_name no)
@@
 			(project "rcm_dish_controller"
 				(path "/10d7c3e5-be4d-4306-a59e-500b86bd141f/a4b43769-68f4-4111-a02f-817ae260783a"
-					(reference "TP14")
+					(reference "TP7")
 					(unit 1)
 				)
@@
 			(project "cm4-robo-controller"
 				(path "/c1285fbe-5f56-49a8-9041-410713cbe619/3cc0f123-2315-4414-aa85-3a1a0bb694eb"
-					(reference "TP14")
+					(reference "TP7")
 					(unit 1)
 				)
@@
 		(in_pos_files yes)
 		(dnp no)
-		(property "Reference" "D54"
+		(property "Reference" "D4"
 			(at 41.91 167.005 0)
 			(show_name no)
@@
 			(project "cm4-robo-controller"
 				(path "/c1285fbe-5f56-49a8-9041-410713cbe619/3cc0f123-2315-4414-aa85-3a1a0bb694eb"
-					(reference "D54")
+					(reference "D4")
 					(unit 1)
 				)
@@
 		(in_pos_files no)
 		(dnp no)
-		(property "Reference" "TP12"
+		(property "Reference" "TP6"
 			(at 152.4 149.86 0)
 			(show_name no)
@@
 			(project "rcm_dish_controller"
 				(path "/10d7c3e5-be4d-4306-a59e-500b86bd141f/a4b43769-68f4-4111-a02f-817ae260783a"
-					(reference "TP12")
+					(reference "TP6")
 					(unit 1)
 				)
@@
 			(project "cm4-robo-controller"
 				(path "/c1285fbe-5f56-49a8-9041-410713cbe619/3cc0f123-2315-4414-aa85-3a1a0bb694eb"
-					(reference "TP12")
+					(reference "TP6")
 					(unit 1)
 				)
@@
 		(in_pos_files yes)
 		(dnp no)
-		(property "Reference" "U19"
+		(property "Reference" "U1"
 			(at 114.3 173.99 270)
 			(show_name no)
@@
 			(project "cm4-robo-controller"
 				(path "/c1285fbe-5f56-49a8-9041-410713cbe619/3cc0f123-2315-4414-aa85-3a1a0bb694eb"
-					(reference "U19")
+					(reference "U1")
 					(unit 1)
 				)
@@
 		(in_pos_files no)
 		(dnp no)
-		(property "Reference" "TP13"
+		(property "Reference" "TP3"
 			(at 130.81 41.91 0)
 			(show_name no)
@@
 			(project "rcm_dish_controller"
 				(path "/10d7c3e5-be4d-4306-a59e-500b86bd141f/a4b43769-68f4-4111-a02f-817ae260783a"
-					(reference "TP13")
+					(reference "TP3")
 					(unit 1)
 				)
@@
 			(project "cm4-robo-controller"
 				(path "/c1285fbe-5f56-49a8-9041-410713cbe619/3cc0f123-2315-4414-aa85-3a1a0bb694eb"
-					(reference "TP13")
+					(reference "TP3")
 					(unit 1)
 				)
@@
 		(in_pos_files yes)
 		(dnp no)
-		(property "Reference" "D55"
+		(property "Reference" "D5"
 			(at 41.91 177.165 0)
 			(show_name no)
@@
 			(project "cm4-robo-controller"
 				(path "/c1285fbe-5f56-49a8-9041-410713cbe619/3cc0f123-2315-4414-aa85-3a1a0bb694eb"
-					(reference "D55")
+					(reference "D5")
 					(unit 1)
 				)
@@
 		(in_pos_files yes)
 		(dnp no)
-		(property "Reference" "R3"
+		(property "Reference" "R4"
 			(at 43.434 66.294 90)
 			(show_name no)
@@
 			(project "cm4-robo-controller"
 				(path "/c1285fbe-5f56-49a8-9041-410713cbe619/3cc0f123-2315-4414-aa85-3a1a0bb694eb"
-					(reference "R3")
+					(reference "R4")
 					(unit 1)
 				)
@@
 		(in_pos_files yes)
 		(dnp no)
-		(property "Reference" "R4"
+		(property "Reference" "R5"
 			(at 43.434 91.694 90)
 			(show_name no)
@@
 			(project "cm4-robo-controller"
 				(path "/c1285fbe-5f56-49a8-9041-410713cbe619/3cc0f123-2315-4414-aa85-3a1a0bb694eb"
-					(reference "R4")
+					(reference "R5")
 					(unit 1)
 				)
@@
 		(in_pos_files yes)
 		(dnp no)
-		(property "Reference" "C108"
+		(property "Reference" "C2"
 			(at 139.065 173.355 0)
 			(show_name no)
@@
 			(project "cm4-robo-controller"
 				(path "/c1285fbe-5f56-49a8-9041-410713cbe619/3cc0f123-2315-4414-aa85-3a1a0bb694eb"
-					(reference "C108")
+					(reference "C2")
 					(unit 1)
 				)

Commit message: Added new sheets, motor notes
Parts:
- removed TP5, TP6: TestPoint_Small, TestPoint:TestPoint_Pad_D1.5mm, symbol Connector:TestPoint_Small
Other:
- note added: "CM4"
- note added: "Suggest a CM4004016. 4GB RAM, 8GB eMMC program storage."
Changed lines of the file:
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@@
 		)
 	)
+	(text "CM4"
+		(exclude_from_sim no)
+		(at 23.876 18.288 0)
+		(effects
+			(font
+				(size 5.08 5.08)
+			)
+		)
+	)
+	(text "Suggest a CM4004016.\n4GB RAM, 8GB eMMC program storage."
+		(exclude_from_sim no)
+		(at 136.906 17.526 0)
+		(effects
+			(font
+				(size 1.778 1.778)
+			)
+		)
+	)
 	(text "From the CM4 Manual:\nActive-low output to \ndrive Power On LED. \nThis signal needs to \nbe buffered."
 		(exclude_from_sim no)
@@
 	(wire
 		(pts
-			(xy 153.67 142.24) (xy 154.94 142.24)
-		)
-		(stroke
-			(width 0)
-			(type default)
-		)
-	)
-	(wire
-		(pts
 			(xy 252.73 30.48) (xy 247.65 30.48)
 		)
@@
 	(wire
 		(pts
-			(xy 153.67 149.86) (xy 154.94 149.86)
-		)
-		(stroke
-			(width 0)
-			(type default)
-		)
-	)
-	(wire
-		(pts
 			(xy 218.44 111.76) (xy 220.98 111.76)
 		)
@@
 	(symbol
 		(lib_id "Connector:TestPoint_Small")
-		(at 153.67 142.24 0)
-		(unit 1)
-		(body_style 1)
-		(exclude_from_sim no)
-		(in_bom no)
-		(on_board yes)
-		(in_pos_files no)
-		(dnp no)
-		(property "Reference" "TP5"
-			(at 152.4 142.24 0)
-			(show_name no)
-			(do_not_autoplace no)
-			(effects
-				(font
-					(size 1.27 1.27)
-				)
-				(justify right)
-			)
-		)
-		(property "Value" "TestPoint_Small"
-			(at 153.67 142.24 0)
-			(hide yes)
-			(show_name no)
-			(do_not_autoplace no)
-			(effects
-				(font
-					(size 1.27 1.27)
-				)
-			)
-		)
-		(property "Footprint" "TestPoint:TestPoint_Pad_D1.5mm"
-			(at 153.67 142.24 0)
-			(hide yes)
-			(show_name no)
-			(do_not_autoplace no)
-			(effects
-				(font
-					(size 1.27 1.27)
-				)
-			)
-		)
-		(property "Datasheet" ""
-			(at 153.67 142.24 0)
-			(hide yes)
-			(show_name no)
-			(do_not_autoplace no)
-			(effects
-				(font
-					(size 1.27 1.27)
-				)
-			)
-		)
-		(property "Description" "test point"
-			(at 153.67 142.24 0)
-			(hide yes)
-			(show_name no)
-			(do_not_autoplace no)
-			(effects
-				(font
-					(size 1.27 1.27)
-				)
-			)
-		)
-		(property "Pkg Type" "SMD Test pad D1.5"
-			(at 153.67 142.24 0)
-			(hide yes)
-			(show_name no)
-			(do_not_autoplace no)
-			(effects
-				(font
-					(size 1.27 1.27)
-				)
-			)
-		)
-		(pin "1"
-		)
-		(instances
-			(project "rcm_dish_controller"
-				(path "/10d7c3e5-be4d-4306-a59e-500b86bd141f/a4b43769-68f4-4111-a02f-817ae260783a"
-					(reference "TP5")
-					(unit 1)
-				)
-			)
-			(project "cm4-robo-controller"
-				(path "/c1285fbe-5f56-49a8-9041-410713cbe619/3cc0f123-2315-4414-aa85-3a1a0bb694eb"
-					(reference "TP5")
-					(unit 1)
-				)
-			)
-		)
-	)
-	(symbol
-		(lib_id "Connector:TestPoint_Small")
 		(at 128.27 184.15 0)
 		(unit 1)
@@
 					(unit 1)
 				)
-			)
-		)
-	)
-	(symbol
-		(lib_id "Connector:TestPoint_Small")
-		(at 153.67 149.86 0)
-		(unit 1)
-		(body_style 1)
-		(exclude_from_sim no)
-		(in_bom no)
-		(on_board yes)
-		(in_pos_files no)
-		(dnp no)
-		(property "Reference" "TP6"
-			(at 152.4 149.86 0)
-			(show_name no)
-			(do_not_autoplace no)
-			(effects
-				(font
-					(size 1.27 1.27)
-				)
-				(justify right)
-			)
-		)
-		(property "Value" "TestPoint_Small"
-			(at 153.67 149.86 0)
-			(hide yes)
-			(show_name no)
-			(do_not_autoplace no)
-			(effects
-				(font
-					(size 1.27 1.27)
-				)
-			)
-		)
-		(property "Footprint" "TestPoint:TestPoint_Pad_D1.5mm"
-			(at 153.67 149.86 0)
-			(hide yes)
-			(show_name no)
-			(do_not_autoplace no)
-			(effects
-				(font
-					(size 1.27 1.27)
-				)
-			)
-		)
-		(property "Datasheet" ""
-			(at 153.67 149.86 0)
-			(hide yes)
-			(show_name no)
-			(do_not_autoplace no)
-			(effects
-				(font
-					(size 1.27 1.27)
-				)
-			)
-		)
-		(property "Description" "test point"
-			(at 153.67 149.86 0)
-			(hide yes)
-			(show_name no)
-			(do_not_autoplace no)
-			(effects
-				(font
-					(size 1.27 1.27)
-				)
-			)
-		)
-		(property "Pkg Type" "SMD Test pad D1.5"
-			(at 153.67 149.86 0)
-			(hide yes)
-			(show_name no)
-			(do_not_autoplace no)
-			(effects
-				(font
-					(size 1.27 1.27)
-				)
-			)
-		)
-		(pin "1"
-		)
-		(instances
-			(project "rcm_dish_controller"
-				(path "/10d7c3e5-be4d-4306-a59e-500b86bd141f/a4b43769-68f4-4111-a02f-817ae260783a"
-					(reference "TP6")
-					(unit 1)
-				)
-			)
-			(project "cm4-robo-controller"
-				(path "/c1285fbe-5f56-49a8-9041-410713cbe619/3cc0f123-2315-4414-aa85-3a1a0bb694eb"
-					(reference "TP6")
-					(unit 1)
-				)

Commit message: IPC footprint renaming, battery sim added
Parts:
- C2: footprint MyParts:C0402 -> MyPartsIPC:CAPC1005X55N
- D4, D5: footprint MyParts:SOT-23-3_L2.9-W1.6-P1.90-LS2.8-BR -> MyPartsIPC:SOT95P280X110-3N
- LED1, LED2: footprint MyParts:LED0805-R-RD -> MyPartsIPC:LEDC2012X110N
- R3, R4, R5, R6, R7, R8, R9: footprint MyParts:R0402 -> MyPartsIPC:RESC1005X40N
- TP4: now left out of the parts list
- U1: footprint MyParts:SC-88A_L2.0-W1.3-P0.65-LS2.1-BL -> MyPartsIPC:SOT65P210X110-5N
Changed lines of the file:
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@@
 		(body_style 1)
 		(exclude_from_sim no)
-		(in_bom yes)
+		(in_bom no)
 		(on_board yes)
 		(in_pos_files yes)
@@
 			)
 		)
-		(property "Footprint" "MyParts:R0402"
+		(property "Footprint" "MyPartsIPC:RESC1005X40N"
 			(at 35.56 149.098 90)
 			(hide yes)
@@
 			)
 		)
-		(property "Footprint" "MyParts:LED0805-R-RD"
+		(property "Footprint" "MyPartsIPC:LEDC2012X110N"
 			(at 125.73 38.1 0)
 			(hide yes)
@@
 			)
 		)
-		(property "Footprint" "MyParts:R0402"
+		(property "Footprint" "MyPartsIPC:RESC1005X40N"
 			(at 151.13 187.96 0)
 			(hide yes)
@@
 			)
 		)
-		(property "Footprint" "MyParts:LED0805-R-RD"
+		(property "Footprint" "MyPartsIPC:LEDC2012X110N"
 			(at 139.7 186.69 0)
 			(hide yes)
@@
 			)
 		)
-		(property "Footprint" "MyParts:R0402"
+		(property "Footprint" "MyPartsIPC:RESC1005X40N"
 			(at 131.572 48.26 90)
 			(hide yes)
@@
 			)
 		)
-		(property "Footprint" "MyParts:R0402"
+		(property "Footprint" "MyPartsIPC:RESC1005X40N"
 			(at 35.56 146.558 90)
 			(hide yes)
@@
 			)
 		)
-		(property "Footprint" "MyParts:R0402"
+		(property "Footprint" "MyPartsIPC:RESC1005X40N"
 			(at 93.98 176.53 0)
 			(hide yes)
@@
 			)
 		)
-		(property "Footprint" "MyParts:SOT-23-3_L2.9-W1.6-P1.90-LS2.8-BR"
+		(property "Footprint" "MyPartsIPC:SOT95P280X110-3N"
 			(at 43.18 172.72 0)
 			(hide yes)
@@
 			)
 		)
-		(property "Footprint" "MyParts:SC-88A_L2.0-W1.3-P0.65-LS2.1-BL"
+		(property "Footprint" "MyPartsIPC:SOT65P210X110-5N"
 			(at 114.3 180.34 0)
 			(hide yes)
@@
 			)
 		)
-		(property "Footprint" "MyParts:SOT-23-3_L2.9-W1.6-P1.90-LS2.8-BR"
+		(property "Footprint" "MyPartsIPC:SOT95P280X110-3N"
 			(at 43.18 182.88 0)
 			(hide yes)
@@
 			)
 		)
-		(property "Footprint" "MyParts:R0402"
+		(property "Footprint" "MyPartsIPC:RESC1005X40N"
 			(at 41.91 70.358 90)
 			(hide yes)
@@
 			)
 		)
-		(property "Footprint" "MyParts:R0402"
+		(property "Footprint" "MyPartsIPC:RESC1005X40N"
 			(at 41.91 95.758 90)
 			(hide yes)
@@
 			)
 		)
-		(property "Footprint" "MyParts:C0402"
+		(property "Footprint" "MyPartsIPC:CAPC1005X55N"
 			(at 137.16 173.99 0)
 			(hide yes)

Commit message: Updates after latest Tomachie review
Other:
- note added: "Suggest a CM4004008. 4GB RAM, 8GB eMMC program storage."
- note removed: "Suggest a CM4004016. 4GB RAM, 8GB eMMC program storage."
Changed lines of the file:
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@@
 		)
 	)
-	(text "Suggest a CM4004016.\n4GB RAM, 8GB eMMC program storage."
+	(text "Suggest a CM4004008.\n4GB RAM, 8GB eMMC program storage."
 		(exclude_from_sim no)
 		(at 136.906 17.526 0)
