File: kicad/gps.kicad_sch (KiCad schematic)
At the start: 21 parts, among them CN1 SMA-KWE_C7498154, U13 MAX-M10S-00B

Commit message: GPIO connectors defined
Parts:
- added C101: 100nF, MyParts:C0603, symbol MyParts:CC0603KRX7R9BB104
- added D43: TPESD0402G05V, MyParts:D0402-BI, symbol MyParts:TPESD0402G05V
- added J3: SMA-KWE_C7498154, MyParts:SMA-TH_SMA-KWE_C7498154, symbol MyParts:SMA-KWE_C7498154
- added R115: 100Ω, MyParts:R0402, symbol MyParts:0402WGF1000TCE
- added R116: 100kΩ, MyParts:R0603, symbol MyParts:0603WAF1003T5E
- added U18: 74LVC1G17SE-7, MyParts:SC-88A_L2.0-W1.3-P0.65-LS2.1-BL, symbol MyParts:74LVC1G17SE-7
- BT1: MPN (none) -> MS621FE-FL11E; Manufacturer (none) -> Seiko Instruments
- C21: footprint PCM_JLCPCB:C_0603 -> MyParts:C0603; symbol PCM_JLCPCB-Capacitors:0603,10uF,(2) -> MyParts:CL10A106MA8NRNC; Attrition Qty 8 -> (none); Capacitance 10uF -> (none); Category Capacitors,Multilayer Ceramic Capacitors MLCC - SMD/SMT -> (none); Class Basic Component -> (none); LCSC C96446 -> (none); LCSC Part (none) -> C96446; MPN (none) -> CL10A106MA8NRNC; Manufacturer Samsung Electro-Mechanics -> SAMSUNG; Minimum Qty 20 -> (none); Part CL10A106MA8NRNC -> (none); Price 0.021USD -> (none); Process SMT -> (none); Stock 3388297 -> (none); Temperature Coefficient X5R -> (none); Voltage Rated 25V -> (none); Voltage Rating (none) -> 25V
- C22, C23: footprint PCM_JLCPCB:C_0603 -> MyParts:C0603; symbol PCM_JLCPCB-Capacitors:0603,100nF -> MyParts:CC0603KRX7R9BB104; Attrition Qty 10 -> (none); Capacitance 100nF -> (none); Category Capacitors,Multilayer Ceramic Capacitors MLCC - SMD/SMT -> (none); Class Basic Component -> (none); LCSC C14663 -> (none); LCSC Part (none) -> C14663; MPN (none) -> CC0603KRX7R9BB104; Minimum Qty 20 -> (none); Part CC0603KRX7R9BB104 -> (none); Price 0.006USD -> (none); Process SMT -> (none); Stock 70324515 -> (none); Temperature Coefficient X7R -> (none); Voltage Rated 50V -> (none); Voltage Rating (none) -> 50V
- C24: footprint PCM_JLCPCB:C_0603 -> MyParts:C0603; symbol PCM_JLCPCB-Capacitors:0603,47pF -> MyParts:CL10C470JB8NNNC; Attrition Qty 10 -> (none); Capacitance 47pF -> (none); Category Capacitors,Multilayer Ceramic Capacitors MLCC - SMD/SMT -> (none); Class Basic Component -> (none); LCSC C1671 -> (none); LCSC Part (none) -> C1671; MPN (none) -> CL10C470JB8NNNC; Manufacturer Samsung Electro-Mechanics -> SAMSUNG; Minimum Qty 20 -> (none); Part CL10C470JB8NNNC -> (none); Price 0.007USD -> (none); Process SMT -> (none); Stock 828046 -> (none); Temperature Coefficient C0G -> (none); Voltage Rated 50V -> (none); Voltage Rating (none) -> 50V
- C25: footprint PCM_JLCPCB:C_0603 -> MyParts:C0603; symbol PCM_JLCPCB-Capacitors:0603,10nF -> MyParts:0603B103K500NT; Attrition Qty 10 -> (none); Capacitance 10nF -> (none); Category Capacitors,Multilayer Ceramic Capacitors MLCC - SMD/SMT -> (none); Class Basic Component -> (none); LCSC C57112 -> (none); LCSC Part (none) -> C57112; MPN (none) -> 0603B103K500NT; Manufacturer FH(Guangdong Fenghua Advanced Tech) -> FH; Minimum Qty 20 -> (none); Part 0603B103K500NT -> (none); Price 0.005USD -> (none); Process SMT -> (none); Stock 5921160 -> (none); Temperature Coefficient X7R -> (none); Voltage Rated 50V -> (none); Voltage Rating (none) -> 50V
- C26: footprint PCM_JLCPCB:C_0603 -> MyParts:C0603; symbol PCM_JLCPCB-Capacitors:0603,1uF -> MyParts:CL10A105KB8NNNC; Attrition Qty 10 -> (none); Capacitance 1uF -> (none); Category Capacitors,Multilayer Ceramic Capacitors MLCC - SMD/SMT -> (none); Class Basic Component -> (none); LCSC C15849 -> (none); LCSC Part (none) -> C15849; MPN (none) -> CL10A105KB8NNNC; Manufacturer Samsung Electro-Mechanics -> SAMSUNG; Minimum Qty 20 -> (none); Part CL10A105KB8NNNC -> (none); Price 0.008USD -> (none); Process SMT -> (none); Stock 11535980 -> (none); Temperature Coefficient X5R -> (none); Voltage Rated 50V -> (none); Voltage Rating (none) -> 50V
- CN1: Manufacturer LX(连欣科技) -> LX
- D4: Manufacturer Littelfuse(美国力特) -> Littelfuse
- D5: Manufacturer CJ(江苏长电/长晶) -> CJ
- L2: value BLM18AG601SN1D -> 120Ω@100MHz; symbol MyParts:BLM18AG601SN1D -> MyParts:BLM18KG121TN1D; Current Rating (none) -> 3A; DC Resistance (none) -> 30mΩ; LCSC Part C19330 -> C85831; MPN BLM18AG601SN1D -> BLM18KG121TN1D; Manufacturer muRata(村田) -> muRata; Tolerance (none) -> ±25%
- L3: value LQG15HS27NJ02D -> 27nH; Current Rating (none) -> 350mA; DC Resistance (none) -> 460mΩ; Manufacturer muRata(村田) -> muRata; Tolerance (none) -> ±5%
- R18, R23: footprint PCM_JLCPCB:R_0603 -> MyParts:R0603; symbol PCM_JLCPCB-Resistors:0603,1kΩ -> MyParts:0603WAF1001T5E; Attrition Qty 10 -> (none); Category Resistors,Chip Resistor - Surface Mount -> (none); Class Basic Component -> (none); LCSC C21190 -> (none); LCSC Part (none) -> C21190; MPN (none) -> 0603WAF1001T5E; Manufacturer UNI-ROYAL(Uniroyal Elec) -> UNI-ROYAL; Minimum Qty 20 -> (none); Operating Temperature Range -55°C~+155°C -> (none); Overload Voltage (Max) 75V -> (none); Part 0603WAF1001T5E -> (none); Power(Watts) 100mW -> (none); Price 0.004USD -> (none); Process SMT -> (none); Resistance 1kΩ -> (none); Stock 27538425 -> (none); Temperature Coefficient ±100ppm/°C -> (none); Type Thick Film Resistors -> (none); Voltage Rating (none) -> 75V
- R19: footprint PCM_JLCPCB:R_0402 -> MyParts:R0402; symbol PCM_JLCPCB-Resistors:0402,1kΩ -> MyParts:0402WGF1001TCE; Attrition Qty 10 -> (none); Category Resistors,Chip Resistor - Surface Mount -> (none); Class Basic Component -> (none); Field4 ${REFERENCE} -> (none); LCSC C11702 -> (none); LCSC Part (none) -> C11702; MPN (none) -> 0402WGF1001TCE; Manufacturer UNI-ROYAL(Uniroyal Elec) -> UNI-ROYAL; Minimum Qty 20 -> (none); Operating Temperature Range -55°C~+155°C -> (none); Overload Voltage (Max) 50V -> (none); Part 0402WGF1001TCE -> (none); Power(Watts) 62.5mW -> (none); Price 0.004USD -> (none); Process SMT -> (none); Resistance 1kΩ -> (none); Stock 13226393 -> (none); Temperature Coefficient ±100ppm/°C -> (none); Type Thick Film Resistors -> (none); Voltage Rating (none) -> 50V
- R20, R21: footprint PCM_JLCPCB:R_0402 -> MyParts:R0402; symbol PCM_JLCPCB-Resistors:0402,100Ω -> MyParts:0402WGF1000TCE; Attrition Qty 10 -> (none); Category Resistors,Chip Resistor - Surface Mount -> (none); Class Basic Component -> (none); Field4 ${REFERENCE} -> (none); LCSC C25076 -> (none); LCSC Part (none) -> C25076; MPN (none) -> 0402WGF1000TCE; Manufacturer UNI-ROYAL(Uniroyal Elec) -> UNI-ROYAL; Minimum Qty 20 -> (none); Operating Temperature Range -55°C~+155°C -> (none); Overload Voltage (Max) 50V -> (none); Part 0402WGF1000TCE -> (none); Power(Watts) 62.5mW -> (none); Price 0.004USD -> (none); Process SMT -> (none); Resistance 100Ω -> (none); Stock 5907585 -> (none); Temperature Coefficient ±200ppm/°C -> (none); Type Thick Film Resistors -> (none); Voltage Rating (none) -> 50V
- R22: Manufacturer UNI-ROYAL(厚声) -> UNI-ROYAL; Tolerance (none) -> ±1%; Voltage Rating (none) -> 200V
- TP1: Manufacturer 荣和 -> ronghe
- U13: Manufacturer U-BLOX(优北罗) -> U-BLOX
Connections:
- net GND: now also C101.2, D43.1 (K), J3.1, J3.2, J3.3, J3.4, R116.2, U18.3 (GND)
- net VCC: now also C101.1, U18.5 (VCC)
- net EXT_1PPS: now reaches U13.5 (EXTINT)
- net EXT_1PPS: now also U18.4 (Y)
- new net: D43.2 (A), J3.5, R115.1
- new net: R115.2, R116.1, U18.2 (A)
- no-connect marks 7 -> 6
Other:
- note added: "1PPS from FEI FE-5680A rubidium clock, 3-5V logic pulse. U18 Schmitt buffer (5V-tolerant input, VT+ <= 2.0V at 3V) shifts it to the 3.3V V_IO level; EXTINT abs max is V_IO+0.3V (3.6V). R116 holds the input low when nothing is connected. Edges on EXTINT are timestamped in UBX-TIM-TM2 (time mark)."
- note added: "D4 (0.25pF) is the antenna ESD clamp - keep it right at CN1. Not lightning protection: an outdoor run still needs a coaxial arrestor at the bulkhead."
- note added: "L2 supply-bead DCR must be < 0.2 Ω (u-blox MAX-M10S IM §3.1.1: series resistance on VCC causes ripple under dynamic current). BLM18KG121TN1D: 0.030 Ω max (0.040 Ω after test). Do not substitute a higher-DCR bead."
- note removed: "AI Note: "Do not add series resistance greater than 0.2 Ω on the supply line to avoid voltage ripple due to the dynamic current conditions." Your L13 is a BLM18AG601SN1D, and ferrite beads have real DC resistance - that part is likely somewhere around 0.3-0.5 Ω, which would exceed u-blox's limit. Worth checking against the Murata datasheet. If it does exceed it, the fix is a lower-DCR bead rather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"
- note removed: "D43 (0.25pF) is the antenna ESD clamp - keep it right at CN7. Not lightning protection: an outdoor run still needs a coaxial arrestor at the bulkhead."
- moved on the sheet: BT1, C21, C22, C23, C24, C25, C26, CN1, D4, D5, L3, LED2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

Commit message: schematic cleanup
Parts:
- added TP15, TP16, TP17, TP25: TestPoint_Small, TestPoint:TestPoint_Pad_D1.5mm, symbol Connector:TestPoint_Small
Connections:
- net GND: now also TP25.1
- net VCC: now also TP15.1
- net VCC_RF: now also TP17.1
- net Net-(LED2-A): now reaches LED2.1 (A), R18.2
- net Net-(LED2-A): now also TP16.1

Commit message: Still refining
Parts:
- BT1: Pkg Type (none) -> SMD Coin cell
- C101, C21, C22, C23, C24, C25, C26, R116, R18, R23: Pkg Type (none) -> SMD 0603
- CN1, J3: Pkg Type (none) -> THT SMA jack
- D4, D43, L3, R115, R19, R20, R21: Pkg Type (none) -> SMD 0402
- D5: Pkg Type (none) -> SMD SOD-323
- FB2: renamed from L2; Pkg Type (none) -> SMD 0603
- LED2: Pkg Type (none) -> SMD 0805
- R22: Pkg Type (none) -> SMD 1206
- TP1: Pkg Type (none) -> SMD Test point loop
- TP15, TP16, TP17, TP25: Pkg Type (none) -> SMD Test pad D1.5
- U13: Pkg Type (none) -> SMD LCC-18 module
- U18: Pkg Type (none) -> SMD SOT-353 (SC-88A)

Commit message: Mods
Parts:
- removed R18: 1kΩ, MyParts:R0603, symbol MyParts:0603WAF1001T5E
- added C114: 100nF, MyParts:C0603, symbol MyParts:CC0603KRX7R9BB104
- added C115: 10uF, MyParts:C0805, symbol MyParts:CL21B106KPQNNNE
- added D51: BZT52C4V7, MyParts:SOD-123_L2.7-W1.6-LS3.7-RD, symbol MyParts:BZT52C4V7
- added R18: 220Ω, MyParts:R0402, symbol MyParts:0402WGF2200TCE
- added TP27, TP32: TestPoint_Small, TestPoint:TestPoint_Pad_D1.5mm, symbol Connector:TestPoint_Small
- added U22: 74LVC1G17SE-7, MyParts:SC-88A_L2.0-W1.3-P0.65-LS2.1-BL, symbol MyParts:74LVC1G17SE-7
- BT1: value MS621FE-FL11E -> ML414H-IV01E; footprint MyParts:BAT_MS621FE-FL11E -> MyParts:ML414H-IV01E; symbol MyParts:MS621FE-FL11E -> MyParts:ML414H-IV01E; MAXIMUM_PACKAGE_HEIGHT 2.8mm -> 1.4mm; MPN MS621FE-FL11E -> ML414H-IV01E; Pkg Type SMD Coin cell -> SMD Coin cell 4.8mm; Sourcing (none) -> Digi-Key or Mouser, consigned to JLCPCB (no LCSC stock); now fitted
- D4: value PESD0402-140 -> SESD0402X1UN-0020-090; footprint MyParts:D0402-BI -> MyParts:DIO-SMD_2P-L1.0-W0.6-P0.65-RD; symbol MyParts:PESD0402-140 -> MyParts:SESD0402X1UN-0020-090; LCSC Part C10662 -> C1973340; MPN PESD0402-140 -> SESD0402X1UN-0020-090; Pkg Type SMD 0402 -> SMD DFN1006-2 (0402)
- D43: value TPESD0402G05V -> TPESD0402G12V; symbol MyParts:TPESD0402G05V -> MyParts:TPESD0402G12V; LCSC Part C558615 -> C558617; MPN TPESD0402G05V -> TPESD0402G12V
- R22: value 10Ω -> 33Ω; footprint MyParts:R1206 -> MyParts:R2512; symbol MyParts:1206W4F100JT5E -> MyParts:25121WF330JT4E; LCSC Part C17903 -> C53728; MPN 1206W4F100JT5E -> 25121WF330JT4E; Pkg Type SMD 1206 -> SMD 2512
- R23: value 1kΩ -> 10kΩ; symbol MyParts:0603WAF1001T5E -> MyParts:0603WAF1002T5E; LCSC Part C21190 -> C25804; MPN 0603WAF1001T5E -> 0603WAF1002T5E
Connections:
- net GND: now also D4.2 (A), C114.2, C115.1, D51.2 (A), TP32.1, U22.3 (GND); no longer D4.1
- net Net-(LED2-A): now also R18.1
- net RF_IN: now also D4.1 (C); no longer D4.2
- net TIMEPULSE: now also U22.2 (A); no longer R19.2
- net VCC: now also C114.1, U22.5 (VCC)
- net VCC_RF: no longer R22.2
- net at C24.1, C25.1, L3.2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: now also C115.2, D51.1 (K)
- net at U13.18 (SAFEBOOT_N): now also TP27.1
- new net 5V: R22.2
- new net PPS_BUF: R18.2, R19.2, U22.4 (Y)
Other:
- note added: "1PPS from FEI FE-5680A rubidium clock, 3-5V logic pulse. U18 Schmitt buffer (5V-tolerant input, VT+ <= 2.0V at 3V) shifts it to the 3.3V V_IO level; EXTINT abs max is V_IO+0.3V (3.6V). R116 holds the input low when nothing is connected. Edges on EXTINT are timestamped in UBX-TIM-TM2 (time mark). J3: bulkhead SMA bonded to the enclosure wall."
- note added: "Antenna LNA 40 dB, ~35 dB at RF_IN: above the 30 dB low-gain limit. At startup set CFG-HW-RF_LNA_MODE = bypass (10-40 dB)."
- note added: "Antenna bias from 5V, not VCC_RF: the Waveshare L1/L2/L5 antenna needs 3.0-18 V at <=45 mA over 5 m RG174; VCC_RF (VCC-0.1 V, 50 mA max) cannot hold 3.0 V through any short-circuit resistor. R22 33R 1W limits a short to ~155 mA (L3 350 mA). C115 filters buck ripple. D51 4.7 V keeps RF_IN < 5.5 V DC abs max (antenna unplugged). Worst-case antenna voltage ~3.3 V at 45 mA."
- note added: "BT1 ML414H-IV01E is reflowable: JLC places it. No LCSC stock: buy from Digi-Key/Mouser and consign to JLCPCB. 1.0 mAh: ~1.5 days at 28 uA. D5+R23 10k charge (SII: R>=3k). Cell: -20 to +60 C."
- note added: "Bring-up: scope V_IO (TP15) at power-on and on a GLOBAL_EN cycle. 0->3.3 V rise must be 82.5 us to 115.5 ms (MAX-M10S DS p.11). If < ~100 us, add bulk C on VCC."
- note added: "D4: Si TVS, 0.25 pF, 9.2 V clamp, K to RF_IN. Install CN1 on a bulkhead SMA bonded to the enclosure, with a DC-pass coax arrestor."
- note added: "TIMEPULSE shares a pin with SAFEBOOT_N (1k inside U13); low at startup = safeboot, no NMEA (MAX-M10S IM 2.3.3.3: no load on it). R18/LED2 and R19 into GPIO16 (default pull-down) could hold it mid-rail. U22 leaves only input leakage on TIMEPULSE and drives the LED and GPIO16. VCC is from 3V3_CM4: no back-power path."
- note removed: "1PPS from FEI FE-5680A rubidium clock, 3-5V logic pulse. U18 Schmitt buffer (5V-tolerant input, VT+ <= 2.0V at 3V) shifts it to the 3.3V V_IO level; EXTINT abs max is V_IO+0.3V (3.6V). R116 holds the input low when nothing is connected. Edges on EXTINT are timestamped in UBX-TIM-TM2 (time mark)."
- note removed: "D4 (0.25pF) is the antenna ESD clamp - keep it right at CN1. Not lightning protection: an outdoor run still needs a coaxial arrestor at the bulkhead."
- moved on the sheet: C24, C25, D4, L3, LED2, R22

Commit message: Ready to start layout
Parts:
- renumbered C101 to C31, C26 to C32, C21 to C33, C22 to C34, C23 to C35, C24 to C36, C25 to C37, C115 to C38, C114 to C39, D5 to D12, D43 to D13, D51 to D14, D4 to D15, J3 to J7, L3 to L1, LED2 to LED4, R20 to R33, R19 to R34, R21 to R35, R23 to R36, R115 to R37, R116 to R38, R18 to R39, R22 to R40, TP16 to TP17, TP27 to TP18, TP25 to TP19, TP1 to TP20, TP15 to TP21, TP32 to TP22, TP17 to TP23, U13 to U12, U18 to U13, U22 to U14
Other:
- note added: "1PPS from FEI FE-5680A rubidium clock, 3-5V logic pulse. U13 Schmitt buffer (5V-tolerant input, VT+ <= 2.0V at 3V) shifts it to the 3.3V V_IO level; EXTINT abs max is V_IO+0.3V (3.6V). R38 holds the input low when nothing is connected. Edges on EXTINT are timestamped in UBX-TIM-TM2 (time mark). J7: bulkhead SMA bonded to the enclosure wall."
- note added: "Antenna bias from 5V, not VCC_RF: the Waveshare L1/L2/L5 antenna needs 3.0-18 V at <=45 mA over 5 m RG174; VCC_RF (VCC-0.1 V, 50 mA max) cannot hold 3.0 V through any short-circuit resistor. R40 33R 1W limits a short to ~155 mA (L1 350 mA). C38 filters buck ripple. D14 4.7 V keeps RF_IN < 5.5 V DC abs max (antenna unplugged). Worst-case antenna voltage ~3.3 V at 45 mA."
- note added: "BT1 ML414H-IV01E is reflowable: JLC places it. No LCSC stock: buy from Digi-Key/Mouser and consign to JLCPCB. 1.0 mAh: ~1.5 days at 28 uA. D12+R36 10k charge (SII: R>=3k). Cell: -20 to +60 C."
- note added: "Bring-up: scope V_IO (TP21) at power-on and on a GLOBAL_EN cycle. 0->3.3 V rise must be 82.5 us to 115.5 ms (MAX-M10S DS p.11). If < ~100 us, add bulk C on VCC."
- note added: "D15: Si TVS, 0.25 pF, 9.2 V clamp, K to RF_IN. Install CN1 on a bulkhead SMA bonded to the enclosure, with a DC-pass coax arrestor."
- note added: "TIMEPULSE shares a pin with SAFEBOOT_N (1k inside U12); low at startup = safeboot, no NMEA (MAX-M10S IM 2.3.3.3: no load on it). R39/LED4 and R34 into GPIO16 (default pull-down) could hold it mid-rail. U14 leaves only input leakage on TIMEPULSE and drives the LED and GPIO16. VCC is from 3V3_CM4: no back-power path."
- note removed: "1PPS from FEI FE-5680A rubidium clock, 3-5V logic pulse. U18 Schmitt buffer (5V-tolerant input, VT+ <= 2.0V at 3V) shifts it to the 3.3V V_IO level; EXTINT abs max is V_IO+0.3V (3.6V). R116 holds the input low when nothing is connected. Edges on EXTINT are timestamped in UBX-TIM-TM2 (time mark). J3: bulkhead SMA bonded to the enclosure wall."
- note removed: "Antenna bias from 5V, not VCC_RF: the Waveshare L1/L2/L5 antenna needs 3.0-18 V at <=45 mA over 5 m RG174; VCC_RF (VCC-0.1 V, 50 mA max) cannot hold 3.0 V through any short-circuit resistor. R22 33R 1W limits a short to ~155 mA (L3 350 mA). C115 filters buck ripple. D51 4.7 V keeps RF_IN < 5.5 V DC abs max (antenna unplugged). Worst-case antenna voltage ~3.3 V at 45 mA."
- note removed: "BT1 ML414H-IV01E is reflowable: JLC places it. No LCSC stock: buy from Digi-Key/Mouser and consign to JLCPCB. 1.0 mAh: ~1.5 days at 28 uA. D5+R23 10k charge (SII: R>=3k). Cell: -20 to +60 C."
- note removed: "Bring-up: scope V_IO (TP15) at power-on and on a GLOBAL_EN cycle. 0->3.3 V rise must be 82.5 us to 115.5 ms (MAX-M10S DS p.11). If < ~100 us, add bulk C on VCC."
- note removed: "D4: Si TVS, 0.25 pF, 9.2 V clamp, K to RF_IN. Install CN1 on a bulkhead SMA bonded to the enclosure, with a DC-pass coax arrestor."
- note removed: "TIMEPULSE shares a pin with SAFEBOOT_N (1k inside U13); low at startup = safeboot, no NMEA (MAX-M10S IM 2.3.3.3: no load on it). R18/LED2 and R19 into GPIO16 (default pull-down) could hold it mid-rail. U22 leaves only input leakage on TIMEPULSE and drives the LED and GPIO16. VCC is from 3V3_CM4: no back-power path."

Commit message: IPC footprint renaming, battery sim added
Parts:
- C31, C32, C33, C34, C35, C36, C37, C39: footprint MyParts:C0603 -> MyPartsIPC:CAPC1608X95N
- C38: footprint MyParts:C0805 -> MyPartsIPC:CAPC2012X145N
- D12: footprint MyParts:SOD-323_L1.8-W1.3-LS2.5-RD -> MyPartsIPC:SOD2513X110N
- D13: footprint MyParts:D0402-BI -> MyPartsIPC:DIOC1005X55N
- D14: footprint MyParts:SOD-123_L2.7-W1.6-LS3.7-RD -> MyPartsIPC:SOD3716X135N
- D15: footprint MyParts:DIO-SMD_2P-L1.0-W0.6-P0.65-RD -> MyPartsIPC:DIOC1006X40N
- FB2: footprint MyParts:L0603 -> MyPartsIPC:INDC1608X95N
- L1: footprint MyParts:L0402-RD -> MyPartsIPC:INDC1005X55N
- LED4: footprint MyParts:LED0805-R-RD -> MyPartsIPC:LEDC2012X110N
- R33, R34, R35, R37, R39: footprint MyParts:R0402 -> MyPartsIPC:RESC1005X40N
- R36, R38: footprint MyParts:R0603 -> MyPartsIPC:RESC1608X55N
- R40: footprint MyParts:R2512 -> MyPartsIPC:RESC6332X70N
- TP22: now left out of the parts list
- U13, U14: footprint MyParts:SC-88A_L2.0-W1.3-P0.65-LS2.1-BL -> MyPartsIPC:SOT65P210X110-5N
Changed lines of the file:
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@@
 			)
 		)
-		(property "Footprint" "MyParts:R0402"
+		(property "Footprint" "MyPartsIPC:RESC1005X40N"
 			(at 229.87 74.93 0)
 			(hide yes)
@@
 			)
 		)
-		(property "Footprint" "MyParts:LED0805-R-RD"
+		(property "Footprint" "MyPartsIPC:LEDC2012X110N"
 			(at 71.12 127 0)
 			(hide yes)
@@
 			)
 		)
-		(property "Footprint" "MyParts:C0603"
+		(property "Footprint" "MyPartsIPC:CAPC1608X95N"
 			(at 74.422 87.63 90)
 			(hide yes)
@@
 			)
 		)
-		(property "Footprint" "MyParts:L0402-RD"
+		(property "Footprint" "MyPartsIPC:INDC1005X55N"
 			(at 99.06 115.57 0)
 			(hide yes)
@@
 			)
 		)
-		(property "Footprint" "MyParts:SC-88A_L2.0-W1.3-P0.65-LS2.1-BL"
+		(property "Footprint" "MyPartsIPC:SOT65P210X110-5N"
 			(at 241.3 139.7 0)
 			(hide yes)
@@
 			)
 		)
-		(property "Footprint" "MyParts:R2512"
+		(property "Footprint" "MyPartsIPC:RESC6332X70N"
 			(at 113.03 129.54 0)
 			(hide yes)
@@
 			)
 		)
-		(property "Footprint" "MyParts:C0603"
+		(property "Footprint" "MyPartsIPC:CAPC1608X95N"
 			(at 66.802 87.63 90)
 			(hide yes)
@@
 			)
 		)
-		(property "Footprint" "MyParts:DIO-SMD_2P-L1.0-W0.6-P0.65-RD"
+		(property "Footprint" "MyPartsIPC:DIOC1006X40N"
 			(at 153.67 127 0)
 			(hide yes)
@@
 			)
 		)
-		(property "Footprint" "MyParts:R0402"
+		(property "Footprint" "MyPartsIPC:RESC1005X40N"
 			(at 82.55 69.088 90)
 			(hide yes)
@@
 			)
 		)
-		(property "Footprint" "MyParts:R0603"
+		(property "Footprint" "MyPartsIPC:RESC1608X55N"
 			(at 236.22 78.74 0)
 			(hide yes)
@@
 			)
 		)
-		(property "Footprint" "MyParts:R0402"
+		(property "Footprint" "MyPartsIPC:RESC1005X40N"
 			(at 59.69 74.168 90)
 			(hide yes)
@@
 			)
 		)
-		(property "Footprint" "MyParts:SOD-123_L2.7-W1.6-LS3.7-RD"
+		(property "Footprint" "MyPartsIPC:SOD3716X135N"
 			(at 125.73 129.54 0)
 			(hide yes)
@@
 			)
 		)
-		(property "Footprint" "MyParts:C0603"
+		(property "Footprint" "MyPartsIPC:CAPC1608X95N"
 			(at 241.3 64.77 0)
 			(hide yes)
@@
 			)
 		)
-		(property "Footprint" "MyParts:L0603"
+		(property "Footprint" "MyPartsIPC:INDC1608X95N"
 			(at 59.69 90.17 0)
 			(hide yes)
@@
 			)
 		)
-		(property "Footprint" "MyParts:R0603"
+		(property "Footprint" "MyPartsIPC:RESC1608X55N"
 			(at 154.432 69.85 90)
 			(hide yes)
@@
 		(body_style 1)
 		(exclude_from_sim no)
-		(in_bom yes)
+		(in_bom no)
 		(on_board yes)
 		(in_pos_files yes)
@@
 			)
 		)
-		(property "Footprint" "MyParts:C0603"
+		(property "Footprint" "MyPartsIPC:CAPC1608X95N"
 			(at 167.132 83.82 90)
 			(hide yes)
@@
 			)
 		)
-		(property "Footprint" "MyParts:C0603"
+		(property "Footprint" "MyPartsIPC:CAPC1608X95N"
 			(at 82.042 87.63 90)
 			(hide yes)
@@
 			)
 		)
-		(property "Footprint" "MyParts:SOD-323_L1.8-W1.3-LS2.5-RD"
+		(property "Footprint" "MyPartsIPC:SOD2513X110N"
 			(at 163.83 59.69 0)
 			(hide yes)
@@
 			)
 		)
-		(property "Footprint" "MyParts:R0402"
+		(property "Footprint" "MyPartsIPC:RESC1005X40N"
 			(at 71.12 115.57 0)
 			(hide yes)
@@
 			)
 		)
-		(property "Footprint" "MyParts:C0603"
+		(property "Footprint" "MyPartsIPC:CAPC1608X95N"
 			(at 101.092 128.27 90)
 			(hide yes)
@@
 			)
 		)
-		(property "Footprint" "MyParts:C0603"
+		(property "Footprint" "MyPartsIPC:CAPC1608X95N"
 			(at 269.24 132.08 0)
 			(hide yes)
@@
 			)
 		)
-		(property "Footprint" "MyParts:SC-88A_L2.0-W1.3-P0.65-LS2.1-BL"
+		(property "Footprint" "MyPartsIPC:SOT65P210X110-5N"
 			(at 248.92 74.93 0)
 			(hide yes)
@@
 			)
 		)
-		(property "Footprint" "MyParts:C0603"
+		(property "Footprint" "MyPartsIPC:CAPC1608X95N"
 			(at 108.712 128.27 90)
 			(hide yes)
@@
 			)
 		)
-		(property "Footprint" "MyParts:C0805"
+		(property "Footprint" "MyPartsIPC:CAPC2012X145N"
 			(at 125.73 128.27 0)
 			(hide yes)
@@
 			)
 		)
-		(property "Footprint" "MyParts:R0402"
+		(property "Footprint" "MyPartsIPC:RESC1005X40N"
 			(at 82.55 71.628 90)
 			(hide yes)
@@
 			)
 		)
-		(property "Footprint" "MyParts:D0402-BI"
+		(property "Footprint" "MyPartsIPC:DIOC1005X55N"
 			(at 223.52 80.01 0)
 			(hide yes)
