File: kicad/gps.kicad_sch (KiCad schematic)
At the start: 39 parts, among them CN1 SMA-KWE_C7498154, J7 SMA-KWE_C7498154, U12 MAX-M10S-00B, U13 74LVC1G17SE-7, U14 74LVC1G17SE-7

Commit message: PCB: RF_IN parts on the line, CN1 -> J2, test point fixes, J15/J16 on A1
- D15 and L1 moved beside the vertical RF_IN run; the 3.8 mm branch is
  gone, bias track re-routed to C36, labels re-placed (TP23 label moved).
- CN1 (GPS antenna SMA) renamed J2 in the schematic, GPS sheet note and
  PCB, matching the J prefix used for every other connector.
- TP22 removed from the schematic and PCB (redundant GND point beside
  TP19); TP19 moved next to D15 with a ground track.
- TP9 (U4 ILIM) and TP10 (GND) moved to the bottom side under U4; the
  ILIM net drops from 30 mm with two vias to 3.1 mm with one.
- J15/J16 RoboClaw sockets moved onto A1's power and signal hole rows
  (they were left behind when A1 was rotated).
- 3D model offsets adjusted on several footprints.
- parts submodule updated to b785c82.
Parts:
- removed TP22: TestPoint_Small, TestPoint:TestPoint_Pad_D1.5mm, symbol Connector:TestPoint_Small
- renumbered CN1 to J2
Other:
- note added: "D15: Si TVS, 0.25 pF, 9.2 V clamp, K to RF_IN. Install J2 on a bulkhead SMA bonded to the enclosure, with a DC-pass coax arrestor."
- note removed: "D15: Si TVS, 0.25 pF, 9.2 V clamp, K to RF_IN. Install CN1 on a bulkhead SMA bonded to the enclosure, with a DC-pass coax arrestor."
Changed lines of the file:
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@@
 		)
 	)
-	(text "D15: Si TVS, 0.25 pF, 9.2 V clamp, K to RF_IN.\nInstall CN1 on a bulkhead SMA bonded to the\nenclosure, with a DC-pass coax arrestor."
+	(text "D15: Si TVS, 0.25 pF, 9.2 V clamp, K to RF_IN.\nInstall J2 on a bulkhead SMA bonded to the\nenclosure, with a DC-pass coax arrestor."
 		(exclude_from_sim no)
 		(at 156.21 136.398 0)
@@
 	)
 	(junction
-		(at 72.39 93.98)
-		(diameter 0)
-		(color 0 0 0 0)
-	)
-	(junction
 		(at 156.21 74.93)
 		(diameter 0)
@@
 	(wire
 		(pts
-			(xy 72.39 95.25) (xy 72.39 93.98)
-		)
-		(stroke
-			(width 0)
-			(type default)
-		)
-	)
-	(wire
-		(pts
 			(xy 167.64 125.73) (xy 165.1 125.73)
 		)
@@
 		(in_pos_files yes)
 		(dnp no)
-		(property "Reference" "CN1"
+		(property "Reference" "J2"
 			(at 181.61 115.5699 0)
 			(show_name no)
@@
 			(project "cm4-robo-controller"
 				(path "/c1285fbe-5f56-49a8-9041-410713cbe619/59179e28-57e7-4020-bfeb-9df0a9a28165"
-					(reference "CN1")
+					(reference "J2")
 					(unit 1)
 				)
@@
 					(unit 1)
 				)
-			)
-		)
-	)
-	(symbol
-		(lib_id "Connector:TestPoint_Small")
-		(at 72.39 95.25 0)
-		(unit 1)
-		(body_style 1)
-		(exclude_from_sim no)
-		(in_bom no)
-		(on_board yes)
-		(in_pos_files yes)
-		(dnp no)
-		(property "Reference" "TP22"
-			(at 71.374 97.028 0)
-			(show_name no)
-			(do_not_autoplace no)
-			(effects
-				(font
-					(size 1.27 1.27)
-				)
-				(justify right)
-			)
-		)
-		(property "Value" "TestPoint_Small"
-			(at 72.39 96.012 0)
-			(hide yes)
-			(show_name no)
-			(do_not_autoplace no)
-			(effects
-				(font
-					(size 1.27 1.27)
-				)
-			)
-		)
-		(property "Footprint" "TestPoint:TestPoint_Pad_D1.5mm"
-			(at 72.39 96.012 0)
-			(hide yes)
-			(show_name no)
-			(do_not_autoplace no)
-			(effects
-				(font
-					(size 1.27 1.27)
-				)
-			)
-		)
-		(property "Datasheet" ""
-			(at 72.39 95.25 0)
-			(show_name no)
-			(do_not_autoplace no)
-			(effects
-				(font
-					(size 1.27 1.27)
-				)
-			)
-		)
-		(property "Description" "Test Point"
-			(at 72.39 96.012 0)
-			(hide yes)
-			(show_name no)
-			(do_not_autoplace no)
-			(effects
-				(font
-					(size 1.27 1.27)
-				)
-			)
-		)
-		(pin "1"
-		)
-		(instances
-			(project "cm4-robo-controller"
-				(path "/c1285fbe-5f56-49a8-9041-410713cbe619/59179e28-57e7-4020-bfeb-9df0a9a28165"
-					(reference "TP22")
-					(unit 1)
-				)
