File: kicad/power.kicad_sch (KiCad schematic)
At the start: 29 parts, among them Q10 NCE6008AS, Q11 BSS138, Q9 DMP6023LE-13, SW3 SS-12F49-G050, U17 MX26631DL

Commit message: GPIO connectors defined
Parts:
- C100: Manufacturer SAMSUNG(三星) -> SAMSUNG; Tolerance (none) -> ±10%; Voltage Rating (none) -> 25V
- C95: Manufacturer JIERR(捷而瑞) -> JIERR; Tolerance (none) -> ±20%
- C96, C97, C98: Manufacturer SAMSUNG(三星) -> SAMSUNG; Tolerance (none) -> ±10%; Voltage Rating (none) -> 16V
- C99: Manufacturer CCTC(三环) -> CCTC; Tolerance (none) -> ±10%; Voltage Rating 25V -> 50V
- D41: symbol PCM_JLCPCB-Diodes:TVS-Uni,SMAJ20A -> MyParts:SMAJ20A; Attrition Qty 2 -> (none); Breakdown Voltage 24.5V -> (none); Category Circuit Protection,ESD And Surge Protection (TVS/ESD) -> (none); Clamping Voltage 45.4V -> (none); Class Preferred Component -> (none); LCSC C41376408 -> (none); LCSC Part (none) -> C41376408; MPN (none) -> SMAJ20A; Maximum Clamping Voltage 32.4V -> (none); Minimum Qty 5 -> (none); Number of Channels Single channel -> (none); Number of Lines Single channel -> (none); Operating Temperature -55°C~+155°C -> (none); Part SMAJ20A -> (none); Peak Pulse Current (Ipp) 8.8A -> (none); Peak Pulse Power Dissipation (Ppp) 400W -> (none); Polarity Unidirectional -> (none); Price 0.037USD -> (none); Process SMT -> (none); Reverse Leakage Current (Ir) 1uA -> (none); Reverse Stand-Off Voltage (Vrwm) 20V -> (none); Stock 8843 -> (none); Type TVS -> (none); Voltage - Breakdown 31.1V -> (none); polarity Unidirectional -> (none)
- D42: symbol PCM_JLCPCB-Diodes:TVS-Bi,SMBJ18CA -> MyParts:SMBJ18CA; Attrition Qty 2 -> (none); Category TVS/Fuse/Board Level Protection,Electrostatic And Surge Pro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 -> (none); Class Preferred Component -> (none); LCSC C19077574 -> (none); LCSC Part C19077585 -> C19077574; MPN SMBJ30CA -> SMBJ18CA; Minimum Qty 5 -> (none); Part SMBJ18CA -> (none); Price 0.048USD -> (none); Process SMT -> (none); Stock 46569 -> (none)
- L1: Current Rating (none) -> 6A; DC Resistance (none) -> 9mΩ; Manufacturer muRata(村田) -> muRata; Tolerance (none) -> ±25%
- Q10: Manufacturer NCE(无锡新洁能) -> NCE
- Q11: symbol PCM_JLCPCB-Transistors:NMOS,BSS138 -> MyParts:BSS138; Attrition Qty 5 -> (none); Category Triode/MOS Tube/Transistor,MOSFETs -> (none); Class Preferred Component -> (none); Continuous Drain Current (Id) 340mA -> (none); Drain Source On Resistance (RDS(on)@Vgs,Id) 2.5Ω@10V,0.34A -> (none); Drain Source Voltage (Vdss) null -> (none); Gate Threshold Voltage (Vgs(th)@Id) 1.6V@250uA -> (none); Input Capacitance (Ciss@Vds) 17.5pF@25V -> (none); LCSC C7420339 -> (none); Minimum Qty 10 -> (none); Operating Temperature -55°C~+150°C -> (none); Part BSS138 -> (none); Power Dissipation (Pd) 350mW -> (none); Price 0.021USD -> (none); Process SMT -> (none); Reverse Transfer Capacitance (Crss@Vds) 6.5pF@25V -> (none); Stock 257620 -> (none); Total Gate Charge (Qg@Vgs) 1.7nC@10V -> (none); Type null -> (none)
- Q9: MPN (none) -> DMP6023LE-13
- R101: footprint PCM_JLCPCB:R_0603 -> MyParts:R0603; symbol PCM_JLCPCB-Resistors:0603,100kΩ -> MyParts:0603WAF1003T5E; Attrition Qty 10 -> (none); Category Resistors,Chip Resistor - Surface Mount -> (none); Class Basic Component -> (none); LCSC C25803 -> (none); LCSC Part (none) -> C25803; MPN (none) -> 0603WAF1003T5E; Manufacturer UNI-ROYAL(Uniroyal Elec) -> UNI-ROYAL; Minimum Qty 20 -> (none); Operating Temperature Range -55°C~+155°C -> (none); Overload Voltage (Max) 75V -> (none); Part 0603WAF1003T5E -> (none); Power(Watts) 100mW -> (none); Price 0.004USD -> (none); Process SMT -> (none); Resistance 100kΩ -> (none); Stock 7820113 -> (none); Temperature Coefficient ±100ppm/°C -> (none); Type Thick Film Resistors -> (none); Voltage Rating (none) -> 75V
- R103: Manufacturer UNI-ROYAL(厚声) -> UNI-ROYAL; Tolerance (none) -> ±1%; Voltage Rating (none) -> 75V
- R104: footprint PCM_JLCPCB:R_0603 -> MyParts:R0603; symbol PCM_JLCPCB-Resistors:0603,13kΩ -> MyParts:0603WAF1302T5E; Attrition Qty 10 -> (none); Category Resistors,Chip Resistor - Surface Mount -> (none); Class Basic Component -> (none); LCSC C22797 -> (none); LCSC Part (none) -> C22797; MPN 0603WAF5102T5E -> 0603WAF1302T5E; Manufacturer UNI-ROYAL(Uniroyal Elec) -> UNI-ROYAL; Minimum Qty 20 -> (none); Operating Temperature Range -55°C~+155°C -> (none); Overload Voltage (Max) 75V -> (none); Part 0603WAF1302T5E -> (none); Power(Watts) 100mW -> (none); Price 0.004USD -> (none); Process SMT -> (none); Resistance 13kΩ -> (none); Stock 264187 -> (none); Temperature Coefficient ±100ppm/°C -> (none); Type Thick Film Resistors -> (none); Voltage Rating (none) -> 75V
- R105: footprint PCM_JLCPCB:R_0603 -> MyParts:R0603; symbol PCM_JLCPCB-Resistors:0603,330kΩ -> MyParts:0603WAF3303T5E; Attrition Qty 10 -> (none); Category Resistors,Chip Resistor - Surface Mount -> (none); Class Basic Component -> (none); LCSC C23137 -> (none); LCSC Part (none) -> C23137; MPN (none) -> 0603WAF3303T5E; Manufacturer UNI-ROYAL(Uniroyal Elec) -> UNI-ROYAL; Minimum Qty 20 -> (none); Operating Temperature Range -55°C~+155°C -> (none); Overload Voltage (Max) 75V -> (none); Part 0603WAF3303T5E -> (none); Power(Watts) 100mW -> (none); Price 0.004USD -> (none); Process SMT -> (none); Resistance 330kΩ -> (none); Stock 575096 -> (none); Temperature Coefficient ±100ppm/°C -> (none); Type Thick Film Resistors -> (none); Voltage Rating (none) -> 75V
- R106: footprint PCM_JLCPCB:R_0603 -> MyParts:R0603; symbol PCM_JLCPCB-Resistors:0603,56kΩ -> MyParts:0603WAF5602T5E; Attrition Qty 10 -> (none); Category Resistors,Chip Resistor - Surface Mount -> (none); Class Basic Component -> (none); LCSC C23206 -> (none); LCSC Part (none) -> C23206; MPN (none) -> 0603WAF5602T5E; Manufacturer UNI-ROYAL(Uniroyal Elec) -> UNI-ROYAL; Minimum Qty 20 -> (none); Operating Temperature Range -55°C~+155°C -> (none); Overload Voltage (Max) 75V -> (none); Part 0603WAF5602T5E -> (none); Power(Watts) 100mW -> (none); Price 0.004USD -> (none); Process SMT -> (none); Resistance 56kΩ -> (none); Stock 358487 -> (none); Temperature Coefficient ±100ppm/°C -> (none); Type Thick Film Resistors -> (none); Voltage Rating (none) -> 75V
- R107: footprint PCM_JLCPCB:R_0603 -> MyParts:R0603; symbol PCM_JLCPCB-Resistors:0603,82kΩ -> MyParts:0603WAF8202T5E; Attrition Qty 10 -> (none); Category Resistors,Chip Resistor - Surface Mount -> (none); Class Basic Component -> (none); LCSC C23254 -> (none); LCSC Part (none) -> C23254; MPN (none) -> 0603WAF8202T5E; Manufacturer UNI-ROYAL(Uniroyal Elec) -> UNI-ROYAL; Minimum Qty 20 -> (none); Operating Temperature Range -55°C~+155°C -> (none); Overload Voltage (Max) 75V -> (none); Part 0603WAF8202T5E -> (none); Power(Watts) 100mW -> (none); Price 0.004USD -> (none); Process SMT -> (none); Resistance 82kΩ -> (none); Stock 541726 -> (none); Temperature Coefficient ±100ppm/°C -> (none); Type Thick Film Resistors -> (none); Voltage Rating (none) -> 75V
- R108, R109, R112: footprint PCM_JLCPCB:R_0603 -> MyParts:R0603; symbol PCM_JLCPCB-Resistors:0603,10kΩ -> MyParts:0603WAF1002T5E; Attrition Qty 10 -> (none); Category Resistors,Chip Resistor - Surface Mount -> (none); Class Basic Component -> (none); LCSC C25804 -> (none); LCSC Part (none) -> C25804; MPN (none) -> 0603WAF1002T5E; Manufacturer UNI-ROYAL(Uniroyal Elec) -> UNI-ROYAL; Minimum Qty 20 -> (none); Operating Temperature Range -55°C~+155°C -> (none); Overload Voltage (Max) 75V -> (none); Part 0603WAF1002T5E -> (none); Power(Watts) 100mW -> (none); Price 0.004USD -> (none); Process SMT -> (none); Resistance 10kΩ -> (none); Stock 51181774 -> (none); Temperature Coefficient ±100ppm/°C -> (none); Type Thick Film Resistors -> (none); Voltage Rating (none) -> 75V
- R110: footprint PCM_JLCPCB:R_0603 -> MyParts:R0603; symbol PCM_JLCPCB-Resistors:0603,180kΩ -> MyParts:0603WAF1803T5E; Attrition Qty 10 -> (none); Category Resistors,Chip Resistor - Surface Mount -> (none); Class Preferred Component -> (none); LCSC C22827 -> (none); LCSC Part (none) -> C22827; MPN (none) -> 0603WAF1803T5E; Manufacturer UNI-ROYAL(Uniroyal Elec) -> UNI-ROYAL; Minimum Qty 20 -> (none); Operating Temperature Range -55°C~+155°C -> (none); Overload Voltage (Max) 75V -> (none); Part 0603WAF1803T5E -> (none); Power(Watts) 100mW -> (none); Price 0.004USD -> (none); Process SMT -> (none); Resistance 180kΩ -> (none); Stock 453075 -> (none); Temperature Coefficient ±100ppm/°C -> (none); Type Thick Film Resistors -> (none); Voltage Rating (none) -> 75V
- R111: footprint PCM_JLCPCB:R_0603 -> MyParts:R0603; symbol PCM_JLCPCB-Resistors:0603,13kΩ -> MyParts:0603WAF1302T5E; Attrition Qty 10 -> (none); Category Resistors,Chip Resistor - Surface Mount -> (none); Class Basic Component -> (none); LCSC C22797 -> (none); LCSC Part (none) -> C22797; MPN (none) -> 0603WAF1302T5E; Manufacturer UNI-ROYAL(Uniroyal Elec) -> UNI-ROYAL; Minimum Qty 20 -> (none); Operating Temperature Range -55°C~+155°C -> (none); Overload Voltage (Max) 75V -> (none); Part 0603WAF1302T5E -> (none); Power(Watts) 100mW -> (none); Price 0.004USD -> (none); Process SMT -> (none); Resistance 13kΩ -> (none); Stock 264187 -> (none); Temperature Coefficient ±100ppm/°C -> (none); Type Thick Film Resistors -> (none); Voltage Rating (none) -> 75V
- SW3: MPN (none) -> SS-12F49-G050
- TP10, TP11, TP9: Manufacturer 荣和 -> ronghe
Other:
- sheet Power_5V ports: added 12V, 5V; removed none

Commit message: schematic cleanup
Parts:
- added TP18, TP26: TestPoint_Small, TestPoint:TestPoint_Pad_D1.5mm, symbol Connector:TestPoint_Small
Connections:
- net GND: now also TP26.1
- net at R104.2, U17.10 (ILIM): now also TP18.1

Commit message: Still refining
Parts:
- C100, R101, R103, R104, R105, R106, R107, R108, R109, R110, R111, R112: Pkg Type (none) -> SMD 0603
- C95: Pkg Type (none) -> SMD Aluminum electrolytic 6.3x7.7
- C96, C98: Pkg Type (none) -> SMD 0402
- C97: footprint MyParts:C0402 -> MyParts:C0603; symbol MyParts:CL05B104KO5NNNC -> MyParts:CC0603KRX7R9BB104; LCSC Part C1525 -> C14663; MPN CL05B104KO5NNNC -> CC0603KRX7R9BB104; Manufacturer SAMSUNG -> YAGEO; Pkg Type (none) -> SMD 0603; Voltage Rated 50V -> (none); Voltage Rating 16V -> 50V
- C99: Pkg Type (none) -> SMD 1206
- D41: Pkg Type (none) -> SMD SMA (DO-214AC)
- D42: Pkg Type (none) -> SMD SMB (DO-214AA)
- FB1: renamed from L1; Pkg Type (none) -> SMD 1206
- LED5: Pkg Type (none) -> SMD 0805
- Q10: Pkg Type (none) -> SMD SOIC-8
- Q11: Pkg Type (none) -> SMD SOT-23-3
- Q9: Pkg Type (none) -> SMD SOT-223
- SW3: Pkg Type (none) -> THT Slide switch
- TP10, TP11, TP9: Pkg Type (none) -> SMD Test point loop
- TP18, TP26: Pkg Type (none) -> SMD Test pad D1.5
- U17: Pkg Type (none) -> SMD QFN-24 4x4 EP
Connections:
- net GND: now also C97.2; no longer C97.1
- net V_BAT_F: now also C97.1; no longer C97.2

Commit message: Mods
Parts:
- added C110: 100nF, MyParts:C0603, symbol MyParts:CC0603KRX7R9BB104
- added TP34: TestPoint_Small, TestPoint:TestPoint_Pad_D1.5mm, symbol Connector:TestPoint_Small
- C96: Voltage Rated 50V -> (none)
- C98: footprint MyParts:C0402 -> MyParts:C0603; symbol MyParts:CL05B104KO5NNNC -> MyParts:CC0603KRX7R9BB104; LCSC Part C1525 -> C14663; MPN CL05B104KO5NNNC -> CC0603KRX7R9BB104; Manufacturer SAMSUNG -> YAGEO; Pkg Type SMD 0402 -> SMD 0603; Voltage Rated 50V -> (none); Voltage Rating 16V -> 50V
Connections:
- net EFUSE_OUT: now also C98.1; no longer C98.2
- net GND: now also C98.2, C110.2, TP34.1; no longer C98.1
- net at Q10.5 (D), Q10.6 (D), Q10.7 (D)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: now also C110.1
Other:
- note added: "EFUSE CURRENT LIMIT: R104 13k -> IOL = 40/13k = 3.08 A typ. Est. 2.7-3.4 A, from the datasheet IOL limits at 20k (-12/+8%) and 7.5k (-10/+11%) plus R104 1%. Branch demand ~1.9 A at 10 V: >= 40% margin at the low corner. REVERSE BATTERY: blocked by Q12 (SP40P04NK P-FET) at J1 on the top sheet, ahead of the F1/F2 split. Reversed: VGS = 0 and the body diode is reverse- biased, so no current flows, n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"
- note added: "Q9 - Services the switch, turn 12V on/off Q10 - reverse current blocking FET Q11 - fast gate pull-down for Q10"
- note added: "This circuit takes 12V from the battery, VBAT. Reverse battery is blocked by Q12 at J1 (top sheet). The eFuse limits to 3.08A typ (2.7-3.4A, see below)."
- note removed: "Q9 - Services the switch, turn 12V on/off Q10 - reverse VBAT polarity + reverse current blocking FET Q11 - fast gate pull-down for Q10"
- note removed: "This circuit takes 12V from the battery, VBAT. VBAT is reverse polarity protected with Q10. The eFuse limits to 3.1A."

Commit message: Ready to start layout
Parts:
- renumbered C110 to C24, C97 to C25, C99 to C26, C98 to C27, C95 to C28, C96 to C29, C100 to C30, D42 to D10, D41 to D11, LED5 to LED3, Q9 to Q2, Q10 to Q3, Q11 to Q4, R101 to R22, R103 to R23, R109 to R24, R112 to R25, R104 to R26, R110 to R27, R107 to R28, R105 to R29, R111 to R30, R108 to R31, R106 to R32, SW3 to SW1, TP9 to TP11, TP11 to TP12, TP10 to TP13, TP18 to TP14, TP26 to TP15, TP34 to TP16, U17 to U11
Other:
- note added: "EFUSE CURRENT LIMIT: R26 13k -> IOL = 40/13k = 3.08 A typ. Est. 2.7-3.4 A, from the datasheet IOL limits at 20k (-12/+8%) and 7.5k (-10/+11%) plus R26 1%. Branch demand ~1.9 A at 10 V: >= 40% margin at the low corner. REVERSE BATTERY: blocked by Q1 (SP40P04NK P-FET) at J1 on the top sheet, ahead of the F2/F1 split. Reversed: VGS = 0 and the body diode is reverse- biased, so no current flows, no f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"
- note added: "Place D10 close to IN_SYS"
- note added: "Q2 - Services the switch, turn 12V on/off Q3 - reverse current blocking FET Q4 - fast gate pull-down for Q3"
- note added: "Q2 = P-FET high-side switch, 12 V logic rail. SW1 closed -> gate pulled to GND, VGS = -12 V, Q2 ON (LED3 lights). SW1 open -> R22 pulls gate to source, VGS = 0, Q2 OFF."
- note added: "This circuit takes 12V from the battery, VBAT. Reverse battery is blocked by Q1 at J1 (top sheet). The eFuse limits to 3.08A typ (2.7-3.4A, see below)."
- note removed: "EFUSE CURRENT LIMIT: R104 13k -> IOL = 40/13k = 3.08 A typ. Est. 2.7-3.4 A, from the datasheet IOL limits at 20k (-12/+8%) and 7.5k (-10/+11%) plus R104 1%. Branch demand ~1.9 A at 10 V: >= 40% margin at the low corner. REVERSE BATTERY: blocked by Q12 (SP40P04NK P-FET) at J1 on the top sheet, ahead of the F1/F2 split. Reversed: VGS = 0 and the body diode is reverse- biased, so no current flows, n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"
- note removed: "Place D42 close to IN_SYS"
- note removed: "Q9 - Services the switch, turn 12V on/off Q10 - reverse current blocking FET Q11 - fast gate pull-down for Q10"
- note removed: "Q9 = P-FET high-side switch, 12 V logic rail. SW3 closed -> gate pulled to GND, VGS = -12 V, Q9 ON (LED5 lights). SW3 open -> R101 pulls gate to source, VGS = 0, Q9 OFF."
- note removed: "This circuit takes 12V from the battery, VBAT. Reverse battery is blocked by Q12 at J1 (top sheet). The eFuse limits to 3.08A typ (2.7-3.4A, see below)."

Commit message: IPC footprint renaming, battery sim added
Parts:
- added TP31: TestPoint_Small, TestPoint:TestPoint_Pad_D1.5mm, symbol Connector:TestPoint_Small
- C24, C25, C27, C30: footprint MyParts:C0603 -> MyPartsIPC:CAPC1608X95N
- C26: footprint MyParts:C1206 -> MyPartsIPC:CAPC3216X180N
- C28: footprint MyParts:CAP-SMD_BD6.3-L6.6-W6.6-FD -> MyPartsIPC:CAPAE660X770N
- C29: footprint MyParts:C0402 -> MyPartsIPC:CAPC1005X55N
- D10: footprint PCM_JLCPCB:D_SMB -> MyPartsIPC:DIOM5436X244N
- D11: footprint PCM_JLCPCB:D_SMA -> MyPartsIPC:DIOM5226X244N
- FB1: footprint MyParts:L1206 -> MyPartsIPC:INDC3216X130N
- LED3: footprint MyParts:LED0805-R-RD -> MyPartsIPC:LEDC2012X110N
- Q2: footprint Package_TO_SOT_SMD:SOT-223-3_TabPin2 -> MyPartsIPC:SOT230P700X180-4N
- Q3: footprint MyParts:SOP-8_L4.9-W3.9-P1.27-LS6.0-BL -> MyPartsIPC:SOIC127P600X175-8N
- Q4: footprint PCM_JLCPCB:Q_SOT-23 -> MyPartsIPC:SOT95P237X112-3N
- R22, R23, R24, R25, R26, R27, R28, R29, R30, R31, R32: footprint MyParts:R0603 -> MyPartsIPC:RESC1608X55N
- TP16: now left out of the parts list
- U11: footprint Package_DFN_QFN:QFN-24-1EP_4x4mm_P0.5mm_EP2.7x2.7mm_ThermalVias -> MyPartsIPC:QFN50P400X400X80-25N
Connections:
- net at C30.2, R29.2, R32.1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: now also TP31.1
Changed lines of the file:
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@@
 	(wire
 		(pts
-			(xy 125.73 110.49) (xy 125.73 125.73)
-		)
-		(stroke
-			(width 0)
-			(type default)
-		)
-	)
-	(wire
-		(pts
 			(xy 86.36 80.01) (xy 87.63 80.01)
 		)
@@
 			)
 		)
-		(property "Footprint" "MyParts:L1206"
+		(property "Footprint" "MyPartsIPC:INDC3216X130N"
 			(at 78.74 87.63 0)
 			(hide yes)
@@
 			)
 		)
-		(property "Footprint" "MyParts:R0603"
+		(property "Footprint" "MyPartsIPC:RESC1608X55N"
 			(at 110.49 129.54 0)
 			(hide yes)
@@
 			)
 		)
-		(property "Footprint" "MyParts:C1206"
+		(property "Footprint" "MyPartsIPC:CAPC3216X180N"
 			(at 100.33 104.14 0)
 			(hide yes)
@@
 			)
 		)
-		(property "Footprint" "MyParts:C0603"
+		(property "Footprint" "MyPartsIPC:CAPC1608X95N"
 			(at 120.65 130.81 0)
 			(hide yes)
@@
 			)
 		)
-		(property "Footprint" "MyParts:R0603"
+		(property "Footprint" "MyPartsIPC:RESC1608X55N"
 			(at 110.49 121.92 0)
 			(hide yes)
@@
 			)
 		)
-		(property "Footprint" "MyParts:R0603"
+		(property "Footprint" "MyPartsIPC:RESC1608X55N"
 			(at 151.13 71.12 0)
 			(hide yes)
@@
 			)
 		)
-		(property "Footprint" "MyParts:R0603"
+		(property "Footprint" "MyPartsIPC:RESC1608X55N"
 			(at 200.66 111.76 0)
 			(hide yes)
@@
 			)
 		)
-		(property "Footprint" "MyParts:R0603"
+		(property "Footprint" "MyPartsIPC:RESC1608X55N"
 			(at 78.74 121.92 0)
 			(hide yes)
@@
 			)
 		)
-		(property "Footprint" "MyParts:SOP-8_L4.9-W3.9-P1.27-LS6.0-BL"
+		(property "Footprint" "MyPartsIPC:SOIC127P600X175-8N"
 			(at 97.79 80.01 0)
 			(hide yes)
@@
 			)
 		)
-		(property "Footprint" "PCM_JLCPCB:D_SMB"
+		(property "Footprint" "MyPartsIPC:DIOM5436X244N"
 			(at 115.57 102.87 0)
 			(hide yes)
@@
 			)
 		)
-		(property "Footprint" "MyParts:LED0805-R-RD"
+		(property "Footprint" "MyPartsIPC:LEDC2012X110N"
 			(at 179.07 91.44 0)
 			(hide yes)
@@
 			)
 		)
-		(property "Footprint" "MyParts:C0603"
+		(property "Footprint" "MyPartsIPC:CAPC1608X95N"
 			(at 111.252 77.47 90)
 			(hide yes)
@@
 			)
 		)
-		(property "Footprint" "MyParts:R0603"
+		(property "Footprint" "MyPartsIPC:RESC1608X55N"
 			(at 158.75 111.76 0)
 			(hide yes)
@@
 			)
 		)
-		(property "Footprint" "MyParts:C0402"
+		(property "Footprint" "MyPartsIPC:CAPC1005X55N"
 			(at 147.32 118.11 0)
 			(hide yes)
@@
 		(body_style 1)
 		(exclude_from_sim no)
-		(in_bom yes)
+		(in_bom no)
 		(on_board yes)
 		(in_pos_files yes)
@@
 			)
 		)
-		(property "Footprint" "MyParts:R0603"
+		(property "Footprint" "MyPartsIPC:RESC1608X55N"
 			(at 48.26 114.3 0)
 			(hide yes)
@@
 			)
 		)
-		(property "Footprint" "Package_DFN_QFN:QFN-24-1EP_4x4mm_P0.5mm_EP2.7x2.7mm_ThermalVias"
+		(property "Footprint" "MyPartsIPC:QFN50P400X400X80-25N"
 			(at 134.62 80.01 0)
 			(hide yes)
@@
 			)
 		)
-		(property "Footprint" "MyParts:CAP-SMD_BD6.3-L6.6-W6.6-FD"
+		(property "Footprint" "MyPartsIPC:CAPAE660X770N"
 			(at 168.91 102.87 0)
 			(hide yes)
@@
 			)
 		)
-		(property "Footprint" "MyParts:R0603"
+		(property "Footprint" "MyPartsIPC:RESC1608X55N"
 			(at 78.74 129.54 0)
 			(hide yes)
@@
 			)
 		)
-		(property "Footprint" "MyParts:C0603"
+		(property "Footprint" "MyPartsIPC:CAPC1608X95N"
 			(at 85.852 104.14 90)
 			(hide yes)
@@
 			)
 		)
-		(property "Footprint" "PCM_JLCPCB:D_SMA"
+		(property "Footprint" "MyPartsIPC:DIOM5226X244N"
 			(at 181.61 102.87 0)
 			(hide yes)
@@
 			)
 		)
-		(property "Footprint" "Package_TO_SOT_SMD:SOT-223-3_TabPin2"
+		(property "Footprint" "MyPartsIPC:SOT230P700X180-4N"
 			(at 161.29 77.47 0)
 			(hide yes)
@@
 			)
 		)
-		(property "Footprint" "MyParts:R0603"
+		(property "Footprint" "MyPartsIPC:RESC1608X55N"
 			(at 181.61 85.09 0)
 			(hide yes)
@@
 			)
 		)
-		(property "Footprint" "PCM_JLCPCB:Q_SOT-23"
+		(property "Footprint" "MyPartsIPC:SOT95P237X112-3N"
 			(at 107.95 92.71 0)
 			(hide yes)
@@
 			)
 		)
-		(property "Footprint" "MyParts:R0603"
+		(property "Footprint" "MyPartsIPC:RESC1608X55N"
 			(at 58.42 114.3 0)
 			(hide yes)
@@
 			)
 		)
-		(property "Footprint" "MyParts:R0603"
+		(property "Footprint" "MyPartsIPC:RESC1608X55N"
 			(at 200.66 121.92 0)
 			(hide yes)
@@
 			)
 		)
-		(property "Footprint" "MyParts:C0603"
+		(property "Footprint" "MyPartsIPC:CAPC1608X95N"
 			(at 156.21 102.87 0)
 			(hide yes)
@@
 				)
 			)
+		)
+	)
+	(wire
+		(pts
+			(xy 125.73 110.49) (xy 125.73 119.38)
+		)
+		(stroke
+			(width 0)
+			(type default)
+		)
+	)
+	(wire
+		(pts
+			(xy 125.73 119.38) (xy 125.73 125.73)
+		)
+		(stroke
+			(width 0)
+			(type default)
+		)
+	)
+	(junction
+		(at 125.73 119.38)
+		(diameter 0)
+		(color 0 0 0 0)
+	)
+	(symbol
+		(lib_id "Connector:TestPoint_Small")
+		(at 125.73 119.38 90)
+		(unit 1)
+		(body_style 1)
+		(exclude_from_sim no)
+		(in_bom no)
+		(on_board yes)
+		(in_pos_files yes)
+		(dnp no)
+		(property "Reference" "TP31"
+			(at 123.19 119.38 0)
+			(show_name no)
+			(do_not_autoplace no)
+			(effects
+				(font
+					(size 1.27 1.27)
+				)
+				(justify right)
+			)
+		)
+		(property "Value" "TestPoint_Small"
+			(at 125.73 120.142 0)
+			(hide yes)
+			(show_name no)
+			(do_not_autoplace no)
+			(effects
+				(font
+					(size 1.27 1.27)
+				)
+			)
+		)
+		(property "Footprint" "TestPoint:TestPoint_Pad_D1.5mm"
+			(at 125.73 120.142 0)
+			(hide yes)
+			(show_name no)
+			(do_not_autoplace no)
+			(effects
+				(font
+					(size 1.27 1.27)
+				)
+			)
+		)
+		(property "Datasheet" ""
+			(at 125.73 119.38 0)
+			(show_name no)
+			(do_not_autoplace no)
+			(effects
+				(font
+					(size 1.27 1.27)
+				)
+			)
+		)
+		(property "Description" "Test Point"
+			(at 125.73 120.142 0)
+			(hide yes)
+			(show_name no)
+			(do_not_autoplace no)
+			(effects
+				(font
+					(size 1.27 1.27)
+				)
+			)
+		)
+		(pin "1"
+		)
+		(instances
+			(project "cm4-robo-controller"
+				(path "/c1285fbe-5f56-49a8-9041-410713cbe619/b81204ce-c2fc-430f-9caf-a4f2d6cea5c9"
+					(reference "TP31")
+					(unit 1)
+				)
+			)

Commit message: Updates after latest Tomachie review
Parts:
- added C82: 47nF, MyPartsIPC:CAPC1608X95N, symbol MyParts:CL10B473KB8NNNC
- added R91: 33kΩ, MyPartsIPC:RESC1608X55N, symbol MyParts:0603WAF3302T5E
- R22: value 100kΩ -> 33kΩ; symbol MyParts:0603WAF1003T5E -> MyParts:0603WAF3302T5E; LCSC Part C25803 -> C4216; MPN 0603WAF1003T5E -> 0603WAF3302T5E
Connections:
- net 12V: now also C82.2
- net at Q2.1 (G), R22.1, TP11.1: now also C82.1, R91.2; no longer SW1.2
- new net: R91.1, SW1.2
Other:
- note added: "Q2 = P-FET high-side switch, 12 V rail. SW1 closed: gate pulled low via R91 33k. R22/R91 halve VGS: -6.3 V at 12.6 V, -9.5 V at the 19 V OVP limit (+/-20 V). C82 47 nF gate-drain ramps 12V in ~2.6 ms, so no C28 inrush (was 63 A). SW1 open: R22 pulls gate to source, OFF."
- note added: "SW1 SWITCHES THE CM4 / LOGIC SUPPLY ONLY. With SW1 off the board still draws about 31 mA from the battery: RoboClaw logic ~30 mA (fed from V_MOTOR), U11 + UVLO/OVP/PGOOD dividers ~1.3 mA. A full 12 Ah battery runs flat in about 16 days. For storage or transport, unplug J1 (or pull F1 and F2), and charge the battery first."
- note removed: "Q2 = P-FET high-side switch, 12 V logic rail. SW1 closed -> gate pulled to GND, VGS = -12 V, Q2 ON (LED3 lights). SW1 open -> R22 pulls gate to source, VGS = 0, Q2 OFF."
