File: kicad/usb.kicad_sch (KiCad schematic)
At the start: 46 parts, among them J2 HX PZ2.54-2X5P TP, U2 FSUSB42MUX, U3 USB2514B-I/M2, U4 AP22653W6-7, U5 TPD4EUSB30DQAR, U6 TPD4EUSB30DQAR, U7 TPD4EUSB30DQAR, X1 24MHz

Commit message: PCB: route the USB differential pairs
- HD1-HD4, hub upstream, USB2 to CM4 and HSD2 to USB-C routed as 90 ohm pairs
- ESD parts (U5/U6/U7) routed flow-through: used N.C. pins tied to their lines
- Swap hub ports at J2 (HD3<->HD4) and USB1 (HD1<->HD2) to avoid pair crossings
- Move U6, U5, R63, R64, R14, C15, C18 to make room for the escapes
Connections:
- net HD1_N: now also U6.6 (N.C.), USB1.2 (D-); no longer USB1.6 (D-)
- net HD1_P: now also U6.7 (N.C.), USB1.3 (D+); no longer USB1.7 (D+)
- net HD2_N: now also U6.9 (N.C.), USB1.6 (D-); no longer USB1.2 (D-)
- net HD2_P: now also U6.10 (N.C.), USB1.7 (D+); no longer USB1.3 (D+)
- net HD3_N: now also J2.4, U7.6 (N.C.); no longer J2.3
- net HD3_P: now also J2.6, U7.7 (N.C.); no longer J2.5
- net HD4_N: now also J2.3, U7.9 (N.C.); no longer J2.4
- net HD4_P: now also J2.5, U7.10 (N.C.); no longer J2.6
- net HSD2+: now also U5.10 (N.C.)
- net HSD2-: now also U5.9 (N.C.)
- no-connect marks 19 -> 9
Changed lines of the file:
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@@
 	)
 	(no_connect
-		(at 50.8 139.7)
-	)
-	(no_connect
 		(at 95.25 55.88)
 	)
@@
 	)
 	(no_connect
-		(at 95.25 142.24)
-	)
-	(no_connect
-		(at 148.59 134.62)
-	)
-	(no_connect
-		(at 50.8 137.16)
-	)
-	(no_connect
-		(at 148.59 137.16)
-	)
-	(no_connect
-		(at 95.25 144.78)
-	)
-	(no_connect
 		(at 50.8 147.32)
 	)
@@
 	)
 	(no_connect
-		(at 148.59 144.78)
-	)
-	(no_connect
-		(at 95.25 137.16)
-	)
-	(no_connect
-		(at 95.25 134.62)
-	)
-	(no_connect
 		(at 153.67 187.96)
 	)
@@
 	)
 	(no_connect
-		(at 148.59 142.24)
-	)
-	(no_connect
 		(at 50.8 144.78)
 	)
@@
 	(wire
 		(pts
-			(xy 97.79 139.7) (xy 97.79 140.97)
-		)
-		(stroke
-			(width 0)
-			(type default)
-		)
-	)
-	(wire
-		(pts
 			(xy 179.07 133.35) (xy 194.31 133.35)
 		)
@@
 	(wire
 		(pts
-			(xy 148.59 139.7) (xy 151.13 139.7)
-		)
-		(stroke
-			(width 0)
-			(type default)
-		)
-	)
-	(wire
-		(pts
 			(xy 162.56 50.8) (xy 165.1 50.8)
 		)
@@
 	(wire
 		(pts
-			(xy 151.13 139.7) (xy 151.13 140.97)
-		)
-		(stroke
-			(width 0)
-			(type default)
-		)
-	)
-	(wire
-		(pts
 			(xy 46.99 80.01) (xy 50.8 80.01)
 		)
@@
 	(wire
 		(pts
-			(xy 95.25 139.7) (xy 97.79 139.7)
-		)
-		(stroke
-			(width 0)
-			(type default)
-		)
-	)
-	(wire
-		(pts
 			(xy 115.57 36.83) (xy 115.57 35.56)
 		)
@@
 		)
 	)
-	(label "HD4_P"
+	(label "HD3_P"
 		(at 162.56 182.88 180)
 		(effects
@@
 		)
 	)
-	(label "HD2_N"
+	(label "HD1_N"
 		(at 204.47 81.28 180)
 		(effects
@@
 		)
 	)
-	(label "HD3_P"
+	(label "HD4_P"
 		(at 132.08 182.88 0)
 		(effects
@@
 		)
 	)
-	(label "HD1_P"
+	(label "HD2_P"
 		(at 229.87 83.82 0)
 		(effects
@@
 		)
 	)
-	(label "HD2_P"
+	(label "HD1_P"
 		(at 204.47 83.82 180)
 		(effects
@@
 		)
 	)
-	(label "HD3_N"
+	(label "HD4_N"
 		(at 132.08 180.34 0)
 		(effects
@@
 		)
 	)
-	(label "HD1_N"
+	(label "HD2_N"
 		(at 229.87 81.28 0)
 		(effects
@@
 		)
 	)
-	(label "HD4_N"
+	(label "HD3_N"
 		(at 162.56 180.34 180)
 		(effects
@@
 	(symbol
 		(lib_id "power:GND")
-		(at 97.79 140.97 0)
+		(at 95.25 139.7 90)
 		(unit 1)
 		(body_style 1)
@@
 		(dnp no)
 		(property "Reference" "#PWR098"
-			(at 101.6 140.97 0)
+			(at 99.06 139.7 90)
 			(hide yes)
 			(show_name no)
@@
 		)
 		(property "Value" "GND"
-			(at 93.98 140.97 0)
+			(at 91.44 139.7 90)
 			(hide yes)
 			(show_name no)
@@
 		)
 		(property "Footprint" ""
-			(at 97.79 140.97 0)
+			(at 95.25 139.7 90)
 			(show_name no)
 			(do_not_autoplace no)
@@
 		)
 		(property "Datasheet" ""
-			(at 97.79 140.97 0)
+			(at 95.25 139.7 90)
 			(show_name no)
 			(do_not_autoplace no)
@@
 		)
 		(property "Description" "Power symbol creates a global label with name \"GND\" , ground"
-			(at 97.79 140.97 0)
+			(at 95.25 139.7 90)
 			(hide yes)
 			(show_name no)
@@
 	(symbol
 		(lib_id "power:GND")
-		(at 151.13 140.97 0)
+		(at 148.59 139.7 90)
 		(unit 1)
 		(body_style 1)
@@
 		(dnp no)
 		(property "Reference" "#PWR0103"
-			(at 154.94 140.97 0)
+			(at 152.4 139.7 90)
 			(hide yes)
 			(show_name no)
@@
 		)
 		(property "Value" "GND"
-			(at 147.32 140.97 0)
+			(at 144.78 139.7 90)
 			(hide yes)
 			(show_name no)
@@
 		)
 		(property "Footprint" ""
-			(at 151.13 140.97 0)
+			(at 148.59 139.7 90)
 			(show_name no)
 			(do_not_autoplace no)
@@
 		)
 		(property "Datasheet" ""
-			(at 151.13 140.97 0)
+			(at 148.59 139.7 90)
 			(show_name no)
 			(do_not_autoplace no)
@@
 		)
 		(property "Description" "Power symbol creates a global label with name \"GND\" , ground"
-			(at 151.13 140.97 0)
+			(at 148.59 139.7 90)
 			(hide yes)
 			(show_name no)
@@
 		)
 	)
+	(label "HD2_P"
+		(at 95.25 134.62 0)
+		(effects
+			(font
+				(size 1.27 1.27)
+			)
+			(justify left bottom)
+		)
+	)
+	(label "HD2_N"
+		(at 95.25 137.16 0)
+		(effects
+			(font
+				(size 1.27 1.27)
+			)
+			(justify left bottom)
+		)
+	)
+	(label "HD1_P"
+		(at 95.25 142.24 0)
+		(effects
+			(font
+				(size 1.27 1.27)
+			)
+			(justify left bottom)
+		)
+	)
+	(label "HD1_N"
+		(at 95.25 144.78 0)
+		(effects
+			(font
+				(size 1.27 1.27)
+			)
+			(justify left bottom)
+		)
+	)
+	(label "HD4_P"
+		(at 148.59 134.62 0)
+		(effects
+			(font
+				(size 1.27 1.27)
+			)
+			(justify left bottom)
+		)
+	)
+	(label "HD4_N"
+		(at 148.59 137.16 0)
+		(effects
+			(font
+				(size 1.27 1.27)
+			)
+			(justify left bottom)
+		)
+	)
+	(label "HD3_P"
+		(at 148.59 142.24 0)
+		(effects
+			(font
+				(size 1.27 1.27)
+			)
+			(justify left bottom)
+		)
+	)
+	(label "HD3_N"
+		(at 148.59 144.78 0)
+		(effects
+			(font
+				(size 1.27 1.27)
+			)
+			(justify left bottom)
+		)
+	)
+	(label "HSD2+"
+		(at 50.8 137.16 0)
+		(effects
+			(font
+				(size 1.27 1.27)
+			)
+			(justify left bottom)
+		)
+	)
+	(label "HSD2-"
+		(at 50.8 139.7 0)
+		(effects
+			(font
+				(size 1.27 1.27)
+			)
+			(justify left bottom)
+		)
+	)
