File: kicad/ethernet.kicad_sch (KiCad schematic)
At the start: 6 parts, among them U7 TPD4EUSB30DQAR, U8 TPD4EUSB30DQAR

Commit message: GPIO connectors defined
Parts:
- C17: footprint PCM_JLCPCB:C_0402 -> MyParts:C0402; symbol PCM_JLCPCB-Capacitors:0402,100nF -> MyParts:CL05B104KO5NNNC_ALT; Attrition Qty 10 -> (none); Capacitance 100nF -> (none); Category Capacitors,Multilayer Ceramic Capacitors MLCC - SMD/SMT -> (none); Class Basic Component -> (none); LCSC C1525 -> (none); LCSC Part (none) -> C1525; MPN (none) -> CL05B104KO5NNNC; Manufacturer Samsung Electro-Mechanics -> SAMSUNG; Minimum Qty 20 -> (none); Part CL05B104KO5NNNC -> (none); Price 0.004USD -> (none); Process SMT -> (none); Stock 20208285 -> (none); Temperature Coefficient X7R -> (none); Voltage Rated 16V -> (none); Voltage Rating (none) -> 16V
- R16, R17: Manufacturer UNI-ROYAL(厚声) -> UNI-ROYAL; Tolerance (none) -> ±1%; Voltage Rating (none) -> 50V
- RJ1: Manufacturer HANRUN(汉仁) -> HANRUN
- U7, U8: Manufacturer TI(德州仪器) -> TI
Changed lines of the file:
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@@
 			)
 		)
-		(property "Datasheet" "https://lcsc.com/product-detail/Chip-Resistor-Surface-Mount-UniOhm_220R-2200-1_C25091.html"
+		(property "Datasheet" "${MYPARTS_DATASHEETS}/0402WGF2200TCE.pdf"
 			(at 102.87 35.56 0)
 			(hide yes)
@@
 			)
 		)
-		(property "Description" "220Ω (2200) ±1%"
+		(property "Description" "-55℃~+155℃ 220Ω 50V 62.5mW Thick Film Resistor ±1% ±100ppm/℃ 0402 Chip Resistor - Surface Mount ROHS"
 			(at 102.87 22.86 0)
 			(hide yes)
@@
 			)
 		)
-		(property "Manufacturer" "UNI-ROYAL(厚声)"
+		(property "Manufacturer" "UNI-ROYAL"
 			(at 102.87 33.02 0)
 			(hide yes)
@@
 		(property "LCSC Part" "C25091"
 			(at 102.87 27.94 0)
+			(hide yes)
+			(show_name no)
+			(do_not_autoplace no)
+			(effects
+				(font
+					(size 1.27 1.27)
+				)
+			)
+		)
+		(property "Tolerance" "±1%"
+			(at 102.87 45.72 0)
+			(hide yes)
+			(show_name no)
+			(do_not_autoplace no)
+			(effects
+				(font
+					(size 1.27 1.27)
+				)
+			)
+		)
+		(property "Voltage Rating" "50V"
+			(at 102.87 45.72 0)
 			(hide yes)
 			(show_name no)
@@
 			)
 		)
-		(property "Datasheet" "https://lcsc.com/product-detail/USB_TI_TPD4EUSB30DQAR_TPD4EUSB30DQAR_C90627.html"
+		(property "Datasheet" "${MYPARTS_DATASHEETS}/TPD4EUSB30DQAR.pdf"
 			(at 203.2 111.76 0)
 			(hide yes)
@@
 			)
 		)
-		(property "Description" ""
+		(property "Description" "-40℃~+85℃ 0.8pF 45W@8/20us 5.5V 5A@8/20us 7V 8V ESD Four channels IEC 61000-4-2, IEC 61000-4-5 Unidirectional USON-10(1x2.5) ESD and Surge Protection (TVS/ESD) ROHS"
 			(at 203.2 96.52 0)
 			(hide yes)
@@
 			)
 		)
-		(property "Manufacturer" "TI(德州仪器)"
+		(property "Manufacturer" "TI"
 			(at 203.2 114.3 0)
 			(hide yes)
@@
 			)
 		)
-		(property "Datasheet" "https://lcsc.com/product-detail/RJ45_HR911130A_C54408.html"
+		(property "Datasheet" "${MYPARTS_DATASHEETS}/HR911130A.pdf"
 			(at 91.44 132.66 0)
 			(hide yes)
@@
 			)
 		)
-		(property "Description" ""
+		(property "Description" "CONN MOD JACK RJ45 TH"
 			(at 91.44 87.63 0)
 			(show_name no)
@@
 			)
 		)
-		(property "Manufacturer" "HANRUN(汉仁)"
+		(property "Manufacturer" "HANRUN"
 			(at 91.44 135.16 0)
 			(hide yes)
@@
 	)
 	(symbol
-		(lib_id "PCM_JLCPCB-Capacitors:0402,100nF")
+		(lib_id "MyParts:CL05B104KO5NNNC_ALT")
 		(at 50.8 116.84 0)
 		(unit 1)
@@
 			)
 		)
-		(property "Footprint" "PCM_JLCPCB:C_0402"
+		(property "Footprint" "MyParts:C0402"
 			(at 49.022 116.84 90)
 			(hide yes)
@@
 			)
 		)
-		(property "Datasheet" "https://www.lcsc.com/datasheet/lcsc_datasheet_2304140030_Samsung-Electro-Mechanics-CL05B104KO5NNNC_C1525.pdf"
+		(property "Datasheet" "${MYPARTS_DATASHEETS}/CL05B104KO5NNNC.pdf"
 			(at 50.8 116.84 0)
 			(hide yes)
@@
 			)
 		)
-		(property "Description" "16V 100nF X7R ±10% 0402 Multilayer Ceramic Capacitors MLCC - SMD/SMT ROHS"
+		(property "Description" "100nF 16V X7R ±10% 0402 Multilayer Ceramic Capacitors MLCC - SMD/SMT ROHS"
 			(at 50.8 116.84 0)
 			(hide yes)
@@
 			)
 		)
-		(property "LCSC" "C1525"
+		(property "Manufacturer" "SAMSUNG"
 			(at 50.8 116.84 0)
 			(hide yes)
@@
 					(size 1.27 1.27)
 				)
-			)
-		)
-		(property "Stock" "20208285"
-			(at 50.8 116.84 0)
-			(hide yes)
-			(show_name no)
-			(do_not_autoplace no)
-			(effects
-				(font
-					(size 1.27 1.27)
-				)
-			)
-		)
-		(property "Price" "0.004USD"
-			(at 50.8 116.84 0)
-			(hide yes)
-			(show_name no)
-			(do_not_autoplace no)
-			(effects
-				(font
-					(size 1.27 1.27)
-				)
-			)
-		)
-		(property "Process" "SMT"
-			(at 50.8 116.84 0)
-			(hide yes)
-			(show_name no)
-			(do_not_autoplace no)
-			(effects
-				(font
-					(size 1.27 1.27)
-				)
-			)
-		)
-		(property "Minimum Qty" "20"
-			(at 50.8 116.84 0)
-			(hide yes)
-			(show_name no)
-			(do_not_autoplace no)
-			(effects
-				(font
-					(size 1.27 1.27)
-				)
-			)
-		)
-		(property "Attrition Qty" "10"
-			(at 50.8 116.84 0)
-			(hide yes)
-			(show_name no)
-			(do_not_autoplace no)
-			(effects
-				(font
-					(size 1.27 1.27)
-				)
-			)
-		)
-		(property "Class" "Basic Component"
-			(at 50.8 116.84 0)
-			(hide yes)
-			(show_name no)
-			(do_not_autoplace no)
-			(effects
-				(font
-					(size 1.27 1.27)
-				)
-			)
-		)
-		(property "Category" "Capacitors,Multilayer Ceramic Capacitors MLCC - SMD/SMT"
-			(at 50.8 116.84 0)
-			(hide yes)
-			(show_name no)
-			(do_not_autoplace no)
-			(effects
-				(font
-					(size 1.27 1.27)
-				)
-			)
-		)
-		(property "Manufacturer" "Samsung Electro-Mechanics"
-			(at 50.8 116.84 0)
-			(hide yes)
-			(show_name no)
-			(do_not_autoplace no)
-			(effects
-				(font
-					(size 1.27 1.27)
-				)
-			)
-		)
-		(property "Part" "CL05B104KO5NNNC"
-			(at 50.8 116.84 0)
-			(hide yes)
-			(show_name no)
-			(do_not_autoplace no)
-			(effects
-				(font
-					(size 1.27 1.27)
-				)
-			)
-		)
-		(property "Voltage Rated" "16V"
-			(at 45.212 118.872 0)
-			(show_name no)
-			(do_not_autoplace no)
-			(effects
-				(font
-					(size 0.8 0.8)
-				)
-				(justify left)
 			)
 		)
@@
 			)
 		)
-		(property "Capacitance" "100nF"
+		(property "MPN" "CL05B104KO5NNNC"
 			(at 50.8 116.84 0)
 			(hide yes)
@@
 			)
 		)
-		(property "Temperature Coefficient" "X7R"
+		(property "Voltage Rating" "16V"
+			(at 50.8 116.84 0)
+			(hide yes)
+			(show_name no)
+			(do_not_autoplace no)
+			(effects
+				(font
+					(size 1.27 1.27)
+				)
+			)
+		)
+		(property "LCSC Part" "C1525"
 			(at 50.8 116.84 0)
 			(hide yes)
@@
 			)
 		)
-		(property "Datasheet" "https://lcsc.com/product-detail/USB_TI_TPD4EUSB30DQAR_TPD4EUSB30DQAR_C90627.html"
+		(property "Datasheet" "${MYPARTS_DATASHEETS}/TPD4EUSB30DQAR.pdf"
 			(at 203.2 81.28 0)
 			(hide yes)
@@
 			)
 		)
-		(property "Description" ""
+		(property "Description" "-40℃~+85℃ 0.8pF 45W@8/20us 5.5V 5A@8/20us 7V 8V ESD Four channels IEC 61000-4-2, IEC 61000-4-5 Unidirectional USON-10(1x2.5) ESD and Surge Protection (TVS/ESD) ROHS"
 			(at 203.2 66.04 0)
 			(hide yes)
@@
 			)
 		)
-		(property "Manufacturer" "TI(德州仪器)"
+		(property "Manufacturer" "TI"
 			(at 203.2 83.82 0)
 			(hide yes)
@@
 			)
 		)
-		(property "Datasheet" "https://lcsc.com/product-detail/Chip-Resistor-Surface-Mount-UniOhm_220R-2200-1_C25091.html"
+		(property "Datasheet" "${MYPARTS_DATASHEETS}/0402WGF2200TCE.pdf"
 			(at 62.23 36.83 0)
 			(hide yes)
@@
 			)
 		)
-		(property "Description" "220Ω (2200) ±1%"
+		(property "Description" "-55℃~+155℃ 220Ω 50V 62.5mW Thick Film Resistor ±1% ±100ppm/℃ 0402 Chip Resistor - Surface Mount ROHS"
 			(at 62.23 24.13 0)
 			(hide yes)
@@
 			)
 		)
-		(property "Manufacturer" "UNI-ROYAL(厚声)"
+		(property "Manufacturer" "UNI-ROYAL"
 			(at 62.23 34.29 0)
 			(hide yes)
@@
 			(hide yes)
 			(show_name no)
+			(do_not_autoplace no)
+			(effects
+				(font
+					(size 1.27 1.27)
+				)
+			)
+		)
+		(property "Tolerance" "±1%"
+			(at 62.23 46.99 0)
+			(hide yes)
+			(show_name no)
+			(do_not_autoplace no)
+			(effects
+				(font
+					(size 1.27 1.27)
+				)
+			)
+		)
+		(property "Voltage Rating" "50V"
+			(at 62.23 46.99 0)
+			(hide yes)
+			(show_name no)

Commit message: Still refining
Parts:
- C17, R16, R17: Pkg Type (none) -> SMD 0402
- RJ1: Pkg Type (none) -> THT RJ45 with magnetics
- U7, U8: Pkg Type (none) -> SMD USON-10 2.5x1.0
Connections:
- net GND: no longer RJ1.P10, RJ1.SHIELD0, RJ1.SHIELD1
- new net CHASSIS: RJ1.P10, RJ1.SHIELD0, RJ1.SHIELD1
Changed lines of the file:
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@@
+			)
+		)
+		(property "Pkg Type" "SMD 0402"
+			(at 102.87 45.72 0)
+			(hide yes)
+			(show_name no)
+			(do_not_autoplace no)
+			(effects
+				(font
+					(size 1.27 1.27)
+				)
 			)
 		)
@@
 			)
 		)
+		(property "Pkg Type" "SMD USON-10 2.5x1.0"
+			(at 203.2 96.52 0)
+			(hide yes)
+			(show_name no)
+			(do_not_autoplace no)
+			(effects
+				(font
+					(size 1.27 1.27)
+				)
+			)
+		)
 		(pin "1"
 		)
@@
 		(property "LCSC Part" "C54408"
 			(at 91.44 140.16 0)
+			(hide yes)
+			(show_name no)
+			(do_not_autoplace no)
+			(effects
+				(font
+					(size 1.27 1.27)
+				)
+			)
+		)
+		(property "Pkg Type" "THT RJ45 with magnetics"
+			(at 91.44 87.63 0)
 			(hide yes)
 			(show_name no)
@@
 	)
 	(symbol
-		(lib_id "power:GND")
+		(lib_id "power:Earth")
 		(at 57.15 128.27 0)
 		(unit 1)
@@
 			)
 		)
-		(property "Value" "GND"
+		(property "Value" "CHASSIS"
 			(at 57.15 133.35 0)
 			(show_name no)
@@
 			)
 		)
-		(property "Description" "Power symbol creates a global label with name \"GND\" , ground"
+		(property "Description" "Power symbol creates a global label with name \"Earth\""
 			(at 57.15 128.27 0)
 			(hide yes)
@@
 		)
 		(property "LCSC Part" "C1525"
+			(at 50.8 116.84 0)
+			(hide yes)
+			(show_name no)
+			(do_not_autoplace no)
+			(effects
+				(font
+					(size 1.27 1.27)
+				)
+			)
+		)
+		(property "Pkg Type" "SMD 0402"
 			(at 50.8 116.84 0)
 			(hide yes)
@@
 			)
 		)
+		(property "Pkg Type" "SMD USON-10 2.5x1.0"
+			(at 203.2 66.04 0)
+			(hide yes)
+			(show_name no)
+			(do_not_autoplace no)
+			(effects
+				(font
+					(size 1.27 1.27)
+				)
+			)
+		)
 		(pin "1"
 		)
@@
 			(at 62.23 46.99 0)
 			(hide yes)
+			(show_name no)
+			(do_not_autoplace no)
+			(effects
+				(font
+					(size 1.27 1.27)
+				)
+			)
+		)
+		(property "Pkg Type" "SMD 0402"
+			(at 62.23 46.99 0)
+			(hide yes)

Commit message: Mods
Other:
- note added: "Clamps all four pairs on the CM4 side of the magnetics. Place both at RJ1. Matches CM4 datasheet Fig. 2 (TPD4EUSB30 on all pairs). TPD4EUSB30 IO range is 0-5.5 V, so EP lines must stay >= 0 V. MDI DC level is set inside the BCM54210PE (not published; CT is AC-grounded only). First boards: scope each EP line to GND at the clamps at 1000/100/10 (ethtool -s eth0 speed N duplex full autoneg off). Min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"
- note added: "HR911130A, shielded, integrated magnetics and LEDs, 100/1000Base-T (LCSC C54408). EP0-EP3 come straight from the CM4 - the PHY is on the module, no external PHY. Chip-side center taps (P1) bypassed to GND by C17 100nF. Bob Smith termination (4x75R + 1000pF/2kV) is built into the jack; P10 is that node, tied to CHASSIS. Shield pins are also on CHASSIS (bled to GND by R136/C109 on the top sheet)."
- note added: "Use JLC's impedance calculator for the stackup to get width and gap for 100 Ω (Ethernet) and 90 Ω (USB) differential on the outer layers. Put those values into ETH_100_OHM and USB_90_OHM. Order with impedance control enabled, so JLC adjusts to the target."
- note removed: "Clamps all four pairs on the CM4 side of the magnetics. Place both at RJ1."
- note removed: "HR911130A, shielded, integrated magnetics and LEDs, 100/1000Base-T (LCSC C54408). EP0-EP3 come straight from the CM4 - the PHY is on the module, no external PHY. Chip-side center taps (P1) bypassed to GND by C17 100nF. Bob Smith termination (4x75R + 1000pF/2kV) is built into the jack; P10 is that node, tied to GND. Shield pins tied to signal GND."
Changed lines of the file:
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@@
 		)
 	)
-	(text "HR911130A, shielded, integrated magnetics and LEDs, 100/1000Base-T (LCSC C54408).\nEP0-EP3 come straight from the CM4 - the PHY is on the module, no external PHY.\nChip-side center taps (P1) bypassed to GND by C17 100nF.\nBob Smith termination (4x75R + 1000pF/2kV) is built into the jack; P10 is that node, tied to GND.\nShield pins tied to signal GND."
+	(text "Use JLC's impedance calculator for the stackup to get \nwidth and gap for 100 Ω (Ethernet) and 90 Ω (USB) differential \non the outer layers. Put those values into ETH_100_OHM and USB_90_OHM.\nOrder with impedance control enabled, so JLC adjusts to the target."
+		(exclude_from_sim no)
+		(at 168.148 149.352 0)
+		(effects
+			(font
+				(size 1.27 1.27)
+			)
+			(justify left)
+		)
+	)
+	(text "HR911130A, shielded, integrated magnetics and LEDs, 100/1000Base-T (LCSC C54408).\nEP0-EP3 come straight from the CM4 - the PHY is on the module, no external PHY.\nChip-side center taps (P1) bypassed to GND by C17 100nF.\nBob Smith termination (4x75R + 1000pF/2kV) is built into the jack;\nP10 is that node, tied to CHASSIS. Shield pins are also on CHASSIS\n(bled to GND by R136/C109 on the top sheet)."
 		(exclude_from_sim no)
 		(at 43.688 142.24 0)
@@
 		)
 	)
-	(text "Clamps all four pairs on the CM4 side of the magnetics. \nPlace both at RJ1."
+	(text "Clamps all four pairs on the CM4 side of the magnetics. \nPlace both at RJ1.\n\nMatches CM4 datasheet Fig. 2 (TPD4EUSB30 on all pairs).\nTPD4EUSB30 IO range is 0-5.5 V, so EP lines must stay\n>= 0 V. MDI DC level is set inside the BCM54210PE\n(not published; CT is AC-grounded only).\nFirst boards: scope each EP line to GND at the clamps\nat 1000/100/10 (ethtool -s eth0 speed N duplex full\nautoneg off). Minimum must be >= -0.3 V."
 		(exclude_from_sim no)
 		(at 177.038 116.078 0)

Commit message: Ready to start layout
Parts:
- renumbered C17 to C23, R16 to R18, R17 to R19, U7 to U8, U8 to U9
Other:
- note added: "CM4 Ethernet_nLED pins are active-low 3.3V sinks, IOL 8mA @ VOL 0.4V. ETH_LEDG = activity (green, RJ1 pin 11 anode / 12 cathode). ETH_LEDY = link speed (yellow, pin 14 anode / 13 cathode). R18/R19 220R gives ~4.5mA through the LED. That is below the 8mA limit."
- note added: "Clamps all four pairs on the CM4 side of the magnetics. Place both at RJ1. Matches CM4 datasheet Fig. 2 (TPD4EUSB30 on all pairs). TPD4EUSB30 IO abs max is 0 to 6 V (TI p.4), so EP lines must stay >= 0 V. MDI DC level is set inside the BCM54210PE (not published; CT is AC-grounded only). First boards: scope each EP line to GND at the clamps at 1000/100/10 (ethtool -s eth0 speed N duplex full auton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"
- note added: "HR911130A, shielded, integrated magnetics and LEDs, 100/1000Base-T (LCSC C54408). EP0-EP3 come straight from the CM4 - the PHY is on the module, no external PHY. Chip-side center taps (P1) bypassed to GND by C23 100nF. Bob Smith termination (4x75R + 1000pF/2kV) is built into the jack; P10 is that node, tied to CHASSIS. Shield pins are also on CHASSIS (bled to GND by R2/C1 on the top sheet)."
- note removed: "CM4 Ethernet_nLED pins are active-low 3.3V sinks, IOL 8mA @ VOL 0.4V. ETH_LEDG = activity (green, RJ1 pin 11 anode / 12 cathode). ETH_LEDY = link speed (yellow, pin 14 anode / 13 cathode). R16/R17 220R gives ~4.5mA through the LED. That is below the 8mA limit."
- note removed: "Clamps all four pairs on the CM4 side of the magnetics. Place both at RJ1. Matches CM4 datasheet Fig. 2 (TPD4EUSB30 on all pairs). TPD4EUSB30 IO range is 0-5.5 V, so EP lines must stay >= 0 V. MDI DC level is set inside the BCM54210PE (not published; CT is AC-grounded only). First boards: scope each EP line to GND at the clamps at 1000/100/10 (ethtool -s eth0 speed N duplex full autoneg off). Min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"
- note removed: "HR911130A, shielded, integrated magnetics and LEDs, 100/1000Base-T (LCSC C54408). EP0-EP3 come straight from the CM4 - the PHY is on the module, no external PHY. Chip-side center taps (P1) bypassed to GND by C17 100nF. Bob Smith termination (4x75R + 1000pF/2kV) is built into the jack; P10 is that node, tied to CHASSIS. Shield pins are also on CHASSIS (bled to GND by R136/C109 on the top sheet)."
Changed lines of the file:
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@@
 		)
 	)
-	(text "HR911130A, shielded, integrated magnetics and LEDs, 100/1000Base-T (LCSC C54408).\nEP0-EP3 come straight from the CM4 - the PHY is on the module, no external PHY.\nChip-side center taps (P1) bypassed to GND by C17 100nF.\nBob Smith termination (4x75R + 1000pF/2kV) is built into the jack;\nP10 is that node, tied to CHASSIS. Shield pins are also on CHASSIS\n(bled to GND by R136/C109 on the top sheet)."
+	(text "HR911130A, shielded, integrated magnetics and LEDs, 100/1000Base-T (LCSC C54408).\nEP0-EP3 come straight from the CM4 - the PHY is on the module, no external PHY.\nChip-side center taps (P1) bypassed to GND by C23 100nF.\nBob Smith termination (4x75R + 1000pF/2kV) is built into the jack;\nP10 is that node, tied to CHASSIS. Shield pins are also on CHASSIS\n(bled to GND by R2/C1 on the top sheet)."
 		(exclude_from_sim no)
 		(at 43.688 142.24 0)
@@
 		)
 	)
-	(text "Clamps all four pairs on the CM4 side of the magnetics. \nPlace both at RJ1.\n\nMatches CM4 datasheet Fig. 2 (TPD4EUSB30 on all pairs).\nTPD4EUSB30 IO range is 0-5.5 V, so EP lines must stay\n>= 0 V. MDI DC level is set inside the BCM54210PE\n(not published; CT is AC-grounded only).\nFirst boards: scope each EP line to GND at the clamps\nat 1000/100/10 (ethtool -s eth0 speed N duplex full\nautoneg off). Minimum must be >= -0.3 V."
+	(text "Clamps all four pairs on the CM4 side of the magnetics. \nPlace both at RJ1.\n\nMatches CM4 datasheet Fig. 2 (TPD4EUSB30 on all pairs).\nTPD4EUSB30 IO abs max is 0 to 6 V (TI p.4), so EP lines must stay\n>= 0 V. MDI DC level is set inside the BCM54210PE\n(not published; CT is AC-grounded only).\nFirst boards: scope each EP line to GND at the clamps\nat 1000/100/10 (ethtool -s eth0 speed N duplex full\nautoneg off). Minimum must be >= 0 V (no undershoot below GND)."
 		(exclude_from_sim no)
 		(at 177.038 116.078 0)
@@
 		)
 	)
-	(text "CM4 Ethernet_nLED pins are active-low 3.3V sinks, IOL 8mA @ VOL 0.4V.\nETH_LEDG = activity (green, RJ1 pin 11 anode / 12 cathode).\nETH_LEDY = link speed (yellow, pin 14 anode / 13 cathode).\nR16/R17 220R gives ~4.5mA through the LED. That is below the 8mA limit.\n"
+	(text "CM4 Ethernet_nLED pins are active-low 3.3V sinks, IOL 8mA @ VOL 0.4V.\nETH_LEDG = activity (green, RJ1 pin 11 anode / 12 cathode).\nETH_LEDY = link speed (yellow, pin 14 anode / 13 cathode).\nR18/R19 220R gives ~4.5mA through the LED. That is below the 8mA limit.\n"
 		(exclude_from_sim no)
 		(at 43.942 154.94 0)
@@
 		(in_pos_files yes)
 		(dnp no)
-		(property "Reference" "R17"
+		(property "Reference" "R19"
 			(at 100.838 43.434 0)
 			(show_name no)
@@
 			(project "cm4-robo-controller"
 				(path "/c1285fbe-5f56-49a8-9041-410713cbe619/3cc0f123-2315-4414-aa85-3a1a0bb694eb/2c385700-431a-4a3a-8a9d-f3682fa19093"
-					(reference "R17")
+					(reference "R19")
 					(unit 1)
 				)
@@
 		(dnp no)
 		(fields_autoplaced yes)
-		(property "Reference" "U8"
+		(property "Reference" "U9"
 			(at 203.2 83.82 0)
 			(show_name no)
@@
 			(project "cm4-robo-controller"
 				(path "/c1285fbe-5f56-49a8-9041-410713cbe619/3cc0f123-2315-4414-aa85-3a1a0bb694eb/2c385700-431a-4a3a-8a9d-f3682fa19093"
-					(reference "U8")
+					(reference "U9")
 					(unit 1)
 				)
@@
 		(in_pos_files yes)
 		(dnp no)
-		(property "Reference" "C17"
+		(property "Reference" "C23"
 			(at 45.212 113.7919 0)
 			(show_name no)
@@
 			(project "cm4-robo-controller"
 				(path "/c1285fbe-5f56-49a8-9041-410713cbe619/3cc0f123-2315-4414-aa85-3a1a0bb694eb/2c385700-431a-4a3a-8a9d-f3682fa19093"
-					(reference "C17")
+					(reference "C23")
 					(unit 1)
 				)
@@
 		(dnp no)
 		(fields_autoplaced yes)
-		(property "Reference" "U7"
+		(property "Reference" "U8"
 			(at 203.2 53.34 0)
 			(show_name no)
@@
 			(project "cm4-robo-controller"
 				(path "/c1285fbe-5f56-49a8-9041-410713cbe619/3cc0f123-2315-4414-aa85-3a1a0bb694eb/2c385700-431a-4a3a-8a9d-f3682fa19093"
-					(reference "U7")
+					(reference "U8")
 					(unit 1)
 				)
@@
 		(in_pos_files yes)
 		(dnp no)
-		(property "Reference" "R16"
+		(property "Reference" "R18"
 			(at 60.198 44.704 0)
 			(show_name no)
@@
 			(project "cm4-robo-controller"
 				(path "/c1285fbe-5f56-49a8-9041-410713cbe619/3cc0f123-2315-4414-aa85-3a1a0bb694eb/2c385700-431a-4a3a-8a9d-f3682fa19093"
-					(reference "R16")
+					(reference "R18")
 					(unit 1)
 				)

Commit message: IPC footprint renaming, battery sim added
Parts:
- C23: footprint MyParts:C0402 -> MyPartsIPC:CAPC1005X55N
- R18, R19: footprint MyParts:R0402 -> MyPartsIPC:RESC1005X40N
- U8, U9: footprint MyParts:USON-10_L2.5-W1.0-P0.50-BL -> MyPartsIPC:SON50P100X250X60-10N
Changed lines of the file:
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@@
 			)
 		)
-		(property "Footprint" "MyParts:R0402"
+		(property "Footprint" "MyPartsIPC:RESC1005X40N"
 			(at 102.87 38.1 0)
 			(hide yes)
@@
 			)
 		)
-		(property "Footprint" "MyParts:USON-10_L2.5-W1.0-P0.50-BL"
+		(property "Footprint" "MyPartsIPC:SON50P100X250X60-10N"
 			(at 203.2 109.22 0)
 			(hide yes)
@@
 			)
 		)
-		(property "Footprint" "MyParts:C0402"
+		(property "Footprint" "MyPartsIPC:CAPC1005X55N"
 			(at 49.022 116.84 90)
 			(hide yes)
@@
 			)
 		)
-		(property "Footprint" "MyParts:USON-10_L2.5-W1.0-P0.50-BL"
+		(property "Footprint" "MyPartsIPC:SON50P100X250X60-10N"
 			(at 203.2 78.74 0)
 			(hide yes)
@@
 			)
 		)
-		(property "Footprint" "MyParts:R0402"
+		(property "Footprint" "MyPartsIPC:RESC1005X40N"
 			(at 62.23 39.37 0)
 			(hide yes)
