File: kicad/robo.kicad_sch (KiCad schematic)
At the start: 34 parts, among them J10 KF2EDGR-2.54-2P, J4 KF7620-7.62-2P, J5 KF7620-7.62-2P, J6 KF2EDGR-2.54-4P, J7 KF2EDGR-2.54-3P, J8 KF2EDGR-2.54-2P, J9 KF2EDGR-2.54-2P

Commit message: Still refining
Parts:
- A1: Pkg Type (none) -> THT Module
- C102, C103, C104, C105, C106, C107, D44, D45, D46, D47, D48, D49, R117, R118, R119, R120, R121, R122, R123, R124, R125, R126, R127, R128, R129, R130: Pkg Type (none) -> SMD 0402
- J10, J8, J9: Pkg Type (none) -> THT Terminal block 1x2 P2.54
- J4, J5: Pkg Type (none) -> THT Terminal block 1x2 P7.62
- J6: Pkg Type (none) -> THT Terminal block 1x4 P2.54
- J7: Pkg Type (none) -> THT Terminal block 1x3 P2.54
Connections:
- net GND renamed PGND

Commit message: Mods
Parts:
- added C113: 100nF, MyParts:C0402, symbol MyParts:CL05B104KO5NNNC_ALT
- added D57: SMF6.0A, PCM_JLCPCB:D_SOD-123FL, symbol MyParts:SMF6.0A
- added D58: SMF5.0A, PCM_JLCPCB:D_SOD-123FL, symbol MyParts:SMF5.0A
- added F3: nSMD010, MyParts:F1206, symbol MyParts:nSMD010
- added U21: 74LVC1G17SE-7, MyParts:SC-88A_L2.0-W1.3-P0.65-LS2.1-BL, symbol MyParts:74LVC1G17SE-7
- D44, D45, D46, D47, D48, D49: value TPESD0402G05V -> TPESD0402G12V; symbol MyParts:TPESD0402G05V -> MyParts:TPESD0402G12V; LCSC Part C558615 -> C558617; MPN TPESD0402G05V -> TPESD0402G12V
Connections:
- net 3V3_CM4: now also C113.1, F3.1, U21.5 (VCC); no longer J7.1
- net PGND: now also D57.2, D58.2
- net RC_5V: now also D57.1
- net ROBO_RX_MCU: now also U21.4 (Y); no longer R118.1
- net V_BAT renamed V_MOTOR
- new net AZ_ENC_3V3: D58.1, F3.2, J7.1
- new net GND: C113.2, U21.3 (GND)
- new net ROBO_S2_TX: R118.1, U21.2 (A)
- no-connect marks 5 -> 6
Other:
- note added: "A1 TX buffer (no CM4 back-power)"
- note added: "EMC: run motor leads in shielded cable, shield clamped 360 deg to the enclosure at the gland (not to J4/J5). Clip-on CM ferrite per pair at entry; 100 nF brush caps at the motors. Keep motor leads away from GNSS/encoder wiring."
- note added: "J7 (azimuth encoder, field-wired) is fed from 3V3_CM4 via F3 (100 mA PTC, 60 V) with D58 (SMF5.0A) clamping the J7 side. Reverse polarity, or a supply above ~6.4 V, makes D58 conduct and trips F3, so it cannot reach 3V3_CM4. Residual: a 5 V miswire is not clamped. Place F3 and D58 at J7. AS5600 draws ~7 mA."
- note added: "J7 3.3 V feed protection"
- note added: "RC_5V budget: <= 800 mA (BEC). Load: ~5 mA pull-ups + sensor."
- note added: "U21 isolates A1 S2 TX from CM4 GPIO13 (ROBO_RX_MCU). A1 runs from the battery while the CM4 can be off (SW3 open, GLOBAL_EN power cycle). A1 TX idles at 3.3 V; via R118 alone it would back-power the CM4 through GPIO13 (abs max VREF+0.5 V). 74LVC1G17 Ioff: with 3V3_CM4 off, Y is high-Z and A takes 3.3 V. CM4 TX -> A1 RX needs none: A1 is always on when the CM4 is."

Commit message: Ready to start layout
Parts:
- renumbered C102 to C57, C105 to C58, C103 to C59, C106 to C60, C107 to C61, C104 to C62, C113 to C63, D44 to D16, D47 to D17, D45 to D18, D48 to D19, D49 to D20, D57 to D21, D46 to D22, D58 to D23, J8 to J10, J4 to J11, J9 to J12, J10 to J13, J5 to J14, J6 to J8, J7 to J9, R118 to R45, R117 to R46, R119 to R47, R128 to R48, R120 to R49, R125 to R50, R121 to R51, R129 to R52, R122 to R53, R126 to R54, R130 to R55, R127 to R56, R123 to R57, R124 to R58, U21 to U16
Other:
- note added: "EMC: run motor leads in shielded cable, shield clamped 360 deg to the enclosure at the gland (not to J11/J14). Clip-on CM ferrite per pair at entry; 100 nF brush caps at the motors. Keep motor leads away from GNSS/encoder wiring."
- note added: "J11 = Firgelli motor (elevation): 1 BLUE (+) 2 BROWN (-) Swap to reverse, or invert M1 in Motion Studio."
- note added: "J9 (azimuth encoder, field-wired) is fed from 3V3_CM4 via F3 (100 mA PTC, 60 V) with D23 (SMF5.0A) clamping the J9 side. Reverse polarity, or a supply above ~6.4 V, makes D23 conduct and trips F3, so it cannot reach 3V3_CM4. Residual: a 5 V miswire is not clamped. Place F3 and D23 at J9. AS5600 draws ~7 mA."
- note added: "J9 3.3 V feed protection"
- note added: "U16 isolates A1 S2 TX from CM4 GPIO13 (ROBO_RX_MCU). A1 runs from the battery while the CM4 can be off (SW1 open, GLOBAL_EN power cycle). A1 TX idles at 3.3 V; via R45 alone it would back-power the CM4 through GPIO13 (abs max VREF+0.5 V). 74LVC1G17 Ioff: with 3V3_CM4 off, Y is high-Z and A takes 3.3 V. CM4 TX -> A1 RX needs none: A1 is always on when the CM4 is."
- note removed: "EMC: run motor leads in shielded cable, shield clamped 360 deg to the enclosure at the gland (not to J4/J5). Clip-on CM ferrite per pair at entry; 100 nF brush caps at the motors. Keep motor leads away from GNSS/encoder wiring."
- note removed: "J4 = Firgelli motor (elevation): 1 BLUE (+) 2 BROWN (-) Swap to reverse, or invert M1 in Motion Studio."
- note removed: "J7 (azimuth encoder, field-wired) is fed from 3V3_CM4 via F3 (100 mA PTC, 60 V) with D58 (SMF5.0A) clamping the J7 side. Reverse polarity, or a supply above ~6.4 V, makes D58 conduct and trips F3, so it cannot reach 3V3_CM4. Residual: a 5 V miswire is not clamped. Place F3 and D58 at J7. AS5600 draws ~7 mA."
- note removed: "J7 3.3 V feed protection"
- note removed: "U21 isolates A1 S2 TX from CM4 GPIO13 (ROBO_RX_MCU). A1 runs from the battery while the CM4 can be off (SW3 open, GLOBAL_EN power cycle). A1 TX idles at 3.3 V; via R118 alone it would back-power the CM4 through GPIO13 (abs max VREF+0.5 V). 74LVC1G17 Ioff: with 3V3_CM4 off, Y is high-Z and A takes 3.3 V. CM4 TX -> A1 RX needs none: A1 is always on when the CM4 is."

Commit message: Added new sheets, motor notes
Parts:
- added J15: PM254-2-12-Z-8.5, MyParts:HDR-F-TH_2x12-P2.54-H8.5_PM254_NOPADS, symbol MyParts:PM254-2-12-Z-8.5
- added J16: PM254-2-09-Z-8.5, MyParts:HDR-F-TH_2x09-P2.54-H8.5_PM254_NOPADS, symbol MyParts:PM254-2-09-Z-8.5
- R57: value 10kΩ -> 68kΩ; symbol MyParts:0402WGF1002TCE -> MyParts:0402WGF6802TCE; LCSC Part C25744 -> C36871; MPN 0402WGF1002TCE -> 0402WGF6802TCE
- R58: value 15kΩ -> 100kΩ; symbol MyParts:0402WGF1502TCE -> MyParts:0402WGF1003TCE; LCSC Part C25756 -> C25741; MPN 0402WGF1502TCE -> 0402WGF1003TCE
Other:
- note added: "Sockets for A1 (RoboClaw plugs in)"

Commit message: IPC footprint renaming, battery sim added
Parts:
- C57, C58, C59, C60, C61, C62, C63: footprint MyParts:C0402 -> MyPartsIPC:CAPC1005X55N
- D16, D17, D18, D19, D20, D22: footprint MyParts:D0402-BI -> MyPartsIPC:DIOC1005X55N
- D21, D23: footprint PCM_JLCPCB:D_SOD-123FL -> MyPartsIPC:SODFL3718X110N
- F3: value nSMD010 -> 100mA; footprint MyParts:F1206 -> MyPartsIPC:FUSC3216X110N
- R45, R46, R47, R48, R49, R50, R51, R52, R53, R54, R55, R56, R57, R58: footprint MyParts:R0402 -> MyPartsIPC:RESC1005X40N
- U16: footprint MyParts:SC-88A_L2.0-W1.3-P0.65-LS2.1-BL -> MyPartsIPC:SOT65P210X110-5N
Changed lines of the file:
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@@
 			)
 		)
-		(property "Footprint" "MyParts:D0402-BI"
+		(property "Footprint" "MyPartsIPC:DIOC1005X55N"
 			(at 158.75 81.28 0)
 			(hide yes)
@@
 			)
 		)
-		(property "Footprint" "MyParts:R0402"
+		(property "Footprint" "MyPartsIPC:RESC1005X40N"
 			(at 171.45 114.3 0)
 			(hide yes)
@@
 			)
 		)
-		(property "Footprint" "MyParts:R0402"
+		(property "Footprint" "MyPartsIPC:RESC1005X40N"
 			(at 231.14 95.25 0)
 			(hide yes)
@@
 			)
 		)
-		(property "Footprint" "MyParts:R0402"
+		(property "Footprint" "MyPartsIPC:RESC1005X40N"
 			(at 241.3 99.06 0)
 			(hide yes)
@@
 			)
 		)
-		(property "Footprint" "MyParts:R0402"
+		(property "Footprint" "MyPartsIPC:RESC1005X40N"
 			(at 158.75 72.39 0)
 			(hide yes)
@@
 			)
 		)
-		(property "Footprint" "MyParts:R0402"
+		(property "Footprint" "MyPartsIPC:RESC1005X40N"
 			(at 168.91 53.34 0)
 			(hide yes)
@@
 			)
 		)
-		(property "Footprint" "MyParts:C0402"
+		(property "Footprint" "MyPartsIPC:CAPC1005X55N"
 			(at 269.24 146.05 0)
 			(hide yes)
@@
 			)
 		)
-		(property "Footprint" "MyParts:R0402"
+		(property "Footprint" "MyPartsIPC:RESC1005X40N"
 			(at 158.75 49.53 0)
 			(hide yes)
@@
 			)
 		)
-		(property "Footprint" "MyParts:C0402"
+		(property "Footprint" "MyPartsIPC:CAPC1005X55N"
 			(at 176.53 81.28 0)
 			(hide yes)
@@
 			)
 		)
-		(property "Footprint" "MyParts:C0402"
+		(property "Footprint" "MyPartsIPC:CAPC1005X55N"
 			(at 176.53 58.42 0)
 			(hide yes)
@@
 			)
 		)
-		(property "Footprint" "MyParts:R0402"
+		(property "Footprint" "MyPartsIPC:RESC1005X40N"
 			(at 168.91 76.2 0)
 			(hide yes)
@@
 			)
 		)
-		(property "Footprint" "MyParts:D0402-BI"
+		(property "Footprint" "MyPartsIPC:DIOC1005X55N"
 			(at 158.75 58.42 0)
 			(hide yes)
@@
 			)
 		)
-		(property "Footprint" "MyParts:R0402"
+		(property "Footprint" "MyPartsIPC:RESC1005X40N"
 			(at 59.69 49.53 0)
 			(hide yes)
@@
 			)
 		)
-		(property "Footprint" "PCM_JLCPCB:D_SOD-123FL"
+		(property "Footprint" "MyPartsIPC:SODFL3718X110N"
 			(at 152.4 140.97 0)
 			(hide yes)
@@
 			)
 		)
-		(property "Footprint" "MyParts:C0402"
+		(property "Footprint" "MyPartsIPC:CAPC1005X55N"
 			(at 248.92 58.42 0)
 			(hide yes)
@@
 			)
 		)
-		(property "Footprint" "MyParts:C0402"
+		(property "Footprint" "MyPartsIPC:CAPC1005X55N"
 			(at 176.53 114.3 0)
 			(hide yes)
@@
 			)
 		)
-		(property "Footprint" "MyParts:R0402"
+		(property "Footprint" "MyPartsIPC:RESC1005X40N"
 			(at 231.14 49.53 0)
 			(hide yes)
@@
 			)
 		)
-		(property "Footprint" "MyParts:D0402-BI"
+		(property "Footprint" "MyPartsIPC:DIOC1005X55N"
 			(at 231.14 81.28 0)
 			(hide yes)
@@
 			)
 		)
-		(property "Footprint" "PCM_JLCPCB:D_SOD-123FL"
+		(property "Footprint" "MyPartsIPC:SODFL3718X110N"
 			(at 27.94 114.3 0)
 			(hide yes)
@@
 			)
 		)
-		(property "Value" "nSMD010"
+		(property "Value" "100mA"
 			(at 138.43 139.7 0)
 			(show_name no)
@@
 			)
 		)
-		(property "Footprint" "MyParts:F1206"
+		(property "Footprint" "MyPartsIPC:FUSC3216X110N"
 			(at 138.43 135.89 0)
 			(hide yes)
@@
 			)
 		)
-		(property "Footprint" "MyParts:C0402"
+		(property "Footprint" "MyPartsIPC:CAPC1005X55N"
 			(at 248.92 104.14 0)
 			(hide yes)
@@
 			)
 		)
-		(property "Footprint" "MyParts:SC-88A_L2.0-W1.3-P0.65-LS2.1-BL"
+		(property "Footprint" "MyPartsIPC:SOT65P210X110-5N"
 			(at 220.98 138.43 0)
 			(hide yes)
@@
 			)
 		)
-		(property "Footprint" "MyParts:R0402"
+		(property "Footprint" "MyPartsIPC:RESC1005X40N"
 			(at 49.53 52.07 0)
 			(hide yes)
@@
 			)
 		)
-		(property "Footprint" "MyParts:R0402"
+		(property "Footprint" "MyPartsIPC:RESC1005X40N"
 			(at 241.3 53.34 0)
 			(hide yes)
@@
 			)
 		)
-		(property "Footprint" "MyParts:R0402"
+		(property "Footprint" "MyPartsIPC:RESC1005X40N"
 			(at 241.3 76.2 0)
 			(hide yes)
@@
 			)
 		)
-		(property "Footprint" "MyParts:R0402"
+		(property "Footprint" "MyPartsIPC:RESC1005X40N"
 			(at 231.14 72.39 0)
 			(hide yes)
@@
 			)
 		)
-		(property "Footprint" "MyParts:D0402-BI"
+		(property "Footprint" "MyPartsIPC:DIOC1005X55N"
 			(at 153.67 115.57 0)
 			(hide yes)
@@
 			)
 		)
-		(property "Footprint" "MyParts:D0402-BI"
+		(property "Footprint" "MyPartsIPC:DIOC1005X55N"
 			(at 231.14 58.42 0)
 			(hide yes)
@@
 			)
 		)
-		(property "Footprint" "MyParts:C0402"
+		(property "Footprint" "MyPartsIPC:CAPC1005X55N"
 			(at 248.92 81.28 0)
 			(hide yes)
@@
 			)
 		)
-		(property "Footprint" "MyParts:R0402"
+		(property "Footprint" "MyPartsIPC:RESC1005X40N"
 			(at 163.83 110.49 0)
 			(hide yes)
@@
 			)
 		)
-		(property "Footprint" "MyParts:D0402-BI"
+		(property "Footprint" "MyPartsIPC:DIOC1005X55N"
 			(at 231.14 104.14 0)
 			(hide yes)

Commit message: Updates after latest Tomachie review
Parts:
- added C80: 1uF, MyPartsIPC:CAPC1608X95N, symbol MyParts:CL10A105KA8NNNC
- added C81: 10uF, MyPartsIPC:CAPC1608X95N, symbol MyParts:CL10A106MA8NRNC
- added C83: 100nF, MyPartsIPC:CAPC1005X55N, symbol MyParts:CL05B104KO5NNNC_ALT
- added U18: TPS70933DBVR, MyPartsIPC:SOT95P280X145-5N, symbol MyParts:TPS70933DBVR
- added U19: 74LVC1G17SE-7, MyPartsIPC:SOT65P210X110-5N, symbol MyParts:74LVC1G17SE-7
Connections:
- net 3V3_CM4: now also C83.1, U19.5 (VCC); no longer F3.1
- net GND: now also C83.2, U19.3 (GND)
- net PGND: now also C80.1, C81.2, U18.2 (GND)
- net RC_5V: now also C80.2, U18.1 (IN)
- net ROBO_TX_MCU: now also U19.2 (A); no longer R46.1
- new net: C81.1, F3.1, U18.5 (OUT)
- new net ROBO_S1_RX: R46.1, U19.4 (Y)
- no-connect marks 6 -> 8
Other:
- note added: "A1 RX buffer (no CM4 back-power)"
- note added: "J9 (azimuth encoder, field-wired) has its own 3.3 V LDO, U18 (TPS70933, 30 V max, from RC_5V), not 3V3_CM4, so a miswired supply on J9 cannot back-feed the CM4 or the GPS. U18 blocks reverse current, so it cannot reach RC_5V either. EN is left open (internal pull-up; never tie EN to IN). F3 (100 mA PTC) limits a shorted cable, D23 (SMF5.0A) clamps J9. C81 >= 1.5 uF effective."
- note added: "J9 3.3 V sensor supply (U18)"
- note added: "U16 isolates A1 S2 TX from CM4 GPIO13 (ROBO_RX_MCU); U19 (below the J9 box) isolates CM4 GPIO12 (ROBO_TX_MCU) from A1 S1 RX and its pull-up. A1 runs from the battery while the CM4 can be off (SW1 open, GLOBAL_EN power cycle). Wired direct, A1 would back-power the CM4 through GPIO13 or GPIO12 (abs max VREF+0.5 V). Both 74LVC1G17 run on 3V3_CM4; with it off, Ioff makes Y high-Z and A tolerates 3.3 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"
- note removed: "J9 (azimuth encoder, field-wired) is fed from 3V3_CM4 via F3 (100 mA PTC, 60 V) with D23 (SMF5.0A) clamping the J9 side. Reverse polarity, or a supply above ~6.4 V, makes D23 conduct and trips F3, so it cannot reach 3V3_CM4. Residual: a 5 V miswire is not clamped. Place F3 and D23 at J9. AS5600 draws ~7 mA."
- note removed: "J9 3.3 V feed protection"
- note removed: "U16 isolates A1 S2 TX from CM4 GPIO13 (ROBO_RX_MCU). A1 runs from the battery while the CM4 can be off (SW1 open, GLOBAL_EN power cycle). A1 TX idles at 3.3 V; via R45 alone it would back-power the CM4 through GPIO13 (abs max VREF+0.5 V). 74LVC1G17 Ioff: with 3V3_CM4 off, Y is high-Z and A takes 3.3 V. CM4 TX -> A1 RX needs none: A1 is always on when the CM4 is."
- moved on the sheet: D23, F3

Commit message: PCB rework: rotate RoboClaw, battery input at top, planes redrawn, right half routed
- A1 rotated 90 CW and moved down; J14/J11 motor pours straight to the A1 pins
- J14 pins swapped (M2 polarity) in the schematic; J14 moved clear of D1
- Battery input, fuses and TVS diodes along the top edge; NT1 at J1-
- In1 (GND/PGND) and In2 (5V/V_MOTOR) split redrawn for the new layout
- Power block re-routed; 12V fed to the buck input on B.Cu
- UART buffers back on logic GND; RoboClaw signal section routed
Connections:
- net M2A: now also J14.2; no longer J14.1
- net M2B: now also J14.1; no longer J14.2
Changed lines of the file:
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@@
 		)
 	)
-	(label "M2A"
+	(label "M2B"
 		(at 80.01 162.56 180)
 		(effects
@@
 		)
 	)
-	(label "M2B"
+	(label "M2A"
 		(at 80.01 165.1 180)
 		(effects

Commit message: Added notes
Parts:
- D23: value SMF5.0A -> SMBJ3V3; footprint MyPartsIPC:SODFL3718X110N -> MyPartsIPC:DIOM5436X244N; symbol MyParts:SMF5.0A -> MyParts:SMBJ3V3; LCSC Part C19077497 -> C82082; MPN SMF5.0A -> SMBJ3V3-E3/52; Manufacturer hongjiacheng -> Vishay; Pkg Type SMD SOD-123FL -> SMD SMB (DO-214AA)
Connections:
- net AZ_ENC_3V3: no longer D23.1
- net at C81.1, F3.1, U18.5 (OUT): now also D23.1
Other:
- note added: "D23: Vishay SMBJ3V3-E3/52, 600 W SMB TVS. VBR >= 4.1 V, VC 7.3 V @ 50 A, IR <= 200 uA. Holds U18 OUT (7 V abs max) on a J9 miswire until F3 trips. Not a generic SMBJ3.3A: some break down at 6.5 V."
- note added: "J9 (azimuth encoder, field-wired) has its own 3.3 V LDO, U18 (TPS70933, 30 V max, from RC_5V), not 3V3_CM4, so a miswired supply on J9 cannot back-feed the CM4 or the GPS. U18 blocks reverse current, so it cannot reach RC_5V either. EN is left open (internal pull-up; never tie EN to IN). F3 (100 mA PTC) sits between J9 and D23 (SMBJ3V3); F3 limits a shorted cable or a miswire onto J9 while D23 cl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"
- note removed: "J9 (azimuth encoder, field-wired) has its own 3.3 V LDO, U18 (TPS70933, 30 V max, from RC_5V), not 3V3_CM4, so a miswired supply on J9 cannot back-feed the CM4 or the GPS. U18 blocks reverse current, so it cannot reach RC_5V either. EN is left open (internal pull-up; never tie EN to IN). F3 (100 mA PTC) limits a shorted cable, D23 (SMF5.0A) clamps J9. C81 >= 1.5 uF effective."
- moved on the sheet: D23, F3
Changed lines of the file:
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@@
 		)
 	)
-	(text "J9 (azimuth encoder, field-wired) has its own 3.3 V LDO, U18 (TPS70933, 30 V max, from RC_5V),\nnot 3V3_CM4, so a miswired supply on J9 cannot back-feed the CM4 or the GPS. U18 blocks reverse\ncurrent, so it cannot reach RC_5V either. EN is left open (internal pull-up; never tie EN to IN).\nF3 (100 mA PTC) limits a shorted cable, D23 (SMF5.0A) clamps J9. C81 >= 1.5 uF effective."
+	(text "J9 (azimuth encoder, field-wired) has its own 3.3 V LDO, U18 (TPS70933, 30 V max, from RC_5V),\nnot 3V3_CM4, so a miswired supply on J9 cannot back-feed the CM4 or the GPS. U18 blocks reverse\ncurrent, so it cannot reach RC_5V either. EN is left open (internal pull-up; never tie EN to IN).\nF3 (100 mA PTC) sits between J9 and D23 (SMBJ3V3); F3 limits a shorted cable or a miswire\nonto J9 while D23 clamps U18 OUT (7 V abs max). C81 >= 1.5 uF effective."
 		(exclude_from_sim no)
-		(at 115.062 151.765 0)
+		(at 115.062 153.67 0)
 		(effects
 			(font
@@
 		)
 	)
+	(text "D23: Vishay SMBJ3V3-E3/52, 600 W\nSMB TVS. VBR >= 4.1 V, VC 7.3 V\n@ 50 A, IR <= 200 uA. Holds U18 OUT\n(7 V abs max) on a J9 miswire until\nF3 trips. Not a generic SMBJ3.3A:\nsome break down at 6.5 V."
+		(exclude_from_sim no)
+		(at 166.37 141.605 0)
+		(effects
+			(font
+				(size 1.016 1.016)
+			)
+			(justify left top)
+		)
+	)
 	(text "EMC: run motor leads in shielded cable, shield\nclamped 360 deg to the enclosure at the gland\n(not to J11/J14). Clip-on CM ferrite per pair at\nentry; 100 nF brush caps at the motors. Keep\nmotor leads away from GNSS/encoder wiring."
 		(exclude_from_sim no)
@@
 	)
 	(junction
-		(at 171.45 110.49)
+		(at 154.94 137.16)
 		(diameter 0)
 		(color 0 0 0 0)
 	)
 	(junction
-		(at 231.14 53.34)
+		(at 171.45 110.49)
 		(diameter 0)
 		(color 0 0 0 0)
 	)
 	(junction
-		(at 248.92 99.06)
+		(at 231.14 53.34)
 		(diameter 0)
 		(color 0 0 0 0)
 	)
 	(junction
-		(at 175.26 137.16)
+		(at 248.92 99.06)
 		(diameter 0)
 		(color 0 0 0 0)
@@
 	(wire
 		(pts
-			(xy 147.32 137.16) (xy 152.4 137.16)
+			(xy 147.32 137.16) (xy 160.02 137.16)
 		)
 		(stroke
@@
 	(wire
 		(pts
-			(xy 170.18 137.16) (xy 182.88 137.16)
+			(xy 177.8 137.16) (xy 182.88 137.16)
 		)
 		(stroke
@@
 	)
 	(symbol
-		(lib_id "MyParts:SMF5.0A")
-		(at 175.26 140.97 180)
+		(lib_id "MyParts:SMBJ3V3")
+		(at 154.94 140.97 180)
 		(unit 1)
 		(body_style 1)
@@
 		(dnp no)
 		(property "Reference" "D23"
-			(at 177.8 139.7 0)
+			(at 157.48 139.7 0)
 			(show_name no)
 			(do_not_autoplace no)
@@
 			)
 		)
-		(property "Value" "SMF5.0A"
-			(at 177.8 142.24 0)
+		(property "Value" "SMBJ3V3"
+			(at 157.48 142.24 0)
 			(show_name no)
 			(do_not_autoplace no)
@@
 			)
 		)
-		(property "Footprint" "MyPartsIPC:SODFL3718X110N"
-			(at 175.26 140.97 0)
+		(property "Footprint" "MyPartsIPC:DIOM5436X244N"
+			(at 154.94 140.97 0)
 			(hide yes)
 			(show_name no)
@@
 			)
 		)
-		(property "Datasheet" "${MYPARTS_DATASHEETS}/SMF5.0A.pdf"
-			(at 175.26 140.97 0)
+		(property "Datasheet" "${MYPARTS_DATASHEETS}/SMBJ3V3.pdf"
+			(at 154.94 140.97 0)
 			(hide yes)
 			(show_name no)
@@
 			)
 		)
-		(property "Description" "-55℃~+150℃ 1 200W@10/1000us 21.7A@10/1000us 400uA 5V 7V 9.2V IEC 61000-4-2 TVS Unidirectional SOD-123FL ESD and Surge Protection (TVS/ESD) ROHS"
-			(at 175.26 140.97 0)
+		(property "Description" "-55℃~+175℃ 1 600W@10/1000us 50A@10/1000us 200uA 3.3V 4.1V 7.3V TVS Unidirectional SMB(DO-214AA) ESD and Surge Protection (TVS/ESD) ROHS"
+			(at 154.94 140.97 0)
 			(hide yes)
 			(show_name no)
@@
 			)
 		)
-		(property "Manufacturer" "hongjiacheng"
-			(at 175.26 140.97 0)
+		(property "Manufacturer" "Vishay"
+			(at 154.94 140.97 0)
 			(hide yes)
 			(show_name no)
@@
 		)
 		(property "ki_keywords" ""
-			(at 175.26 140.97 0)
+			(at 154.94 140.97 0)
 			(hide yes)
 			(show_name no)
@@
 		)
 		(property "ki_fp_filters" "D_*"
-			(at 175.26 140.97 0)
+			(at 154.94 140.97 0)
 			(hide yes)
 			(show_name no)
@@
 			)
 		)
-		(property "MPN" "SMF5.0A"
-			(at 175.26 140.97 0)
+		(property "MPN" "SMBJ3V3-E3/52"
+			(at 154.94 140.97 0)
 			(hide yes)
 			(show_name no)
@@
 			)
 		)
-		(property "LCSC Part" "C19077497"
-			(at 175.26 140.97 0)
+		(property "LCSC Part" "C82082"
+			(at 154.94 140.97 0)
 			(hide yes)
 			(show_name no)
@@
 			)
 		)
-		(property "Pkg Type" "SMD SOD-123FL"
-			(at 175.26 140.97 0)
+		(property "Pkg Type" "SMD SMB (DO-214AA)"
+			(at 154.94 140.97 0)
 			(hide yes)
 			(show_name no)
@@
 	(symbol
 		(lib_id "MyParts:nSMD010")
-		(at 161.29 135.89 0)
+		(at 168.91 135.89 0)
 		(unit 1)
 		(body_style 1)
@@
 		(dnp no)
 		(property "Reference" "F3"
-			(at 161.29 132.08 0)
+			(at 168.91 132.08 0)
 			(show_name no)
 			(do_not_autoplace no)
@@
 		)
 		(property "Value" "100mA"
-			(at 161.29 139.7 0)
+			(at 168.91 139.7 0)
 			(show_name no)
 			(do_not_autoplace yes)
@@
 		)
 		(property "Footprint" "MyPartsIPC:FUSC3216X110N"
-			(at 161.29 135.89 0)
+			(at 168.91 135.89 0)
 			(hide yes)
 			(show_name no)
@@
 		)
 		(property "Datasheet" "${MYPARTS_DATASHEETS}/nSMD010.pdf"
-			(at 161.29 135.89 0)
+			(at 168.91 135.89 0)
 			(hide yes)
 			(show_name no)
@@
 		)
 		(property "Description" "PTC resettable fuse 100mA hold 250mA trip 60V 1206, 1.6 ohm initial"
-			(at 161.29 135.89 0)
+			(at 168.91 135.89 0)
 			(hide yes)
 			(show_name no)
@@
 		)
 		(property "Manufacturer" "TECHFUSE"
-			(at 161.29 135.89 0)
+			(at 168.91 135.89 0)
 			(hide yes)
 			(show_name no)
@@
 		)
 		(property "MPN" "nSMD010"
-			(at 161.29 135.89 0)
+			(at 168.91 135.89 0)
 			(hide yes)
 			(show_name no)
@@
 		)
 		(property "LCSC Part" "C70065"
-			(at 161.29 135.89 0)
+			(at 168.91 135.89 0)
 			(hide yes)
 			(show_name no)
@@
 		)
 		(property "Pkg Type" "SMD 1206"
-			(at 161.29 135.89 0)
+			(at 168.91 135.89 0)
 			(hide yes)
 			(show_name no)
@@
 	(symbol
 		(lib_id "power:GNDPWR")
-		(at 175.26 144.78 0)
+		(at 154.94 144.78 0)
 		(unit 1)
 		(body_style 1)
@@
 		(dnp no)
 		(property "Reference" "#PWR0456"
-			(at 175.26 151.13 0)
+			(at 154.94 151.13 0)
 			(hide yes)
 			(show_name no)
@@
 		)
 		(property "Value" "PGND"
-			(at 175.26 148.59 0)
+			(at 154.94 148.59 0)
 			(hide yes)
 			(show_name no)
@@
 		)
 		(property "Footprint" ""
-			(at 175.26 144.78 0)
+			(at 154.94 144.78 0)
 			(hide yes)
 			(show_name no)
@@
 		)
 		(property "Datasheet" ""
-			(at 175.26 144.78 0)
+			(at 154.94 144.78 0)
 			(hide yes)
 			(show_name no)
@@
 		)
 		(property "Description" "Power symbol creates a global label with name \"GNDPWR\" , global ground"
-			(at 175.26 144.78 0)
+			(at 154.94 144.78 0)
 			(hide yes)
 			(show_name no)
