File: kicad/cm4_connectors.kicad_sch (KiCad schematic)
At the start: 9 parts, among them J3 Header-Male-2.54_2x3, J4 2541WV-2X12P, J5 Header-Male-2.54_1x3, J6 Header-Male-2.54_2x3, U10 74LVC1G07SE-7

Commit message: IPC footprint renaming, battery sim added
Parts:
- R20, R21: footprint MyParts:R0402 -> MyPartsIPC:RESC1005X40N
- U10: footprint MyParts:SC-88A_L2.0-W1.3-P0.65-LS2.1-BL -> MyPartsIPC:SOT65P210X110-5N
Other:
- note added: "I2C PULL-UPS I2C1: GPIO2 = I2C1_SDA (J4-16), GPIO3 = I2C1_SCL (J4-18) Pulled up to 3.3 V (GPIO_VREF) by 1.8 kΩ inside the CM4 (CM4 datasheet section 2.5, pins 56/58). No board pull-ups are needed. R20/R21 (2.2k, fitted via H5/H6) are optional. I2C0: GPIO0 = ID_SD (J4-22), GPIO1 = ID_SC (J4-23) No I2C pull-ups on the CM4, only the BCM2711's weak reset pull-ups (33-73 kΩ). If J4-22/23 are used as a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"
Changed lines of the file:
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@@
 			)
 		)
-		(property "Footprint" "MyParts:R0402"
+		(property "Footprint" "MyPartsIPC:RESC1005X40N"
 			(at 134.62 171.45 0)
 			(hide yes)
@@
 			)
 		)
-		(property "Footprint" "MyParts:SC-88A_L2.0-W1.3-P0.65-LS2.1-BL"
+		(property "Footprint" "MyPartsIPC:SOT65P210X110-5N"
 			(at 137.16 64.77 0)
 			(hide yes)
@@
 			)
 		)
-		(property "Footprint" "MyParts:R0402"
+		(property "Footprint" "MyPartsIPC:RESC1005X40N"
 			(at 158.75 171.45 0)
 			(hide yes)
@@
 		)
 	)
+	(text "I2C PULL-UPS\nI2C1: GPIO2 = I2C1_SDA (J4-16), GPIO3 = I2C1_SCL (J4-18)\nPulled up to 3.3 V (GPIO_VREF) by 1.8 kΩ inside the CM4\n(CM4 datasheet section 2.5, pins 56/58). No board pull-ups\nare needed. R20/R21 (2.2k, fitted via H5/H6) are optional.\n\nI2C0: GPIO0 = ID_SD (J4-22), GPIO1 = ID_SC (J4-23)\nNo I2C pull-ups on the CM4, only the BCM2711's weak reset\npull-ups (33-73 kΩ). If J4-22/23 are used as an I2C bus, the\ndevice on J4 must supply the pull-ups (2.2k-4.7k to 3.3 V)."
+		(exclude_from_sim no)
+		(at 220.98 129.54 0)
+		(effects
+			(font
+				(size 1.016 1.016)
+			)
+			(justify left top)
+		)
+	)

Commit message: PCB: decoupling caps at IC supply pins, route GPS area
- Add 100nF decoupling for U10 (C84) and U17 (C85)
- Move C15, C18, C21, C25, C27, C32 next to their IC supply pins; shift R10
- Route the GPS section: RF_IN, antenna bias, GPS VCC, V_BCKP, local signals, GND/5V plane vias
Parts:
- added C84: 100nF, MyPartsIPC:CAPC1005X55N, symbol MyParts:CL05B104KO5NNNC_ALT
Connections:
- net 3V3_CM4: now also C84.1
- net GND: now also C84.2

Commit message: PCB: swap GPS and USB areas, drop J2 and hub ports 3/4, remap J4
- Remove expansion header J2 with C22, U7, D9 and D7; disable USB2514B
  ports 3 and 4 with 10k pull-ups (R94-R97) on their D-/D+ straps.
- Remap J4 GPIO pins so they route to the CM4 connector without
  crossovers (schematic labels, notes and PCB pad nets).
- Add decoupling caps C84 (U10) and C85 (U17); add HUB_CTRL net class.
- Move USB (USB1, USBC1, hub) to the top edge and GPS (U12, CN1, J7) to
  the bottom-left; R4/R5 move with the GPS group. First-pass placement,
  all USB and GPS copper removed for manual routing.
- Relabel bottom-edge silk text for the SMA connectors.
- README and usb-power sim note updated for the two-port hub.
Connections:
- net 3V3_CM4: now also J4.5; no longer J4.7
- net 5V: now also J4.7; no longer J4.5
- net GPIO0: now also J4.13; no longer J4.22
- net GPIO1: now also J4.10; no longer J4.23
- net GPIO17: now also J4.20; no longer J4.9
- net GPIO18: now also J4.18; no longer J4.11
- net GPIO19: now also J4.11; no longer J4.13
- net GPIO20: now also J4.8; no longer J4.15
- net GPIO21: now also J4.6; no longer J4.17
- net GPIO22: now also J4.21; no longer J4.24
- net GPIO23: now also J4.16; no longer J4.19
- net GPIO26: now also J4.9; no longer J4.20
- net GPIO27: now also J4.23; no longer J4.21
- net I2C1_SCL: now also J4.22; no longer J4.18
- net I2C1_SDA: now also J4.24; no longer J4.16
- net SPI0_CE0: now also J4.14; no longer J4.12
- net SPI0_CE1: now also J4.12; no longer J4.14
- net SPI0_MISO: now also J4.17; no longer J4.10
- net SPI0_MOSI: now also J4.19; no longer J4.8
- net SPI0_SCLK: now also J4.15; no longer J4.6
Other:
- note added: "GPIO0 / GPIO1 (J4-13 / J4-10) CM4 pins 36 (ID_SD = GPIO0) and 35 (ID_SC = GPIO1). This is the I2C0 bus the firmware normally uses to look for a HAT EEPROM and to control CSI0/DSI0 cameras and displays. This board has no HAT, camera or display, so the pins are free for general use. To use them as GPIO, add to config.txt (CM4 datasheet section 2.10): force_eeprom_read=0 disable_poe_fan=1 Without th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"
- note added: "I2C PULL-UPS I2C1: GPIO2 = I2C1_SDA (J4-24), GPIO3 = I2C1_SCL (J4-22) Pulled up to 3.3 V (GPIO_VREF) by 1.8 kΩ inside the CM4 (CM4 datasheet section 2.5, pins 56/58). No board pull-ups are needed. R20/R21 (2.2k, fitted via H5/H6) are optional. I2C0: GPIO0 = ID_SD (J4-22), GPIO1 = ID_SC (J4-23) No I2C pull-ups on the CM4, only the BCM2711's weak reset pull-ups (33-73 kΩ). If J4-22/23 are used as a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"
- note removed: "GPIO0 / GPIO1 (J4-22 / J4-23) CM4 pins 36 (ID_SD = GPIO0) and 35 (ID_SC = GPIO1). This is the I2C0 bus the firmware normally uses to look for a HAT EEPROM and to control CSI0/DSI0 cameras and displays. This board has no HAT, camera or display, so the pins are free for general use. To use them as GPIO, add to config.txt (CM4 datasheet section 2.10): force_eeprom_read=0 disable_poe_fan=1 Without th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"
- note removed: "I2C PULL-UPS I2C1: GPIO2 = I2C1_SDA (J4-16), GPIO3 = I2C1_SCL (J4-18) Pulled up to 3.3 V (GPIO_VREF) by 1.8 kΩ inside the CM4 (CM4 datasheet section 2.5, pins 56/58). No board pull-ups are needed. R20/R21 (2.2k, fitted via H5/H6) are optional. I2C0: GPIO0 = ID_SD (J4-22), GPIO1 = ID_SC (J4-23) No I2C pull-ups on the CM4, only the BCM2711's weak reset pull-ups (33-73 kΩ). If J4-22/23 are used as a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"

Commit message: J4 outer row to GND, route SPI0 CE0/CE1, PCB review fixes
Schematic: J4 pins 6, 8, 10, 16, 18 (GPIO21, GPIO20, GPIO1, GPIO23,
GPIO18) are now GND; CM4 pins 25, 27, 35, 47, 49 get no-connect flags.
The five labels, wires and CM4_Connectors sheet pins are removed.

PCB: J4 pad nets updated to match, SPI0_CE0 and SPI0_CE1 routed to the
CM4, the 11 inner J4 nets restored.

Review fixes:
- PGND: solid zone connections on In1 for J1 pin 2 and the RoboClaw
  BAT- pins (were thermal spokes carrying the motor return).
- FUSE_IN: zone outlines widened below the fuse pads so the Q1 source
  arm is ~4 mm instead of 1.2 mm; two more 1.0 mm vias.
- HD2 pair rerouted as a coupled pair on B.Cu through the USB-A pin
  corridor; HD2_P via moved.
- Second 5V via at the U4 input.
- Pair length matching: meanders on EP0-, EP1-, EP2+, EP3-, USB_HUB_N,
  HSD2-, HD1_N; RJ45 legs end at the pin centres. All pairs within
  0.03 mm.
- RF_IN from CN1 re-routed at the 0.18 mm class width (was 1.0/0.3 mm).

Project: DRC exclusions for the silk-to-edge warnings.
Connections:
- net GPIO1 is gone; now on net GND: J4.10
- net GPIO18 is gone; now on net GND: J4.18
- net GPIO20 is gone; now on net GND: J4.8
- net GPIO21 is gone; now on net GND: J4.6
- net GPIO23 is gone; now on net GND: J4.16

Commit message: Added I2C and battery 3d file
Other:
- note added: "GPIO0 (J4-13) as plain GPIO: add to config.txt force_eeprom_read=0 disable_poe_fan=1 or the firmware probes GPIO0/1 (I2C0) for a HAT EEPROM at boot."
- note added: "I2C PULL-UPS I2C1: GPIO2 = I2C1_SDA (J4-24), GPIO3 = I2C1_SCL (J4-22) Pulled up to 3.3 V (GPIO_VREF) by 1.8 kΩ inside the CM4 (CM4 datasheet section 2.5, pins 56/58). No board pull-ups are needed. R20/R21 (2.2k, fitted via H5/H6) are optional."
- note removed: "GPIO0 / GPIO1 (J4-13 / J4-10) CM4 pins 36 (ID_SD = GPIO0) and 35 (ID_SC = GPIO1). This is the I2C0 bus the firmware normally uses to look for a HAT EEPROM and to control CSI0/DSI0 cameras and displays. This board has no HAT, camera or display, so the pins are free for general use. To use them as GPIO, add to config.txt (CM4 datasheet section 2.10): force_eeprom_read=0 disable_poe_fan=1 Without th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"
- note removed: "I2C PULL-UPS I2C1: GPIO2 = I2C1_SDA (J4-24), GPIO3 = I2C1_SCL (J4-22) Pulled up to 3.3 V (GPIO_VREF) by 1.8 kΩ inside the CM4 (CM4 datasheet section 2.5, pins 56/58). No board pull-ups are needed. R20/R21 (2.2k, fitted via H5/H6) are optional. I2C0: GPIO0 = ID_SD (J4-22), GPIO1 = ID_SC (J4-23) No I2C pull-ups on the CM4, only the BCM2711's weak reset pull-ups (33-73 kΩ). If J4-22/23 are used as a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"
Changed lines of the file:
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@@
 	(rectangle
 		(start 50.8 48.26)
-		(end 118.11 142.24)
+		(end 118.11 121.92)
 		(stroke
 			(width 0)
@@
 		)
 	)
+	(text "GPIO0 (J4-13) as plain GPIO: add to config.txt\n  force_eeprom_read=0\n  disable_poe_fan=1\nor the firmware probes GPIO0/1 (I2C0) for a HAT EEPROM at boot."
+		(exclude_from_sim no)
+		(at 60.96 112.522 0)
+		(effects
+			(font
+				(size 1.016 1.016)
+			)
+			(justify left top)
+		)
+	)
 	(text "EEPROM WRITE PROTECT (EEPROM_nWP, J3 3-4)\nThe CM4 pulls EEPROM_nWP up internally (100k), so the\nbootloader EEPROM is writable unless J3 3-4 is fitted.\nThe jumper only takes effect once protection is enabled\nin the bootloader config (CM4 datasheet 2.18).\n\nProduction:\n- Set eeprom_write_protect=1 in the bootloader config\n  (via usbboot or rpi-eeprom-config) before shipping.\n- Fit the J3 3-4 jumper. The EEPROM is then protected\n  from power-up (CM4 datasheet 5.1).\n\nBootloader update:\n- Remove J3 3-4, update via usbboot or self-update,\n  then refit the jumper.\n\nWhy not a GPIO with a pull-down: CM4 EEPROM updates run\nonly via usbboot or bootloader self-update (datasheet\n6.3), before Linux can drive a GPIO, so the pin could\nnever be released for an update."
 		(exclude_from_sim no)
@@
 		)
 	)
-	(text "I2C PULL-UPS\nI2C1: GPIO2 = I2C1_SDA (J4-24), GPIO3 = I2C1_SCL (J4-22)\nPulled up to 3.3 V (GPIO_VREF) by 1.8 kΩ inside the CM4\n(CM4 datasheet section 2.5, pins 56/58). No board pull-ups\nare needed. R20/R21 (2.2k, fitted via H5/H6) are optional.\n\nI2C0: GPIO0 = ID_SD (J4-22), GPIO1 = ID_SC (J4-23)\nNo I2C pull-ups on the CM4, only the BCM2711's weak reset\npull-ups (33-73 kΩ). If J4-22/23 are used as an I2C bus, the\ndevice on J4 must supply the pull-ups (2.2k-4.7k to 3.3 V)."
+	(text "I2C PULL-UPS\nI2C1: GPIO2 = I2C1_SDA (J4-24), GPIO3 = I2C1_SCL (J4-22)\nPulled up to 3.3 V (GPIO_VREF) by 1.8 kΩ inside the CM4\n(CM4 datasheet section 2.5, pins 56/58). No board pull-ups\nare needed. R20/R21 (2.2k, fitted via H5/H6) are optional."
 		(exclude_from_sim no)
 		(at 220.98 129.54 0)
@@
 	(text "AIN0 / AIN1 (J4-2 / J4-4), field wired, to CM4\nAnalogIP0/1 (MxL7704 ADC). Measures 0 to 2.55 V (8-bit).\nSurvives +/-24 V either polarity: R7/R6 10k series\n+ D4/D5 BAT54S clamps to GND and 3V3_CM4 (RCM4 sheet)\nhold the pins within -0.3 V / +3.6 V (abs max -0.3/+6.0).\nError: ADC input < 1 uA x 10k = 10 mV, plus clamp leakage\n(up to ~1-2 % hot). With the CM4 off, a driven input feeds\n< 0.3 mA (at 6 V) into 3V3_CM4 through the upper clamp."
 		(exclude_from_sim no)
-		(at 55.626 138.176 0)
+		(at 60.452 108.712 0)
 		(effects
 			(font
@@
 		)
 	)
-	(text "GPIO0 / GPIO1 (J4-13 / J4-10)\nCM4 pins 36 (ID_SD = GPIO0) and 35 (ID_SC = GPIO1). This is the\nI2C0 bus the firmware normally uses to look for a HAT EEPROM and to\ncontrol CSI0/DSI0 cameras and displays. This board has no HAT, camera\nor display, so the pins are free for general use.\n\nTo use them as GPIO, add to config.txt (CM4 datasheet section 2.10):\n  force_eeprom_read=0\n  disable_poe_fan=1\nWithout these, the firmware drives the bus at boot to look for an\nEEPROM, and anything wired to these pins sees I2C activity.\n\n- Both pins are pulled up (high) at reset.\n- 3.3 V logic. Not 5 V tolerant.\n- They can also be used as an I2C bus (I2C0: GPIO0 = SDA,\n  GPIO1 = SCL). Add external pull-ups if you do.\n"
-		(exclude_from_sim no)
-		(at 54.356 106.934 0)
-		(effects
-			(font
-				(size 1.016 1.016)
-			)
-			(justify left)
-		)
-	)
