File: kicad/usb2.kicad_sch (KiCad schematic)
At the start: 9 parts, among them U20 74LVC1G07SE-7

Commit message: Ready to start layout
Parts:
- renumbered D56 to D24, R8 to R59, R137 to R60, R6 to R61, R7 to R62, R9 to R63, TP20 to TP28, U20 to U17
Other:
- note added: "U17 is open-drain, powered from 3V3_CM4. With the CM4 off, Y is high-Z and R60 is unpowered, so U2 Sel and CM4 USB_OTG_ID are never driven (CM4 datasheet 5.1). 74LVC Ioff: A tolerates VBUS_DET at VCC = 0."
- note added: "USB_OTG_ID: high = CM4 device mode (rpiboot), low/GND = CM4 host. Needs otg_mode=1 in config.txt. USBC1 VBUS: 5.0 V nom (4.75 V min / 5.5 V max). No USB-PD controller; CC has 5.1 kΩ Rd only. VBUS detect: R59/R61 (2.75 V max) -> U17 open-drain -> USB_OTG_ID. VBUS current: 1.25 mA continuous / 1.25 mA peak. VBUS survives 6.0 V DC (D24 SMF6.0A stand-off), surges clamped to 10.3 V; -0.7 V (D24 forwar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"
- note removed: "U20 is open-drain, powered from 3V3_CM4. With the CM4 off, Y is high-Z and R137 is unpowered, so U3 Sel and CM4 USB_OTG_ID are never driven (CM4 datasheet 5.1). 74LVC Ioff: A tolerates VBUS_DET at VCC = 0."
- note removed: "USB_OTG_ID: high = CM4 device mode (rpiboot), low/GND = CM4 host. Needs otg_mode=1 in config.txt. USBC1 VBUS: 5.0 V nom (4.75 V min / 5.5 V max). No USB-PD controller; CC has 5.1 kΩ Rd only. VBUS detect: R8/R6 (2.75 V max) -> U20 open-drain -> USB_OTG_ID. VBUS current: 1.25 mA continuous / 1.25 mA peak. VBUS survives 6.0 V DC (D56 SMF6.0A stand-off), surges clamped to 10.3 V; -0.7 V (D56 forward)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"
Changed lines of the file:
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@@
 		)
 	)
-	(text "U20 is open-drain, powered from 3V3_CM4. With the CM4 off, Y is\nhigh-Z and R137 is unpowered, so U3 Sel and CM4 USB_OTG_ID are never\ndriven (CM4 datasheet 5.1). 74LVC Ioff: A tolerates VBUS_DET at VCC = 0."
+	(text "U17 is open-drain, powered from 3V3_CM4. With the CM4 off, Y is\nhigh-Z and R60 is unpowered, so U2 Sel and CM4 USB_OTG_ID are never\ndriven (CM4 datasheet 5.1). 74LVC Ioff: A tolerates VBUS_DET at VCC = 0."
 		(exclude_from_sim no)
 		(at 115.824 63.5 0)
@@
 		)
 	)
-	(text "USB_OTG_ID: high = CM4 device mode (rpiboot), \nlow/GND = CM4 host. Needs otg_mode=1 in config.txt.\nUSBC1 VBUS: 5.0 V nom (4.75 V min / 5.5 V max).\nNo USB-PD controller; CC has 5.1 kΩ Rd only.\nVBUS detect: R8/R6 (2.75 V max) -> U20 open-drain -> USB_OTG_ID.\nVBUS current: 1.25 mA continuous / 1.25 mA peak.\nVBUS survives 6.0 V DC (D56 SMF6.0A stand-off), surges\nclamped to 10.3 V; -0.7 V (D56 forward). U20 A sees half via R8/R6."
+	(text "USB_OTG_ID: high = CM4 device mode (rpiboot), \nlow/GND = CM4 host. Needs otg_mode=1 in config.txt.\nUSBC1 VBUS: 5.0 V nom (4.75 V min / 5.5 V max).\nNo USB-PD controller; CC has 5.1 kΩ Rd only.\nVBUS detect: R59/R61 (2.75 V max) -> U17 open-drain -> USB_OTG_ID.\nVBUS current: 1.25 mA continuous / 1.25 mA peak.\nVBUS survives 6.0 V DC (D24 SMF6.0A stand-off), surges\nclamped to 10.3 V; -0.7 V (D24 forward). U17 A sees half via R59/R61."
 		(exclude_from_sim no)
 		(at 26.67 81.788 0)
@@
 		(in_pos_files no)
 		(dnp no)
-		(property "Reference" "TP20"
+		(property "Reference" "TP28"
 			(at 54.61 38.862 0)
 			(show_name no)
@@
 			(project "cm4-robo-controller"
 				(path "/c1285fbe-5f56-49a8-9041-410713cbe619/3cc0f123-2315-4414-aa85-3a1a0bb694eb/d3e40802-8c80-491e-9238-e962cd612968/47c45030-5e0e-4373-90dd-e8e713456a1d"
-					(reference "TP20")
+					(reference "TP28")
 					(unit 1)
 				)
@@
 		(in_pos_files yes)
 		(dnp no)
-		(property "Reference" "R9"
+		(property "Reference" "R63"
 			(at 47.244 67.31 0)
 			(show_name no)
@@
 			(project "cm4-robo-controller"
 				(path "/c1285fbe-5f56-49a8-9041-410713cbe619/3cc0f123-2315-4414-aa85-3a1a0bb694eb/d3e40802-8c80-491e-9238-e962cd612968/47c45030-5e0e-4373-90dd-e8e713456a1d"
-					(reference "R9")
+					(reference "R63")
 					(unit 1)
 				)
@@
 		(in_pos_files yes)
 		(dnp no)
-		(property "Reference" "R8"
+		(property "Reference" "R59"
 			(at 49.53 39.878 90)
 			(show_name no)
@@
 			(project "cm4-robo-controller"
 				(path "/c1285fbe-5f56-49a8-9041-410713cbe619/3cc0f123-2315-4414-aa85-3a1a0bb694eb/d3e40802-8c80-491e-9238-e962cd612968/47c45030-5e0e-4373-90dd-e8e713456a1d"
-					(reference "R8")
+					(reference "R59")
 					(unit 1)
 				)
@@
 		(dnp no)
 		(fields_autoplaced yes)
-		(property "Reference" "R6"
+		(property "Reference" "R61"
 			(at 129.54 54.102 90)
 			(show_name no)
@@
 			(project "cm4-robo-controller"
 				(path "/c1285fbe-5f56-49a8-9041-410713cbe619/3cc0f123-2315-4414-aa85-3a1a0bb694eb/d3e40802-8c80-491e-9238-e962cd612968/47c45030-5e0e-4373-90dd-e8e713456a1d"
-					(reference "R6")
+					(reference "R61")
 					(unit 1)
 				)
@@
 		(in_pos_files yes)
 		(dnp no)
-		(property "Reference" "R7"
+		(property "Reference" "R62"
 			(at 40.894 67.31 0)
 			(show_name no)
@@
 			(project "cm4-robo-controller"
 				(path "/c1285fbe-5f56-49a8-9041-410713cbe619/3cc0f123-2315-4414-aa85-3a1a0bb694eb/d3e40802-8c80-491e-9238-e962cd612968/47c45030-5e0e-4373-90dd-e8e713456a1d"
-					(reference "R7")
+					(reference "R62")
 					(unit 1)
 				)
@@
 		(in_pos_files yes)
 		(dnp no)
-		(property "Reference" "R137"
+		(property "Reference" "R60"
 			(at 181.61 44.958 90)
 			(show_name no)
@@
 			(project "cm4-robo-controller"
 				(path "/c1285fbe-5f56-49a8-9041-410713cbe619/3cc0f123-2315-4414-aa85-3a1a0bb694eb/d3e40802-8c80-491e-9238-e962cd612968/47c45030-5e0e-4373-90dd-e8e713456a1d"
-					(reference "R137")
+					(reference "R60")
 					(unit 1)
 				)
@@
 		(in_pos_files yes)
 		(dnp no)
-		(property "Reference" "D56"
+		(property "Reference" "D24"
 			(at 91.44 45.974 0)
 			(show_name no)
@@
 			(project "cm4-robo-controller"
 				(path "/c1285fbe-5f56-49a8-9041-410713cbe619/3cc0f123-2315-4414-aa85-3a1a0bb694eb/d3e40802-8c80-491e-9238-e962cd612968/47c45030-5e0e-4373-90dd-e8e713456a1d"
-					(reference "D56")
+					(reference "D24")
 					(unit 1)
 				)
@@
 		(in_pos_files yes)
 		(dnp no)
-		(property "Reference" "U20"
+		(property "Reference" "U17"
 			(at 154.94 48.26 90)
 			(show_name no)
@@
 			(project "cm4-robo-controller"
 				(path "/c1285fbe-5f56-49a8-9041-410713cbe619/3cc0f123-2315-4414-aa85-3a1a0bb694eb/d3e40802-8c80-491e-9238-e962cd612968/47c45030-5e0e-4373-90dd-e8e713456a1d"
-					(reference "U20")
+					(reference "U17")
 					(unit 1)
 				)

Commit message: IPC footprint renaming, battery sim added
Parts:
- D24: footprint PCM_JLCPCB:D_SOD-123FL -> MyPartsIPC:SODFL3718X110N
- R59, R60, R61, R62, R63: footprint MyParts:R0402 -> MyPartsIPC:RESC1005X40N
- U17: footprint MyParts:SC-88A_L2.0-W1.3-P0.65-LS2.1-BL -> MyPartsIPC:SOT65P210X110-5N
Changed lines of the file:
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@@
 			)
 		)
-		(property "Footprint" "MyParts:R0402"
+		(property "Footprint" "MyPartsIPC:RESC1005X40N"
 			(at 50.292 67.31 90)
 			(hide yes)
@@
 			)
 		)
-		(property "Footprint" "MyParts:R0402"
+		(property "Footprint" "MyPartsIPC:RESC1005X40N"
 			(at 49.53 43.688 90)
 			(hide yes)
@@
 			)
 		)
-		(property "Footprint" "MyParts:R0402"
+		(property "Footprint" "MyPartsIPC:RESC1005X40N"
 			(at 129.54 52.07 90)
 			(hide yes)
@@
 			)
 		)
-		(property "Footprint" "MyParts:R0402"
+		(property "Footprint" "MyPartsIPC:RESC1005X40N"
 			(at 43.942 67.31 90)
 			(hide yes)
@@
 			)
 		)
-		(property "Footprint" "MyParts:R0402"
+		(property "Footprint" "MyPartsIPC:RESC1005X40N"
 			(at 181.61 46.99 0)
 			(hide yes)
@@
 			)
 		)
-		(property "Footprint" "PCM_JLCPCB:D_SOD-123FL"
+		(property "Footprint" "MyPartsIPC:SODFL3718X110N"
 			(at 86.36 45.72 0)
 			(hide yes)
@@
 			)
 		)
-		(property "Footprint" "MyParts:SC-88A_L2.0-W1.3-P0.65-LS2.1-BL"
+		(property "Footprint" "MyPartsIPC:SOT65P210X110-5N"
 			(at 134.62 49.53 0)
 			(hide yes)

Commit message: PCB: decoupling caps at IC supply pins, route GPS area
- Add 100nF decoupling for U10 (C84) and U17 (C85)
- Move C15, C18, C21, C25, C27, C32 next to their IC supply pins; shift R10
- Route the GPS section: RF_IN, antenna bias, GPS VCC, V_BCKP, local signals, GND/5V plane vias
Parts:
- added C85: 100nF, MyPartsIPC:CAPC1005X55N, symbol MyParts:CL05B104KO5NNNC_ALT
Connections:
- net 3V3_CM4: now also C85.1
- net GND: now also C85.2
Changed lines of the file:
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@@
+		)
+	)
+	(wire
+		(pts
+			(xy 172.72 41.91) (xy 203.2 41.91)
+		)
+		(stroke
+			(width 0)
+			(type default)
+		)
+	)
+	(symbol
+		(lib_id "MyParts:CL05B104KO5NNNC_ALT")
+		(at 203.2 45.72 0)
+		(unit 1)
+		(body_style 1)
+		(exclude_from_sim no)
+		(in_bom yes)
+		(on_board yes)
+		(in_pos_files yes)
+		(dnp no)
+		(property "Reference" "C85"
+			(at 201.93 43.18 0)
+			(show_name no)
+			(do_not_autoplace no)
+			(effects
+				(font
+					(size 1.27 1.27)
+				)
+				(justify right)
+			)
+		)
+		(property "Value" "100nF"
+			(at 201.93 45.72 0)
+			(show_name no)
+			(do_not_autoplace no)
+			(effects
+				(font
+					(size 1.27 1.27)
+				)
+				(justify right)
+			)
+		)
+		(property "Footprint" "MyPartsIPC:CAPC1005X55N"
+			(at 203.2 60.96 0)
+			(hide yes)
+			(show_name no)
+			(do_not_autoplace no)
+			(effects
+				(font
+					(size 1.27 1.27)
+				)
+			)
+		)
+		(property "Datasheet" "${MYPARTS_DATASHEETS}/CL05B104KO5NNNC.pdf"
+			(at 203.2 63.5 0)
+			(hide yes)
+			(show_name no)
+			(do_not_autoplace no)
+			(effects
+				(font
+					(size 1.27 1.27)
+				)
+			)
+		)
+		(property "Description" "100nF 16V X7R ±10% 0402 Multilayer Ceramic Capacitors MLCC - SMD/SMT ROHS"
+			(at 203.2 66.04 0)
+			(hide yes)
+			(show_name no)
+			(do_not_autoplace no)
+			(effects
+				(font
+					(size 1.27 1.27)
+				)
+			)
+		)
+		(property "Manufacturer" "SAMSUNG"
+			(at 203.2 68.58 0)
+			(hide yes)
+			(show_name no)
+			(do_not_autoplace no)
+			(effects
+				(font
+					(size 1.27 1.27)
+				)
+			)
+		)
+		(property "Tolerance" "±10%"
+			(at 203.2 45.72 0)
+			(hide yes)
+			(show_name no)
+			(do_not_autoplace no)
+			(effects
+				(font
+					(size 1.27 1.27)
+				)
+			)
+		)
+		(property "MPN" "CL05B104KO5NNNC"
+			(at 203.2 45.72 0)
+			(hide yes)
+			(show_name no)
+			(do_not_autoplace no)
+			(effects
+				(font
+					(size 1.27 1.27)
+				)
+			)
+		)
+		(property "Voltage Rating" "16V"
+			(at 203.2 45.72 0)
+			(hide yes)
+			(show_name no)
+			(do_not_autoplace no)
+			(effects
+				(font
+					(size 1.27 1.27)
+				)
+			)
+		)
+		(property "LCSC Part" "C1525"
+			(at 203.2 45.72 0)
+			(hide yes)
+			(show_name no)
+			(do_not_autoplace no)
+			(effects
+				(font
+					(size 1.27 1.27)
+				)
+			)
+		)
+		(property "Pkg Type" "SMD 0402"
+			(at 203.2 45.72 0)
+			(hide yes)
+			(show_name no)
+			(do_not_autoplace no)
+			(effects
+				(font
+					(size 1.27 1.27)
+				)
+			)
+		)
+		(pin "1"
+		)
+		(pin "2"
+		)
+		(instances
+			(project "cm4-robo-controller"
+				(path "/c1285fbe-5f56-49a8-9041-410713cbe619/3cc0f123-2315-4414-aa85-3a1a0bb694eb/d3e40802-8c80-491e-9238-e962cd612968/47c45030-5e0e-4373-90dd-e8e713456a1d"
+					(reference "C85")
+					(unit 1)
+				)
+			)
+		)
+	)
+	(symbol
+		(lib_id "power:GND")
+		(at 203.2 49.53 0)
+		(unit 1)
+		(body_style 1)
+		(exclude_from_sim no)
+		(in_bom yes)
+		(on_board yes)
+		(in_pos_files yes)
+		(dnp no)
+		(fields_autoplaced yes)
+		(property "Reference" "#PWR0466"
+			(at 203.2 55.88 0)
+			(hide yes)
+			(show_name no)
+			(do_not_autoplace no)
+			(effects
+				(font
+					(size 1.27 1.27)
+				)
+			)
+		)
+		(property "Value" "GND"
+			(at 203.2 54.61 0)
+			(hide yes)
+			(show_name no)
+			(do_not_autoplace no)
+			(effects
+				(font
+					(size 1.27 1.27)
+				)
+			)
+		)
+		(property "Footprint" ""
+			(at 203.2 49.53 0)
+			(hide yes)
+			(show_name no)
+			(do_not_autoplace no)
+			(effects
+				(font
+					(size 1.27 1.27)
+				)
+			)
+		)
+		(property "Datasheet" ""
+			(at 203.2 49.53 0)
+			(hide yes)
+			(show_name no)
+			(do_not_autoplace no)
+			(effects
+				(font
+					(size 1.27 1.27)
+				)
+			)
+		)
+		(property "Description" "Power symbol creates a global label with name \"GND\" , ground"
+			(at 203.2 49.53 0)
+			(hide yes)
+			(show_name no)
+			(do_not_autoplace no)
+			(effects
+				(font
+					(size 1.27 1.27)
+				)
+			)
+		)
+		(pin "1"
+		)
+		(instances
+			(project "cm4-robo-controller"
+				(path "/c1285fbe-5f56-49a8-9041-410713cbe619/3cc0f123-2315-4414-aa85-3a1a0bb694eb/d3e40802-8c80-491e-9238-e962cd612968/47c45030-5e0e-4373-90dd-e8e713456a1d"
+					(reference "#PWR0466")
+					(unit 1)
+				)
+			)
 		)
 	)

Commit message: Added notes
Other:
- note added: "No fuse on USBC1 VBUS, on purpose: it is a 1.25 mA sense line, not a rail, and nothing on the board draws power from it. The USB host or charger current-limits VBUS at the source, as USB requires. A short (D24 failed, TP28 probe slip) trips the host limit; the 0.3 mm track carries that without fusing. If needed: 0603 PTC (~50 mA) USBC1 -> D24."
Changed lines of the file:
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@@
 	(rectangle
 		(start 25.4 25.4)
-		(end 99.06 91.44)
+		(end 104.14 105.41)
 		(stroke
 			(width 0)
@@
 		)
 	)
+	(text "No fuse on USBC1 VBUS, on purpose: it is a 1.25 mA sense line, not a\nrail, and nothing on the board draws power from it. The USB host or\ncharger current-limits VBUS at the source, as USB requires. A short\n(D24 failed, TP28 probe slip) trips the host limit; the 0.3 mm track\ncarries that without fusing. If needed: 0603 PTC (~50 mA) USBC1 -> D24."
+		(exclude_from_sim no)
+		(at 27.178 94.234 0)
+		(effects
+			(font
+				(size 1.27 1.27)
+			)
+			(justify left top)
+		)
+	)
 	(text "USB_OTG_ID: high = CM4 device mode (rpiboot), \nlow/GND = CM4 host. Needs otg_mode=1 in config.txt.\nUSBC1 VBUS: 5.0 V nom (4.75 V min / 5.5 V max).\nNo USB-PD controller; CC has 5.1 kΩ Rd only.\nVBUS detect: R59/R61 (2.75 V max) -> U17 open-drain -> USB_OTG_ID.\nVBUS current: 1.25 mA continuous / 1.25 mA peak.\nVBUS survives 6.0 V DC (D24 SMF6.0A stand-off), surges\nclamped to 10.3 V; -0.7 V (D24 forward). U17 A sees half via R59/R61."
 		(exclude_from_sim no)
-		(at 26.67 81.788 0)
+		(at 27.178 84.836 0)
 		(effects
 			(font
