File: kicad/power_5v.kicad_sch (KiCad schematic)
At the start: 29 parts, among them U15 AP64501SP-13

Commit message: U15 replacement due to low inventory
Parts:
- R98: renamed from C54; value 100nF -> 174kΩ; footprint MyPartsIPC:CAPC1005X55N -> MyPartsIPC:RESC1005X40N; symbol MyParts:CL05B104KO5NNNC_ALT -> MyParts:0402WGF1743TCE; LCSC Part C1525 -> C26994; MPN CL05B104KO5NNNC -> 0402WGF1743TCE; Manufacturer SAMSUNG -> UNI-ROYAL; Tolerance ±10% -> ±1%; Voltage Rating 16V -> 50V
- U15: value AP64501SP-13 -> AP64500SP-13; symbol MyParts:AP64501SP-13 -> MyParts:AP64500SP-13; LCSC Part C2071517 -> C2070920; MPN AP64501SP-13 -> AP64500SP-13
Other:
- note added: "12V to 5V Buck - AP64500 (5A, 575kHz set by R98, 0.8V reference) Vout = 5.16V, designed for 3A. Input 8.3V-19V (eFuse UVLO cuts in at 8.3V, OVP cuts out at 17.5-19V). EN pulled up to VIN by R65 (100k): starts automatically, the eFuse upstream provides the UVLO. TP30 on EN lets a test fixture hold the buck off. Output voltage set by the FB divider Vout = 0.8V x (1 + R42/R44) = 0.8 x (1 + 12k/2.2k)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"
- note added: "U15 SUBSTITUTION (2026-10-27) Preferred part: AP64501SP-13 (LCSC C2071517), fixed 570kHz, adjustable soft-start. It is out of stock (JLCPCB 1 pc, Mouser 0, DigiKey 0), so AP64500SP-13 (C2070920) is fitted. Same die, pinout and SO-8EP footprint; only pin 4 differs: SS on the AP64501, RT/CLK on the AP64500. Loop gm, current sense, Vref, limits and compensation are identical, so R42/R44, R43/C56 and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"
- note removed: "12V to 5V Buck - AP64501 (5A, 570kHz, 0.8V reference) Vout = 5.16V, designed for 3A. Input 8.3V-19V (eFuse UVLO cuts in at 8.3V, OVP cuts out at 17.5-19V). EN pulled up to VIN by R65 (100k): starts automatically, the eFuse upstream provides the UVLO. TP30 on EN lets a test fixture hold the buck off. Output voltage set by the FB divider Vout = 0.8V x (1 + R42/R44) = 0.8 x (1 + 12k/2.2k) = 5.16V Co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"
Changed lines of the file:
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@@
 	(generator_version "10.0")
 	(paper "A4")
+	(text "U15 SUBSTITUTION (2026-10-27)\nPreferred part: AP64501SP-13 (LCSC C2071517), fixed 570kHz, adjustable soft-start.\nIt is out of stock (JLCPCB 1 pc, Mouser 0, DigiKey 0), so AP64500SP-13 (C2070920) is fitted.\nSame die, pinout and SO-8EP footprint; only pin 4 differs: SS on the AP64501, RT/CLK on the\nAP64500. Loop gm, current sense, Vref, limits and compensation are identical, so R42/R44,\nR43/C56 and L2 are unchanged.\nR98 174k sets 575kHz; spread-spectrum stays on. The external-clock sync is not used\n(it needs a >3.5V clock and turns spread-spectrum off).\nTo go back to the AP64501: fit AP64501SP-13 and replace R98 with a 100nF 0402 cap\n(CL05B104KO5NNNC, C1525) for the ~20ms soft-start."
+		(exclude_from_sim no)
+		(at 152.4 130.81 0)
+		(effects
+			(font
+				(size 1.27 1.27)
+			)
+			(justify left top)
+		)
+	)
 	(text "12V to 5V"
 		(exclude_from_sim no)
@@
 		)
 	)
-	(text "12V to 5V Buck - AP64501 (5A, 570kHz, 0.8V reference)\nVout = 5.16V, designed for 3A. Input 8.3V-19V (eFuse UVLO cuts in at 8.3V, OVP cuts out at 17.5-19V).\nEN pulled up to VIN by R65 (100k): starts automatically, the eFuse upstream provides\nthe UVLO. TP30 on EN lets a test fixture hold the buck off.\n\nOutput voltage set by the FB divider\n\nVout = 0.8V x (1 + R42/R44) = 0.8 x (1 + 12k/2.2k) = 5.16V\nCorners 5.10-5.22V (Vref 792-808mV, R42/R44 0.1%). Worst-case USB VBUS\n= 5.10V - 40mV load reg - 1.908A x 135mΩ (U4) = 4.81V >= 4.75V;\nmax 5.22V stays within the CM4 5.25V limit. 1% resistors cannot meet both.\nR42 12k   0.1% thin film  top leg, 5V to FB\nR44 2.2k  0.1% thin film  bottom leg, FB to GND\nC46 DNP 470pF optional feedforward across R42 for transient tuning\n              (datasheet example 47pF across 115k, scaled for R42 = 12k)\n\nLoop compensation\n\nR43 20k + C56 1.2nF  series RC on COMP sets the loop response\nC55 DNP 33pF         optional HF pole (datasheet Table 1, 5V), fit only if needed\n\nGate drive and soft-start\n\nC40 100nF  bootstrap cap, BST to SW - powers the high-side FET driver\nR41 10R    boot resistor, slows the SW rising edge to cut EMI\nC54 100nF  soft-start; the internal 4uA source gives a ~20ms ramp\n\nInput bulk and bypass\n\nC48-C53  6 x 10uF 35V  bulk; carries ~1.5A RMS ripple at 3A out\nC47      0.1uF         HF bypass, place closest to VIN/GND\n\nOutput filter\n\nL2 3.3uH SRP7028A-3R3M  Bourns molded, 6A Irms, 12A Isat, 30mΩ DCR\n                     with 570kHz gives 1.56A p-p ripple at 12V in\n                     (2.0A p-p at 19V in; peak coil current 4.0A at 3A load)\n                     Isat 12A > U15 peak current limit (9.2A max), so L2\n                     does not saturate during overload before hiccup\nC41-C44 4 x 10uF 10V ceramic, low ESR\nC45 100uF 6.3V       polymer bulk for load steps; 5.16V = 82% of rating\n"
+	(text "12V to 5V Buck - AP64500 (5A, 575kHz set by R98, 0.8V reference)\nVout = 5.16V, designed for 3A. Input 8.3V-19V (eFuse UVLO cuts in at 8.3V, OVP cuts out at 17.5-19V).\nEN pulled up to VIN by R65 (100k): starts automatically, the eFuse upstream provides\nthe UVLO. TP30 on EN lets a test fixture hold the buck off.\n\nOutput voltage set by the FB divider\n\nVout = 0.8V x (1 + R42/R44) = 0.8 x (1 + 12k/2.2k) = 5.16V\nCorners 5.10-5.22V (Vref 792-808mV, R42/R44 0.1%). Worst-case USB VBUS\n= 5.10V - 40mV load reg - 1.908A x 135mΩ (U4) = 4.81V >= 4.75V;\nmax 5.22V stays within the CM4 5.25V limit. 1% resistors cannot meet both.\nR42 12k   0.1% thin film  top leg, 5V to FB\nR44 2.2k  0.1% thin film  bottom leg, FB to GND\nC46 DNP 470pF optional feedforward across R42 for transient tuning\n              (datasheet example 47pF across 115k, scaled for R42 = 12k)\n\nLoop compensation\n\nR43 20k + C56 1.2nF  series RC on COMP sets the loop response\nC55 DNP 33pF         optional HF pole (datasheet Table 1, 5V), fit only if needed\n\nGate drive and soft-start\n\nC40 100nF  bootstrap cap, BST to SW - powers the high-side FET driver\nR41 10R    boot resistor, slows the SW rising edge to cut EMI\nR98 174k   RT/CLK to GND: fsw = 100000/174k = 575kHz (AP64500 Eq. 7);\n           never leave RT/CLK open. Soft-start is fixed at 4ms inside the AP64500\n\nInput bulk and bypass\n\nC48-C53  6 x 10uF 35V  bulk; carries ~1.5A RMS ripple at 3A out\nC47      0.1uF         HF bypass, place closest to VIN/GND\n\nOutput filter\n\nL2 3.3uH SRP7028A-3R3M  Bourns molded, 6A Irms, 12A Isat, 30mΩ DCR\n                     with 575kHz gives 1.55A p-p ripple at 12V in\n                     (2.0A p-p at 19V in; peak coil current 4.0A at 3A load)\n                     Isat 12A > U15 peak current limit (9.2A max), so L2\n                     does not saturate during overload before hiccup\nC41-C44 4 x 10uF 10V ceramic, low ESR\nC45 100uF 6.3V       polymer bulk for load steps; 5.16V = 82% of rating\n"
 		(exclude_from_sim no)
 		(at 30.226 150.622 0)
@@
 	)
 	(symbol
-		(lib_id "MyParts:AP64501SP-13")
+		(lib_id "MyParts:AP64500SP-13")
 		(at 129.54 71.12 0)
 		(unit 1)
@@
 			)
 		)
-		(property "Value" "AP64501SP-13"
+		(property "Value" "AP64500SP-13"
 			(at 130.048 63.5 0)
 			(show_name no)
@@
 			)
 		)
-		(property "Datasheet" "${MYPARTS_DATASHEETS}/AP64501SP-13.pdf"
+		(property "Datasheet" "${MYPARTS_DATASHEETS}/AP64500SP-13.pdf"
 			(at 129.54 86.36 0)
 			(hide yes)
@@
 			)
 		)
-		(property "Description" "-40℃~+85℃ 1 25uA 3.8V~40V 570kHz 5A 800mV~39V Adjustable Buck Built-in Overcurrent Protection, Light load efficient mode, Adjustable soft-start, Cycle-by-cycle current limiting, Hiccup current limiting, External compensation, EMI optimization (spread spectrum) Step-down type Yes SOIC-8-EP DC-DC Converters ROHS"
+		(property "Description" "-40℃~+85℃ 1 25uA 3.8V~40V 100kHz~2.2MHz (RT) 5A 800mV~39V Adjustable Buck Built-in"
 			(at 129.54 71.12 0)
 			(hide yes)
@@
 			)
 		)
-		(property "MPN" "AP64501SP-13"
+		(property "MPN" "AP64500SP-13"
 			(at 129.54 91.44 0)
 			(hide yes)
@@
 			)
 		)
-		(property "LCSC Part" "C2071517"
+		(property "LCSC Part" "C2070920"
 			(at 129.54 93.98 0)
 			(hide yes)
@@
 	)
 	(symbol
-		(lib_id "MyParts:CL05B104KO5NNNC_ALT")
+		(lib_id "MyParts:0402WGF1743TCE")
 		(at 116.84 82.55 0)
 		(unit 1)
@@
 		(dnp no)
 		(fields_autoplaced yes)
-		(property "Reference" "C54"
+		(property "Reference" "R98"
 			(at 119.38 80.0099 0)
 			(show_name no)
@@
 			)
 		)
-		(property "Value" "100nF"
+		(property "Value" "174kΩ"
 			(at 119.38 82.55 0)
 			(show_name no)
@@
 			)
 		)
-		(property "Footprint" "MyPartsIPC:CAPC1005X55N"
+		(property "Footprint" "MyPartsIPC:RESC1005X40N"
 			(at 115.062 82.55 90)
 			(hide yes)
@@
 			)
 		)
-		(property "Datasheet" "${MYPARTS_DATASHEETS}/CL05B104KO5NNNC.pdf"
+		(property "Datasheet" "${MYPARTS_DATASHEETS}/0402WGF1743TCE.pdf"
 			(at 116.84 82.55 0)
 			(hide yes)
@@
 			)
 		)
-		(property "Description" "100nF 16V X7R ±10% 0402 Multilayer Ceramic Capacitors MLCC - SMD/SMT ROHS"
+		(property "Description" "-55℃~+155℃ 174kΩ 50V 62.5mW Thick Film Resistor ±1% ±100ppm/℃ 0402 Chip Resistor - Surface Mount ROHS"
 			(at 116.84 82.55 0)
 			(hide yes)
@@
 			)
 		)
-		(property "Manufacturer" "SAMSUNG"
+		(property "Manufacturer" "UNI-ROYAL"
 			(at 116.84 82.55 0)
 			(hide yes)
@@
 			)
 		)
-		(property "Tolerance" "±10%"
+		(property "Tolerance" "±1%"
 			(at 116.84 82.55 0)
 			(hide yes)
@@
 			)
 		)
-		(property "MPN" "CL05B104KO5NNNC"
+		(property "MPN" "0402WGF1743TCE"
 			(at 116.84 82.55 0)
 			(hide yes)
@@
 			)
 		)
-		(property "Voltage Rating" "16V"
+		(property "Voltage Rating" "50V"
 			(at 116.84 82.55 0)
 			(hide yes)
@@
 			)
 		)
-		(property "LCSC Part" "C1525"
+		(property "LCSC Part" "C26994"
 			(at 116.84 82.55 0)
 			(hide yes)
@@
 			(project "cm4-robo-controller"
 				(path "/c1285fbe-5f56-49a8-9041-410713cbe619/b81204ce-c2fc-430f-9caf-a4f2d6cea5c9/2b73156f-617f-4ddb-9603-19922a26015d"
-					(reference "C54")
+					(reference "R98")
 					(unit 1)
 				)
