File: kicad/i2c.kicad_sch (KiCad schematic)
At the start: 12 parts, among them CN3 SM04B-SRSS-TB (LF)(SN), U20 LTC4311ISC6#TRPBF, U7 LM75BIMX-3/NOPB

Commit message: Update with I2C and new images
Parts:
- C22: LCSC C23733 -> (none); LCSC Part (none) -> C23733; MPN (none) -> CL05A475MP5NRNC; Manufacturer Samsung Electro-Mechanics -> SAMSUNG; Pkg Type (none) -> SMD 0402
- C64, C66: LCSC C1525 -> (none); LCSC Part (none) -> C1525; MPN (none) -> CL05B104KO5NNNC; Manufacturer Samsung Electro-Mechanics -> SAMSUNG; Pkg Type (none) -> SMD 0402
- C65: LCSC C19702 -> (none); LCSC Part (none) -> C19702; MPN (none) -> CL10A106KP8NNNC; Manufacturer Samsung Electro-Mechanics -> SAMSUNG; Pkg Type (none) -> SMD 0603
- D26: MPN (none) -> TPESD0402G05V; Pkg Type (none) -> SMD 0402
- R66: LCSC C25744 -> (none); LCSC Part (none) -> C25744; MPN (none) -> 0402WGF1002TCE; Manufacturer UNI-ROYAL(Uniroyal Elec) -> UNI-ROYAL; Pkg Type (none) -> SMD 0402
- R69: LCSC C25092 -> (none); LCSC Part (none) -> C25092; MPN (none) -> 0402WGF220JTCE; Manufacturer UNI-ROYAL(Uniroyal Elec) -> UNI-ROYAL; Pkg Type (none) -> SMD 0402
- R70: LCSC C25092 -> (none); LCSC Part (none) -> C25092; MPN TPESD0402G05V -> 0402WGF220JTCE; Manufacturer UNI-ROYAL(Uniroyal Elec) -> UNI-ROYAL
Changed lines of the file:
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@@
 			)
 		)
-		(property "Datasheet" "${MYPARTS_DATASHEETS}/TPESD0402G05V.pdf"
+		(property "Datasheet" "${MYPARTS_DATASHEETS}/0402WGF220JTCE.pdf"
 			(at 118.11 115.57 0)
 			(hide yes)
@@
 			)
 		)
-		(property "Description" "5VWM 40VC 0402"
+		(property "Description" "62.5mW Thick Film Resistors 50V ±1% ±100ppm/°C 22Ω 0402 Chip Resistor - Surface Mount ROHS"
 			(at 118.11 115.57 0)
 			(hide yes)
@@
 			)
 		)
-		(property "LCSC" "C25092"
+		(property "LCSC Part" "C25092"
 			(at 118.11 115.57 0)
 			(hide yes)
@@
 			)
 		)
-		(property "Manufacturer" "UNI-ROYAL(Uniroyal Elec)"
+		(property "Manufacturer" "UNI-ROYAL"
 			(at 118.11 115.57 0)
 			(hide yes)
@@
 			)
 		)
-		(property "MPN" "TPESD0402G05V"
+		(property "MPN" "0402WGF220JTCE"
 			(at 118.11 115.57 90)
 			(hide yes)
@@
 			)
 		)
-		(property "Datasheet" "https://www.lcsc.com/datasheet/C558615.pdf?spm=wm.sxq.inf.ggs___wm.ssy.bg.0.xh&lcsc_vid=FFBaV1wHQFldUVICFgBfBVJTQVJWXgBfEQRYBAFQE1YxVlNRQFVXU1JRQVReUTsOAxUeFF5JWBYZEEoKFBINSQcJGk4eFQsCAgIaSgADAwAHC0slRldcU1ZUWQkaCgg%3D"
+		(property "Datasheet" "${MYPARTS_DATASHEETS}/TPESD0402G05V.pdf"
+			(at 129.54 123.19 0)
+			(hide yes)
+			(show_name no)
+			(do_not_autoplace no)
+			(effects
+				(font
+					(size 1.27 1.27)
+				)
+			)
+		)
+		(property "Pkg Type" "SMD 0402"
+			(at 129.54 123.19 0)
+			(hide yes)
+			(show_name no)
+			(do_not_autoplace no)
+			(effects
+				(font
+					(size 1.27 1.27)
+				)
+			)
+		)
+		(property "MPN" "TPESD0402G05V"
 			(at 129.54 123.19 0)
 			(hide yes)
@@
 			)
 		)
+		(property "Pkg Type" "SMD 0603"
+			(at 125.73 63.5 0)
+			(hide yes)
+			(show_name no)
+			(do_not_autoplace no)
+			(effects
+				(font
+					(size 1.27 1.27)
+				)
+			)
+		)
+		(property "MPN" "CL10A106KP8NNNC"
+			(at 125.73 63.5 0)
+			(hide yes)
+			(show_name no)
+			(do_not_autoplace no)
+			(effects
+				(font
+					(size 1.27 1.27)
+				)
+			)
+		)
 		(property "Description" "10V 10uF X5R ±10% 0603 Multilayer Ceramic Capacitors MLCC - SMD/SMT ROHS"
 			(at 125.73 63.5 0)
@@
 			)
 		)
-		(property "LCSC" "C19702"
+		(property "LCSC Part" "C19702"
 			(at 125.73 63.5 0)
 			(hide yes)
@@
 			)
 		)
-		(property "Manufacturer" "Samsung Electro-Mechanics"
+		(property "Manufacturer" "SAMSUNG"
 			(at 125.73 63.5 0)
 			(hide yes)
@@
 			)
 		)
-		(property "Datasheet" "https://www.lcsc.com/datasheet/lcsc_datasheet_2205311900_UNI-ROYAL-Uniroyal-Elec-0402WGF220JTCE_C25092.pdf"
+		(property "Datasheet" "${MYPARTS_DATASHEETS}/0402WGF220JTCE.pdf"
+			(at 118.11 113.03 0)
+			(hide yes)
+			(show_name no)
+			(do_not_autoplace no)
+			(effects
+				(font
+					(size 1.27 1.27)
+				)
+			)
+		)
+		(property "Pkg Type" "SMD 0402"
+			(at 118.11 113.03 0)
+			(hide yes)
+			(show_name no)
+			(do_not_autoplace no)
+			(effects
+				(font
+					(size 1.27 1.27)
+				)
+			)
+		)
+		(property "MPN" "0402WGF220JTCE"
 			(at 118.11 113.03 0)
 			(hide yes)
@@
 			)
 		)
-		(property "LCSC" "C25092"
+		(property "LCSC Part" "C25092"
 			(at 118.11 113.03 0)
 			(hide yes)
@@
 			)
 		)
-		(property "Manufacturer" "UNI-ROYAL(Uniroyal Elec)"
+		(property "Manufacturer" "UNI-ROYAL"
 			(at 118.11 113.03 0)
 			(hide yes)
@@
 			)
 		)
-		(property "Datasheet" "https://www.lcsc.com/datasheet/lcsc_datasheet_2304140030_Samsung-Electro-Mechanics-CL05B104KO5NNNC_C1525.pdf"
+		(property "Datasheet" "${MYPARTS_DATASHEETS}/CL05B104KO5NNNC.pdf"
+			(at 157.48 59.69 0)
+			(hide yes)
+			(show_name no)
+			(do_not_autoplace no)
+			(effects
+				(font
+					(size 1.27 1.27)
+				)
+			)
+		)
+		(property "Pkg Type" "SMD 0402"
+			(at 157.48 59.69 0)
+			(hide yes)
+			(show_name no)
+			(do_not_autoplace no)
+			(effects
+				(font
+					(size 1.27 1.27)
+				)
+			)
+		)
+		(property "MPN" "CL05B104KO5NNNC"
 			(at 157.48 59.69 0)
 			(hide yes)
@@
 			)
 		)
-		(property "LCSC" "C1525"
+		(property "LCSC Part" "C1525"
 			(at 157.48 59.69 0)
 			(hide yes)
@@
 			)
 		)
-		(property "Manufacturer" "Samsung Electro-Mechanics"
+		(property "Manufacturer" "SAMSUNG"
 			(at 157.48 59.69 0)
 			(hide yes)
@@
 			)
 		)
-		(property "Datasheet" "https://www.lcsc.com/datasheet/lcsc_datasheet_2411221126_UNI-ROYAL-Uniroyal-Elec-0402WGF1002TCE_C25744.pdf"
+		(property "Datasheet" "${MYPARTS_DATASHEETS}/0402WGF1002TCE.pdf"
+			(at 80.01 71.12 0)
+			(hide yes)
+			(show_name no)
+			(do_not_autoplace no)
+			(effects
+				(font
+					(size 1.27 1.27)
+				)
+			)
+		)
+		(property "Pkg Type" "SMD 0402"
+			(at 80.01 71.12 0)
+			(hide yes)
+			(show_name no)
+			(do_not_autoplace no)
+			(effects
+				(font
+					(size 1.27 1.27)
+				)
+			)
+		)
+		(property "MPN" "0402WGF1002TCE"
 			(at 80.01 71.12 0)
 			(hide yes)
@@
 			)
 		)
-		(property "LCSC" "C25744"
+		(property "LCSC Part" "C25744"
 			(at 80.01 71.12 0)
 			(hide yes)
@@
 			)
 		)
-		(property "Manufacturer" "UNI-ROYAL(Uniroyal Elec)"
+		(property "Manufacturer" "UNI-ROYAL"
 			(at 80.01 71.12 0)
 			(hide yes)
@@
 			)
 		)
+		(property "Pkg Type" "SMD 0402"
+			(at 153.67 59.69 0)
+			(hide yes)
+			(show_name no)
+			(do_not_autoplace no)
+			(effects
+				(font
+					(size 1.27 1.27)
+				)
+			)
+		)
+		(property "MPN" "CL05A475MP5NRNC"
+			(at 153.67 59.69 0)
+			(hide yes)
+			(show_name no)
+			(do_not_autoplace no)
+			(effects
+				(font
+					(size 1.27 1.27)
+				)
+			)
+		)
 		(property "Description" "10V 4.7uF X5R ±20% 0402 Multilayer Ceramic Capacitors MLCC - SMD/SMT ROHS"
 			(at 153.67 59.69 0)
@@
 			)
 		)
-		(property "LCSC" "C23733"
+		(property "LCSC Part" "C23733"
 			(at 153.67 59.69 0)
 			(hide yes)
@@
 			)
 		)
-		(property "Manufacturer" "Samsung Electro-Mechanics"
+		(property "Manufacturer" "SAMSUNG"
 			(at 153.67 59.69 0)
 			(hide yes)
@@
 			)
 		)
-		(property "Datasheet" "https://www.lcsc.com/datasheet/lcsc_datasheet_2304140030_Samsung-Electro-Mechanics-CL05B104KO5NNNC_C1525.pdf"
+		(property "Datasheet" "${MYPARTS_DATASHEETS}/CL05B104KO5NNNC.pdf"
+			(at 116.84 63.5 0)
+			(hide yes)
+			(show_name no)
+			(do_not_autoplace no)
+			(effects
+				(font
+					(size 1.27 1.27)
+				)
+			)
+		)
+		(property "Pkg Type" "SMD 0402"
+			(at 116.84 63.5 0)
+			(hide yes)
+			(show_name no)
+			(do_not_autoplace no)
+			(effects
+				(font
+					(size 1.27 1.27)
+				)
+			)
+		)
+		(property "MPN" "CL05B104KO5NNNC"
 			(at 116.84 63.5 0)
 			(hide yes)
@@
 			)
 		)
-		(property "LCSC" "C1525"
+		(property "LCSC Part" "C1525"
 			(at 116.84 63.5 0)
 			(hide yes)
@@
 			)
 		)
-		(property "Manufacturer" "Samsung Electro-Mechanics"
+		(property "Manufacturer" "SAMSUNG"
 			(at 116.84 63.5 0)
 			(hide yes)
